File: pcb/cad/analog-front-end.kicad_sch (KiCad schematic)
At the start: 0 parts

Commit message: Analog front-end schematic created
Parts:
- added C?: 330p, symbol Device:C
- added C?: 100n, symbol Device:C
- added R? (x4): 48.7k, Resistor_SMD:R_1206_3216Metric_Pad1.30x1.75mm_HandSolder, symbol Device:R_US
- added R?: 2.49k, Resistor_SMD:R_0805_2012Metric_Pad1.20x1.40mm_HandSolder, symbol Device:R_US
- added R? (x2): 12, Resistor_SMD:R_0805_2012Metric_Pad1.20x1.40mm_HandSolder, symbol Device:R_US
- added R?: 2.7k, symbol Device:R_US
- added R?: 50, symbol Device:R_US
- added R? (x3): 1.5k, Resistor_SMD:R_0805_2012Metric_Pad1.20x1.40mm_HandSolder, symbol Device:R_US
- added R?: 47k, Resistor_SMD:R_0603_1608Metric, symbol Device:R_US
- added R?: 2.49k, Resistor_SMD:R_0805_2012Metric_Pad1.20x1.40mm_HandSolder, symbol Device:R_Small_US
- added U?: AD8421, Package_SO:SOIC-8_3.9x4.9mm_P1.27mm, symbol Amplifier_Instrumentation:AD8421BRZ
- added U? (x3): OPA2227, Package_SO:SOIC-8_3.9x4.9mm_P1.27mm, symbol qds-cv-lib-sym:OPA2227
- added U?: AMC1200, Package_SO:SOP-8_6.62x9.15mm_P2.54mm, symbol qds-cv-lib-sym:AMC1200
Connections:
- net +5VREF: now also R?.2, U?.3 (+)
- net V-DET: now also R?.2, U?.1
- net VOLTAGE-TAP-IN-N: now also R?.1
- net VOLTAGE-TAP-IN-P: now also R?.1
- new net: U?.1 (-), U?.7 (+)
- new net: R?.2, U?.2 (Rg)
- new net: R?.1, U?.3 (Rg)
- new net: U?.4 (+), U?.6 (-)
- new net: R?.1, R?.1, U?.7
- new net: R?.1, R?.2 (x2)
- new net: R?.1, R?.1, R?.2
- new net: C?.1, R?.2, U?.2 (+)
- new net: C?.2, R?.2, U?.3 (-)
- new net: R?.1, R?.2, R?.2
- new net: R?.1, R?.2, U?.2 (-)
- new net: R?.1, R?.2, U?.7
- new net: C?.1, R?.2, U?.5 (+)
- new net: R?.1, U?.6 (-)
- new net +14V: U?.8 (V+), U?.8 (Vs+)
- new net +5V: U?.8 (V2+)
- new net +5V-ISO-A: U?.1 (V1+)
- new net -14V: U?.4 (V-), U?.5 (Vs-)
- new net Earth: C?.2, R?.1, U?.5 (V2-), U?.6 (Ref)
- new net GND-ISO-A: U?.4 (V1-)
- new net V-MON: R?.2

Commit message: Comparator circuit included on the front-end sheet
Parts:
- added R?: 5k, symbol Device:R_US
- added R? (x2): 620, symbol Device:R_US
- added RV?: 5k, symbol Device:R_Potentiometer_Trim_US
- added U? (x3): LM393-N, Package_SO:SOIC-8_3.9x4.9mm_P1.27mm, symbol qds-cv-lib-sym:LM393-N
Connections:
- net +14V: now also U?.8 (V+)
- net +5V: now also R?.1, R?.1
- net -14V: no longer U?.4 (V-)
- net Earth: now also U?.4 (V-), R?.2, U?.4 (V-)
- net V-DET: now also U?.2 (-), U?.5 (+)
- net V-MON: no longer names the net of R?.2
- new net: R?.1, RV?.3, U?.6 (-)
- new net: R?.2, RV?.1, RV?.2, U?.3 (+)
- new net V-VAL: R?.2, U?.1, U?.7
Other:
- moved on the sheet: C?, R?, U?, U?A, U?B, U?C

Commit message: Included power supplies circuits and +5V-REF RC circuit in analog front-end
Parts:
- added C?: 100n, Capacitor_SMD:C_0603_1608Metric_Pad1.08x0.95mm_HandSolder, symbol Device:C
- added R?: 60k4, Resistor_SMD:R_0603_1608Metric_Pad0.98x0.95mm_HandSolder, symbol Device:R_US
- C?: footprint (none) -> Capacitor_SMD:C_0603_1608Metric_Pad1.08x0.95mm_HandSolder; CNPEM Code (none) -> AP107349; Manufacturer (none) -> TDK; Part Number (none) -> C1608X7R1H104K080AA; Vendor Link (none) -> https://br.mouser.com/ProductDetail/TDK/C1608X7R1H104K080AA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
Connections:
- net +5VREF: now also R?.1; no longer R?.2, U?.3 (+)
- net Earth: now also C?.2
- new net: C?.1, R?.2, R?.2, U?.3 (+)
Other:
- moved on the sheet: C?, R?, U?B

Commit message: specify components used in front-end, validation and power circuits, except resistors
Parts:
- C?: footprint (none) -> Capacitor_SMD:C_0805_2012Metric_Pad1.18x1.45mm_HandSolder; Manufacturer (none) -> Prosperity Dielectrics Co; Part Number (none) -> MA0805CG-331J-500PR
- R?: footprint Resistor_SMD:R_0603_1608Metric -> Resistor_SMD:R_0603_1608Metric_Pad0.98x0.95mm_HandSolder; Vendor Link (none) -> https://www.digikey.com/en/products/detail/ERA-3AEB473V/P47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
- RV?: footprint (none) -> Potentiometer_SMD:Potentiometer_Bourns_3224X_Vertical; Manufacturer (none) -> Bourns; Part Number (none) -> 3224X-1-502E
Changed lines of the file:
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@@
       (effects (font (size 1.27 1.27)) (justify left))
     )
-    (property "Footprint" "" (id 2) (at 100.0252 67.31 0)
-      (effects (font (size 1.27 1.27)) hide)
-    )
-    (property "Datasheet" "~" (id 3) (at 99.06 63.5 0)
+    (property "Footprint" "Capacitor_SMD:C_0805_2012Metric_Pad1.18x1.45mm_HandSolder" (id 2) (at 100.0252 67.31 0)
+      (effects (font (size 1.27 1.27)) hide)
+    )
+    (property "Datasheet" "https://download.datasheets.com/pdfs/2015/3/22/4/27/47/982/pdc_/manual/ma0603cg-151j-500prg.pdf" (id 3) (at 99.06 63.5 0)
+      (effects (font (size 1.27 1.27)) hide)
+    )
+    (property "Description" "Ceramic Capacitor 330 pF 50V 5% SMD 0805 NPO" (id 4) (at 99.06 63.5 0)
+      (effects (font (size 1.27 1.27)) hide)
+    )
+    (property "Manufacturer" "Prosperity Dielectrics Co" (id 5) (at 99.06 63.5 0)
+      (effects (font (size 1.27 1.27)) hide)
+    )
+    (property "Part Number" "MA0805CG-331J-500PR" (id 6) (at 99.06 63.5 0)
       (effects (font (size 1.27 1.27)) hide)
     )
@@
       (effects (font (size 1.27 1.27)) (justify right))
     )
-    (property "Footprint" "" (id 2) (at 58.42 148.59 0)
-      (effects (font (size 1.27 1.27)) hide)
-    )
-    (property "Datasheet" "~" (id 3) (at 58.42 148.59 0)
+    (property "Footprint" "Potentiometer_SMD:Potentiometer_Bourns_3224X_Vertical" (id 2) (at 58.42 148.59 0)
+      (effects (font (size 1.27 1.27)) hide)
+    )
+    (property "Datasheet" "https://www.bourns.com/docs/Product-Datasheets/3224.pdf" (id 3) (at 58.42 148.59 0)
+      (effects (font (size 1.27 1.27)) hide)
+    )
+    (property "Manufacturer" "Bourns" (id 4) (at 58.42 148.59 0)
+      (effects (font (size 1.27 1.27)) hide)
+    )
+    (property "Part Number" "3224X-1-502E" (id 5) (at 58.42 148.59 0)
       (effects (font (size 1.27 1.27)) hide)
     )
@@
     (property "Reference" "R?" (id 0) (at 240.03 43.18 90))
     (property "Value" "47k" (id 1) (at 240.03 45.72 90))
-    (property "Footprint" "Resistor_SMD:R_0603_1608Metric" (id 2) (at 240.284 48.514 90)
+    (property "Footprint" "Resistor_SMD:R_0603_1608Metric_Pad0.98x0.95mm_HandSolder" (id 2) (at 240.284 48.514 90)
       (effects (font (size 1.27 1.27)) hide)
     )
@@
       (effects (font (size 1.27 1.27)) hide)
     )
+    (property "Description" "Resistor 47k 0.1% 0.1W SMD 0603" (id 7) (at 240.03 49.53 0)
+      (effects (font (size 1.27 1.27)) hide)
+    )
+    (property "Vendor Link" "https://www.digikey.com/en/products/detail/ERA-3AEB473V/P47KDBCT-ND/1466092" (id 8) (at 240.03 49.53 0)
+      (effects (font (size 1.27 1.27)) hide)
+    )

Commit message: create schematic for trigger aggregation, indication and actuation circuits
Parts:
- U? (x3): Part Number (none) -> LM393N
Changed lines of the file:
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@@
+      (effects (font (size 1.27 1.27)) hide)
+    )
+    (property "Part Number" "LM393N" (id 4) (at 93.98 142.24 0)
       (effects (font (size 1.27 1.27)) hide)
     )
@@
       (effects (font (size 1.27 1.27)) hide)
     )
+    (property "Part Number" "LM393N" (id 4) (at 93.98 154.94 0)
+      (effects (font (size 1.27 1.27)) hide)
+    )
     (pin "1")
     (pin "2")
@@
       (effects (font (size 1.27 1.27)) hide)
     )
+    (property "Part Number" "LM393N" (id 4) (at 135.89 179.07 0)
+      (effects (font (size 1.27 1.27)) hide)
+    )

Commit message: Created hierarchy connections, updates on analog-front-end and included 5V reference circuit
Parts:
- removed R? (x2): 620, symbol Device:R_US
- added C? (x9): 100n, Capacitor_SMD:C_0603_1608Metric_Pad1.08x0.95mm_HandSolder, symbol Device:C
- added C? (x2): 10u, Capacitor_SMD:C_0805_2012Metric_Pad1.18x1.45mm_HandSolder, symbol Device:C
- added D? (x2): BAT54S, Package_TO_SOT_SMD:SOT-23, symbol Diode:BAT54S
- added J?: Conn_Coaxial, symbol Connector:Conn_Coaxial
- added R? (x2): 620, Resistor_SMD:R_0805_2012Metric_Pad1.20x1.40mm_HandSolder, symbol Device:R_US
- added R?: NP, Resistor_SMD:R_0805_2012Metric_Pad1.20x1.40mm_HandSolder, symbol Device:R_US
Connections:
- net +14V: now also C?.1, C?.1, C?.1
- net +5V: now also C?.1, C?.1, R?.2
- net +5V-ISO-A: now also C?.1, C?.1, D?.2, D?.2, R?.2
- net -14V: now also U?.4 (V-), C?.1, C?.2
- net Earth: now also C?.1, C?.2, C?.2, C?.2, C?.2, C?.2, C?.2, C?.2, C?.2, J?.2 (Ext), R?.1; no longer U?.4 (V-)
- net GND-ISO-A: now also C?.2, C?.2, D?.1, D?.1
- net at C?.1, R?.2, U?.2 (+): now also D?.3, R?.1
- net at C?.2, R?.2, U?.3 (-): now also D?.3
- net at RV?.3, U?.6 (-): now also C?.1, R?.2
- net at R?.2: now also J?.1 (In)
- net at RV?.1, RV?.2, U?.3 (+): now also C?.1, R?.1
Other:
- note added: "BNC monitor Output range: ±10 V"
- note added: "Input overvoltage protection: ±425 V"
- note added: "Isolated detection channel"
- note added: "Place next to AMC1200 supply pins"
- note added: "Place next to LM393 supply pins"
- note added: "Place next to OPA2227 supply pins"
- note added: "Pull-up resistor to rest broken-wire protection"
- note removed: "Isolated analog front-end"
- moved on the sheet: C?, R?, RV?, U?, U?A, U?B, U?C

Commit message: update components specification
Parts:
- R?: value 5k -> 4.7k; footprint (none) -> Resistor_SMD:R_1206_3216Metric_Pad1.30x1.75mm_HandSolder; Part Number (none) -> RC1206FR-074K7L
Changed lines of the file:
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@@
       (effects (font (size 1.27 1.27)) (justify right))
     )
-    (property "Value" "5k" (id 1) (at 105.41 135.8899 0)
+    (property "Value" "4.7k" (id 1) (at 111.76 134.6199 0)
       (effects (font (size 1.27 1.27)) (justify right))
     )
-    (property "Footprint" "" (id 2) (at 101.854 134.874 90)
+    (property "Footprint" "Resistor_SMD:R_1206_3216Metric_Pad1.30x1.75mm_HandSolder" (id 2) (at 108.204 133.604 90)
       (effects (font (size 1.27 1.27)) hide)
     )
-    (property "Datasheet" "~" (id 3) (at 102.87 134.62 0)
+    (property "Datasheet" "https://media.digikey.com/pdf/Data%20Sheets/Samsung%20PDFs/RC_Series_ds.pdf" (id 3) (at 109.22 133.35 0)
       (effects (font (size 1.27 1.27)) hide)
     )
+    (property "Part Number" "RC1206FR-074K7L" (id 4) (at 109.22 133.35 0)
+      (effects (font (size 1.27 1.27)) hide)
+    )

Commit message: Update componentes fields and reference circuit
Parts:
- D? (x2): CNPEM Code (none) -> AP105030; Manufacturer (none) -> On Semiconductor; Part Number (none) -> BAT54S; Vendor Link (none) -> https://www.digikey.com/en/products/detail/onsemi/BAT54SLT1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
- J?: footprint (none) -> Connector_Coaxial:BNC_Amphenol_B6252HB-NPP3G-50_Horizontal; CNPEM Code (none) -> AP107369; Manufacturer (none) -> Molex; Part Number (none) -> 0731375003; Vendor Link (none) -> https://www.digikey.com/en/products/detail/molex/0731375003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
- R?: Manufacturer (none) -> Yageo; Vendor Link (none) -> https://www.digikey.com/en/products/detail/yageo/RC1206FR-0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
- R? (x2): Vendor Link (none) -> https://www.digikey.com/en/products/detail/te-connectivity-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
- R? (x2): Vendor Link (none) -> https://www.digikey.in/en/products/detail/te-connectivity-p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
- R?: footprint (none) -> Resistor_SMD:R_1206_3216Metric_Pad1.30x1.75mm_HandSolder; CNPEM Code (none) -> MC128223; Manufacturer (none) -> Yageo; Part Number (none) -> RT1206BRD072K7L; Vendor Link (none) -> https://www.digikey.com/en/products/detail/yageo/RT1206BRD0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
- R?: value 50 -> 49.9; footprint (none) -> Resistor_SMD:R_0805_2012Metric_Pad1.20x1.40mm_HandSolder; CNPEM Code (none) -> AP108391; Manufacturer (none) -> Yageo; Part Number (none) -> RT0805DRE0749R9L; Vendor Link (none) -> https://www.digikey.com/en/products/detail/yageo/RT0805DRE0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
- R?: value 60k4 -> 60.4k; Manufacturer Panasonic -> Panasonic Electronic Components; Vendor Link (none) -> https://br.mouser.com/ProductDetail/Panasonic/ERA-3AEB6042V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
- R?: Manufacturer Panasonic -> Panasonic Electronic Components
- RV?: Vendor Link (none) -> https://br.mouser.com/ProductDetail/Bourns/3224X-1-502E?qs=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
Other:
- title: (none) -> Isolation Detection Channel
