File: pcb/cad/analog-front-end.kicad_sch (KiCad schematic)
At the start: 50 parts, among them J201 Conn_Coaxial, U201 OPA2227, U202 AMC1200, U203 AD8421, U204 LM393-N

Commit message: Remake some logic connections and update PCB
Connections:
- net GND-ISO-A: now also R207.2, R211.2, R212.1
Changed lines of the file:
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@@
     (pin "8")
+  )
+  (symbol (lib_id "qds-cv-lib-sym:GND-ISO-A") (at 74.93 80.01 0) (unit 1)
+    (in_bom yes) (on_board yes) (fields_autoplaced)
+    (property "Reference" "#PWR?" (id 0) (at 74.93 86.36 0)
+      (effects (font (size 1.27 1.27)) hide)
+    )
+    (property "Value" "GND-ISO-A" (id 1) (at 74.93 85.09 0))
+    (property "Footprint" "" (id 2) (at 74.93 80.01 0)
+      (effects (font (size 1.27 1.27)) hide)
+    )
+    (property "Datasheet" "" (id 3) (at 74.93 80.01 0)
+      (effects (font (size 1.27 1.27)) hide)
+    )
+    (pin "1")
   )
   (symbol (lib_id "Device:R_US") (at 226.06 124.46 90) (unit 1)

Commit message: Last commit before flipping PTH components
Parts:
- C207: now left out of the parts list
- C208: footprint Capacitor_SMD:C_0603_1608Metric_Pad1.08x0.95mm_HandSolder -> Capacitor_SMD:C_1206_3216Metric; Manufacturer TDK -> KEMET; Part Number C1608X7R1H104K080AA -> C1206C104K5RAC7800; Vendor Link https://br.mouser.com/ProductDetail/TDK/C1608X7R1H104K080AA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 -> https://br.mouser.com/ProductDetail/KEMET/C1206C104K5RAC780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
Other:
- moved on the sheet: C212, C213, C214, R215, R216, R219, RV201, TP201, TP202, TP203, U204A, U204B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

Commit message: Update PCB layout
Parts:
- R216: Manufacturer Yageo -> (none); Vendor Link https://www.digikey.com/en/products/detail/yageo/RC1206FR-0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 -> (none)
Changed lines of the file:
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@@
       (effects (font (size 1.27 1.27)) hide)
     )
-    (property "Description" "Resistor 4k7 1% 0.25W SMD 1206" (id 5) (at 99.06 145.415 0)
+    (property "Description" "Resistor 4k7 1% 0.125W SMD 0805" (id 5) (at 99.06 145.415 0)
       (effects (font (size 1.27 1.27)) hide)
     )
-    (property "Manufacturer" "Yageo" (id 6) (at 99.06 145.415 0)
+    (property "Manufacturer" "" (id 6) (at 99.06 145.415 0)
       (effects (font (size 1.27 1.27)) hide)
     )
-    (property "Vendor Link" "https://www.digikey.com/en/products/detail/yageo/RC1206FR-074K7L/728887?s=N4IgTCBcDaIEoGECMYAMA2AYnAtKg7ACwDS%2BAMiALoC%2BQA" (id 7) (at 99.06 145.415 0)
+    (property "Vendor Link" "" (id 7) (at 99.06 145.415 0)
       (effects (font (size 1.27 1.27)) hide)
     )

Commit message: Finish routing
Connections:
- net at C212.1, R215.1, RV201.2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: no longer RV201.1
Changed lines of the file:
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@@
   (junction (at 140.335 74.93) (diameter 0) (color 0 0 0 0)
   )
-  (junction (at 41.91 155.575) (diameter 0) (color 0 0 0 0)
-  )
   (junction (at 171.45 85.09) (diameter 0) (color 0 0 0 0)
   )
@@
     (stroke (width 0) (type default) (color 0 0 0 0))
   )
-  (wire (pts (xy 41.91 155.575) (xy 41.91 156.845))
-    (stroke (width 0) (type default) (color 0 0 0 0))
-  )
   (wire (pts (xy 135.255 174.625) (xy 135.255 169.545))
     (stroke (width 0) (type default) (color 0 0 0 0))
@@
     (stroke (width 0) (type default) (color 0 0 0 0))
   )
-  (wire (pts (xy 41.91 155.575) (xy 41.91 151.765))
+  (wire (pts (xy 41.91 154.305) (xy 41.91 151.765))
     (stroke (width 0) (type default) (color 0 0 0 0))
   )
@@
     (stroke (width 0) (type default) (color 0 0 0 0))
   )
-  (wire (pts (xy 36.83 155.575) (xy 41.91 155.575))
+  (wire (pts (xy 36.83 154.305) (xy 41.91 154.305))
     (stroke (width 0) (type default) (color 0 0 0 0))
   )
@@
     (stroke (width 0) (type default) (color 0 0 0 0))
   )
-  (wire (pts (xy 36.83 155.575) (xy 36.83 160.655))
-    (stroke (width 0) (type default) (color 0 0 0 0))
-  )
+  (wire (pts (xy 36.83 154.305) (xy 36.83 160.655))
+    (stroke (width 0) (type default) (color 0 0 0 0))
+  )

Commit message: Assign test point values, arrange PCB fabrication layers
Parts:
- TP203: value TestPoint -> V-VAL
- TP204: value TestPoint -> Vdiff1+
- TP205: value TestPoint -> Vdiff1-
- TP206: value TestPoint -> Vdiff2+
- TP207: value TestPoint -> Vdiff2-
- TP208: value TestPoint -> Vsing
Changed lines of the file:
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@@
     (in_bom yes) (on_board yes)
     (property "Reference" "TP206" (id 0) (at 140.335 64.135 90))
-    (property "Value" "TestPoint" (id 1) (at 144.145 66.548 90)
+    (property "Value" "Vdiff2+" (id 1) (at 144.145 66.548 90)
       (effects (font (size 1.27 1.27)) hide)
     )
@@
     (in_bom yes) (on_board yes)
     (property "Reference" "TP204" (id 0) (at 113.03 62.865 90))
-    (property "Value" "TestPoint" (id 1) (at 116.84 66.548 90)
+    (property "Value" "Vdiff1+" (id 1) (at 116.84 66.548 90)
       (effects (font (size 1.27 1.27)) hide)
     )
@@
     (in_bom yes) (on_board yes)
     (property "Reference" "TP208" (id 0) (at 186.055 80.01 90))
-    (property "Value" "TestPoint" (id 1) (at 182.245 75.692 90)
+    (property "Value" "Vsing" (id 1) (at 182.245 75.692 90)
       (effects (font (size 1.27 1.27)) hide)
     )
@@
     (in_bom yes) (on_board yes)
     (property "Reference" "TP207" (id 0) (at 140.335 81.28 90))
-    (property "Value" "TestPoint" (id 1) (at 136.525 78.232 90)
+    (property "Value" "Vdiff2-" (id 1) (at 136.525 78.232 90)
       (effects (font (size 1.27 1.27)) hide)
     )
@@
     (in_bom yes) (on_board yes)
     (property "Reference" "TP205" (id 0) (at 113.03 82.55 90))
-    (property "Value" "TestPoint" (id 1) (at 109.22 78.232 90)
+    (property "Value" "Vdiff1-" (id 1) (at 109.22 78.232 90)
       (effects (font (size 1.27 1.27)) hide)
     )
@@
     (in_bom yes) (on_board yes)
     (property "Reference" "TP203" (id 0) (at 104.775 161.925 90))
-    (property "Value" "TestPoint" (id 1) (at 100.965 157.607 90)
-      (effects (font (size 1.27 1.27)) hide)
-    )
+    (property "Value" "V-VAL" (id 1) (at 100.965 157.607 90)
+      (effects (font (size 1.27 1.27)) hide)
+    )

Commit message: Increase value of resistor in series with relay coil (R707)
Parts:
- C208: footprint Capacitor_SMD:C_1206_3216Metric -> qds-cv-lib:C_1206_3216Metric_Small_Pad
Changed lines of the file:
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@@
       (effects (font (size 1.27 1.27)) (justify left))
     )
-    (property "Footprint" "Capacitor_SMD:C_1206_3216Metric" (id 2) (at 141.9352 116.84 0)
+    (property "Footprint" "qds-cv-lib:C_1206_3216Metric_Small_Pad" (id 2) (at 141.9352 116.84 0)
       (effects (font (size 1.27 1.27)) hide)
     )
