File: pcb/cad/analog-front-end.kicad_sch (KiCad schematic)
At the start: 45 parts

Commit message: replace 4k7 resistors part number
Parts:
- R?: footprint Resistor_SMD:R_1206_3216Metric_Pad1.30x1.75mm_HandSolder -> Resistor_SMD:R_0805_2012Metric_Pad1.20x1.40mm_HandSolder; Part Number RC1206FR-074K7L -> 0805W8F1200T5E
Changed lines of the file:
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@@
       (effects (font (size 1.27 1.27)) (justify right))
     )
-    (property "Footprint" "Resistor_SMD:R_1206_3216Metric_Pad1.30x1.75mm_HandSolder" (id 2) (at 108.204 133.604 90)
+    (property "Footprint" "Resistor_SMD:R_0805_2012Metric_Pad1.20x1.40mm_HandSolder" (id 2) (at 108.204 133.604 90)
       (effects (font (size 1.27 1.27)) hide)
     )
-    (property "Datasheet" "https://www.yageo.com/upload/media/product/productsearch/datasheet/rchip/PYu-RC_Group_51_RoHS_L_12.pdf" (id 3) (at 109.22 133.35 0)
+    (property "Datasheet" "https://datasheet.lcsc.com/lcsc/2206010216_UNI-ROYAL-Uniroyal-Elec-0805W8F1002T5E_C17414.pdf" (id 3) (at 109.22 133.35 0)
       (effects (font (size 1.27 1.27)) hide)
     )
-    (property "Part Number" "RC1206FR-074K7L" (id 4) (at 109.22 133.35 0)
+    (property "Part Number" "0805W8F1200T5E" (id 4) (at 109.22 133.35 0)
       (effects (font (size 1.27 1.27)) hide)
     )

Commit message: Fixed footprints 3D models orientation
Parts:
- RV?: footprint Potentiometer_SMD:Potentiometer_Bourns_3224X_Vertical -> qds-cv-lib:Potentiometer_Bourns_3224X_Vertical
Other:
- note added: "Detection window comparator"
- note added: "Differential-to-Single"
- note added: "Gain & Offset"
Changed lines of the file:
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@@
+    (effects (font (size 1.27 1.27)) (justify left bottom))
+  )
+  (text "Gain & Offset" (at 218.44 46.99 0)
     (effects (font (size 1.27 1.27)) (justify left bottom))
   )
@@
   )
   (text "   Input\novervoltage\nprotection:\n  ±425 V" (at 78.74 96.52 0)
+    (effects (font (size 1.27 1.27)) (justify left bottom))
+  )
+  (text "Differential-to-Single" (at 158.75 46.99 0)
     (effects (font (size 1.27 1.27)) (justify left bottom))
   )
@@
   )
   (text " BNC monitor\nOutput range:\n    ±10 V" (at 250.19 129.54 0)
+    (effects (font (size 1.27 1.27)) (justify left bottom))
+  )
+  (text "Detection window comparator" (at 62.23 127 0)
     (effects (font (size 1.27 1.27)) (justify left bottom))
   )
@@
       (effects (font (size 1.27 1.27)) (justify right))
     )
-    (property "Footprint" "Potentiometer_SMD:Potentiometer_Bourns_3224X_Vertical" (id 2) (at 45.72 149.86 0)
-      (effects (font (size 1.27 1.27)) hide)
-    )
+    (property "Footprint" "qds-cv-lib:Potentiometer_Bourns_3224X_Vertical" (id 2) (at 45.72 149.86 0)
+      (effects (font (size 1.27 1.27)) hide)
+    )

Commit message: Update power supplies, symbols and footprint libs
Parts:
- gave numbers to parts that had none: 41

Commit message: Grouped 74HC123 into two IC's and updated BNC connector 3D model
Parts:
- J201: footprint Connector_Coaxial:BNC_Amphenol_B6252HB-NPP3G-50_Horizontal -> qds-cv-lib:Molex_0731375003
Changed lines of the file:
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@@
       (effects (font (size 1.27 1.27)) (justify left) hide)
     )
-    (property "Footprint" "Connector_Coaxial:BNC_Amphenol_B6252HB-NPP3G-50_Horizontal" (id 2) (at 257.81 134.62 0)
+    (property "Footprint" "qds-cv-lib:Molex_0731375003" (id 2) (at 257.81 134.62 0)
       (effects (font (size 1.27 1.27)) hide)
     )

Commit message: Fix isolated supplies from analog-front-end, include no-connection flags, move itens in root sheet for better view, redefine pin types to fix ERC
Connections:
- net GND-ISO-A is gone; now on net GND-ISO: C207.2, C208.2, D201.1, D202.1, U202.4 (V1-)
- net GND-ISO: now reaches R207.2, R211.2, R212.1
- net +5V-ISO-A renamed +5V-ISO
Other:
- moved on the sheet: C207

Commit message: Several updates on schematic - close #5, close #6, close #7, close #8. - include test points - change relay supply to 15V and its series resistor to 180 ohm - replace AMC1200 VDD1 capacitor of 100nF by a 1206 model
Parts:
- added TP201, TP202, TP203: TestPoint, symbol Connector:TestPoint
- added TP204: Vth-H, symbol Connector:TestPoint
- added TP205: Vth-L, symbol Connector:TestPoint
- added TP206: V-VAL, symbol Connector:TestPoint
- added TP207: V-DET, symbol Connector:TestPoint
- C208: footprint Capacitor_SMD:C_0603_1608Metric_Pad1.08x0.95mm_HandSolder -> qds-cv-lib:C_1206_3216Metric_Small_Pad; CNPEM Code AP107349 -> (none); Manufacturer TDK -> KEMET; Part Number C1608X7R1H104K080AA -> C1206C104K5RAC7800; Vendor Link https://br.mouser.com/ProductDetail/TDK/C1608X7R1H104K080AA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 -> (none)
- R216: Manufacturer Yageo -> Royalohm; Vendor Link https://www.digikey.com/en/products/detail/yageo/RC1206FR-0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 -> (none)
Connections:
- net V-DET: now also TP207.1
- net V-VAL: now also TP206.1
- net at C213.1, R219.2, RV201.3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: now also TP205.1
- net at C212.1, R215.1, RV201.1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: now also TP204.1
Other:
- note added: "Input range: ±20 V Saturation: ±24 V"
- note added: "Treshold adjustment: V-DET: 0.5 to 4.5 V Voltage taps: ±200 mV"

Commit message: Include resistors tied to +5V and GND in isolated front-end circuits
Parts:
- removed TP201, TP202, TP203: TestPoint, symbol Connector:TestPoint
- added R220, R221: 2M, Resistor_SMD:R_0805_2012Metric_Pad1.20x1.40mm_HandSolder, symbol Device:R_Small_US
- added R222, R223: 1M, Resistor_SMD:R_0805_2012Metric_Pad1.20x1.40mm_HandSolder, symbol Device:R_Small_US
Connections:
- net +5V-ISO: now also R220.2
- net GND-ISO: now also R221.1, R222.2, R223.1; no longer R207.2, R211.2, R212.1
- net VOLTAGE-TAP-IN-N: now also R221.2
- net VOLTAGE-TAP-IN-P: now also R220.1
- net at R205.2, R206.1, R207.1: now also R222.1
- net at C212.1, R215.1, RV201.2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: no longer RV201.1
- new net: R207.2, R211.2, R212.1, R223.2
Other:
- note added: "safety resistors tied to +5V and GND will be confirmed"
- moved on the sheet: C205, C206, C207, C208, C209, C210, C211, C212, C213, C214, D202, J201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

Commit message: Improve window comparator, +5V-REF and relay driver circuits close #19 close #20 close #22
Parts:
- added D203: BAT165, Diode_SMD:D_SOD-323_HandSoldering, symbol Device:D
- added R224: 2.2k, Resistor_SMD:R_0805_2012Metric_Pad1.20x1.40mm_HandSolder, symbol Device:R_US
Connections:
- net Earth: now also D203.2 (A)
- net V-DET: now also R224.1; no longer U204.2 (-), U204.5 (+)
- new net: D203.1 (K), R224.2, U204.2 (-), U204.5 (+)
Other:
- moved on the sheet: C212, C213, C214, R215, R216, R219, RV201, TP204, TP205, TP206, U204A, U204B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
