File: pcb/cad/quench-trigger.kicad_sch (KiCad schematic)
At the start: 0 parts

Commit message: Power supplies schematic created
Other:
- company: (none) -> CNPEM - Brazilian Center for Research in Energy and Materials
Changed lines of the file:
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@@
 (kicad_sch (version 20211123) (generator eeschema)
   (paper "A4")
+  (title_block
+    (rev "v1.0.0")
+    (company "CNPEM - Brazilian Center for Research in Energy and Materials")
+    (comment 1 "Group: ENT/AIS")
+    (comment 2 "Authors: Gabriel Brunheira / Samuel Fraga")
+  )
   (text "Triggers aggregation, indication and actuation" (at 69.85 27.94 0)
     (effects (font (size 5 5) (thickness 1) bold) (justify left bottom))

Commit message: create schematic for trigger aggregation, indication and actuation circuits
Parts:
- added C? (x4): 100n, Capacitor_SMD:C_0603_1608Metric_Pad1.08x0.95mm_HandSolder, symbol Device:C
- added D?: D, symbol Device:D
- added J?: DB9_Female, Connector_Dsub:DSUB-9_Female_Horizontal_P2.77x2.84mm_EdgePinOffset7.70mm_Housed_MountingHolesOffset9.12mm, symbol Connector:DB9_Female_MountingHoles
- added J?: Conn_Coaxial, symbol Connector:Conn_Coaxial
- added K?: FINDER-30.22, Relay_THT:Relay_DPDT_Finder_30.22, symbol qds-cv-lib-sym:FINDER-30.22
- added LD? (x5): Red, qds-cv-lib:LED_WP934CB_ID, symbol Device:LED
- added Q?: BC846b, Package_TO_SOT_SMD:SOT-23, symbol Transistor_BJT:BC846
- added R?: 50, symbol Device:R_US
- added R? (x5): 270, symbol Device:R_US
- added R?: 75, symbol Device:R_US
- added R?: 120, symbol Device:R_US
- added R? (x2): 5k, symbol Device:R_US
- added R?: 2.3k, symbol Device:R_US
- added R?: 50k, symbol Device:R_US
- added SW?: TRIG, Button_Switch_THT:SW_Tactile_SPST_Angled_PTS645Vx39-2LFS, symbol Switch:SW_Push
- added SW?: RST, symbol Switch:SW_Push
- added U? (x6): 74LVC2G17, Package_TO_SOT_SMD:SOT-23-6_Handsoldering, symbol qds-cv-lib-sym:74LVC2G17
- added U? (x5): 74HCS08, Package_SO:SO-14_3.9x8.65mm_P1.27mm, symbol qds-cv-lib-sym:74HCS08
- added U? (x5): 74LV132, Package_SO:SO-14_3.9x8.65mm_P1.27mm, symbol qds-cv-lib-sym:74LV132
- added U?: 74HC574, Package_SO:TSSOP-20_4.4x6.5mm_P0.65mm, symbol qds-cv-lib-sym:74HC574
- added U?: HFBR-1521Z, qds-cv-lib:HFBR-1521Z, symbol qds-cv-lib-sym:HFBR-1521Z
Connections:
- net TRIG-CH-A: now also U?.1, U?.3 (D1)
- net TRIG-CH-B: now also U?.2, U?.4 (D2)
- net TRIG-CH-C: now also U?.4, U?.5 (D3)
- net TRIG-CH-D: now also U?.5, U?.6 (D4)
- new net: U?.1, U?.1, U?.19 (Q0), U?.3, U?.5
- new net: R?.1, U?.4
- new net: R?.1, U?.6 (x2)
- new net: J?.1 (In), R?.2
- new net: LD?.2 (A), R?.2 (x5)
- new net: U?.1, U?.11, U?.2, U?.2 (D0)
- new net: U?.3, U?.4
- new net: D?.1 (K), K?.A1, R?.2
- new net: D?.2 (A), K?.A2, Q?.3 (C)
- new net: U?.11 (Cp), U?.8
- new net: LD?.1 (K), U?.14 (Q5)
- new net: LD?.1 (K), U?.15 (Q4)
- new net: LD?.1 (K), U?.16 (Q3)
- new net: LD?.1 (K), U?.17 (Q2)
- new net: LD?.1 (K), U?.18 (Q1)
- new net: R?.2, U?.1 (Anode)
- new net: U?.10, U?.6
- new net: U?.12, U?.8
- new net: U?.3, U?.9
- new net: U?.6, U?.9
- new net: Q?.1 (B), R?.2
- new net +14V: R?.1
- new net +5V: C?.1, C?.1, C?.1, C?.1, R?.1, R?.1, R?.1, R?.1, R?.1, R?.1, R?.1, U?.14 (VCC), U?.14 (VCC), U?.2 (GND), U?.20 (VCC), U?.5 (VCC)
- new net Earth: C?.2, C?.2, C?.2, C?.2, J?.0 (PAD), J?.2 (Ext), J?.6, Q?.2 (E), R?.2, SW?.1, SW?.1, U?.1 (OE), U?.10 (GND), U?.12, U?.13, U?.2 (Cathode), U?.2 (GND), U?.3, U?.3 (NC), U?.4 (NC), U?.5 (VCC), U?.7 (GND), U?.7 (GND), U?.8 (D6), U?.9 (D7)
- new net ILCOK_21: K?.21
- new net ILOCK_11: J?.3, K?.11
- new net ILOCK_12: J?.8, K?.14
- new net ILOCK_21: J?.4
- new net ILOCK_22: J?.9, K?.24
- new net REMOTE_RST+: J?.1, R?.2, SW?.2, U?.10
- new net SW_TRIG+: J?.2, R?.2
- new net SW_TRIG-: J?.7, R?.1, SW?.2, U?.13, U?.7 (D5)

Commit message: Created hierarchy connections, updates on analog-front-end and included 5V reference circuit
Changed lines of the file:
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@@
     (stroke (width 0) (type default) (color 0 0 0 0))
   )
-  (text "Triggers aggregation, indication and actuation" (at 69.85 27.94 0)
+  (text "Triggers aggregation, indication and actuation" (at 59.69 26.67 0)
     (effects (font (size 5 5) (thickness 1) bold) (justify left bottom))
   )

Commit message: update components specification
Parts:
- D?: value D -> B220A; footprint (none) -> Diode_SMD:D_SMA_Handsoldering; Part Number (none) -> 621-B220A-F
- J?: footprint (none) -> Connector_Coaxial:BNC_Amphenol_B6252HB-NPP3G-50_Horizontal; Manufacturer (none) -> Molex; Part Number (none) -> 0731375003
- R? (x5): footprint (none) -> Resistor_SMD:R_0805_2012Metric_Pad1.20x1.40mm_HandSolder; CNPEM Code (none) -> MT104052; Manufacturer (none) -> Yageo; Part Number (none) -> RC0805FR-07270RL; Vendor Link (none) -> https://www.digikey.com/en/products/detail/yageo/RC0805FR-0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
- R?: value 75 -> 82; footprint (none) -> Resistor_SMD:R_0805_2012Metric_Pad1.20x1.40mm_HandSolder; Part Number (none) -> RK73H2ATTD82R0F
- R?: footprint (none) -> Resistor_SMD:R_0805_2012Metric_Pad1.20x1.40mm_HandSolder; Part Number (none) -> RC0805FR-07120RL
- R? (x2): value 5k -> 4.7k; footprint (none) -> Resistor_SMD:R_1206_3216Metric_Pad1.30x1.75mm_HandSolder; Part Number (none) -> RC1206FR-074K7L
- R?: value 2.3k -> 2.2k; footprint (none) -> Resistor_SMD:R_0805_2012Metric_Pad1.20x1.40mm_HandSolder; Part Number (none) -> RC0805FR-072K2L
- R?: value 50k -> 47k; footprint (none) -> Resistor_SMD:R_0603_1608Metric_Pad0.98x0.95mm_HandSolder; CNPEM Code (none) -> AP107380; Part Number (none) -> ERA-3AEB473V
- SW?: footprint (none) -> Button_Switch_THT:SW_Tactile_SPST_Angled_PTS645Vx39-2LFS

Commit message: Update componentes fields and reference circuit
Parts:
- D?: Manufacturer (none) -> Diodes Inc.; Vendor Link (none) -> https://br.mouser.com/ProductDetail/Diodes-Incorporated/B22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
- J?: Manufacturer (none) -> Amphenol FCI
- J?: CNPEM Code (none) -> AP107369; Vendor Link (none) -> https://www.digikey.com/en/products/detail/molex/0731375003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
- K?: CNPEM Code (none) -> AO102294; Manufacturer (none) -> Finder; Vendor Link (none) -> https://pt.farnell.com/finder/30-22-7-012-0010/relay-signal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
- LD? (x5): Vendor Link (none) -> https://www.digikey.com/en/products/detail/kingbright/WP934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
- Q?: value BC846b -> BC846B; CNPEM Code (none) -> AP105095
- R?: value 50 -> 49.9; footprint (none) -> Resistor_SMD:R_0805_2012Metric_Pad1.20x1.40mm_HandSolder; CNPEM Code (none) -> AP108391; Manufacturer (none) -> Yageo; Part Number (none) -> RT0805DRE0749R9L; Vendor Link (none) -> https://www.digikey.com/en/products/detail/yageo/RT0805DRE0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
- R? (x5): CNPEM Code MT104052 -> (none); Manufacturer Yageo -> Fenghua Advance Technology; Part Number RC0805FR-07270RL -> RC-05K203JT; Vendor Link https://www.digikey.com/en/products/detail/yageo/RC0805FR-0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 -> (none)
- R?: CNPEM Code (none) -> MT100270; Manufacturer (none) -> Panasonic Electronic Components; Part Number RC0805FR-07120RL -> ERJ-6ENF1200V; Vendor Link (none) -> https://www.digikey.com/en/products/detail/panasonic-electr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
- R? (x2): Manufacturer (none) -> Yageo; Vendor Link (none) -> https://www.digikey.com/en/products/detail/yageo/RC1206FR-0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
- R?: CNPEM Code (none) -> MT104237; Manufacturer (none) -> Yageo; Vendor Link (none) -> https://www.digikey.com/en/products/detail/yageo/RC0805FR-0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
- R?: Manufacturer (none) -> Panasonic Electronic Components; Vendor Link (none) -> https://www.digikey.com/en/products/detail/ERA-3AEB473V/P47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
Other:
- title: (none) -> Triggers Aggregation, Indication and Actuation

Commit message: replace 4k7 resistors part number
Parts:
- R? (x2): footprint Resistor_SMD:R_1206_3216Metric_Pad1.30x1.75mm_HandSolder -> Resistor_SMD:R_0805_2012Metric_Pad1.20x1.40mm_HandSolder; Part Number RC1206FR-074K7L -> 0805W8F1200T5E
Changed lines of the file:
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@@
       (effects (font (size 1.27 1.27)) (justify left))
     )
-    (property "Footprint" "Resistor_SMD:R_1206_3216Metric_Pad1.30x1.75mm_HandSolder" (id 2) (at 69.596 108.839 90)
-      (effects (font (size 1.27 1.27)) hide)
-    )
-    (property "Datasheet" "https://www.yageo.com/upload/media/product/productsearch/datasheet/rchip/PYu-RC_Group_51_RoHS_L_12.pdf" (id 3) (at 68.58 108.585 0)
-      (effects (font (size 1.27 1.27)) hide)
-    )
-    (property "Part Number" "RC1206FR-074K7L" (id 4) (at 68.58 108.585 0)
+    (property "Footprint" "Resistor_SMD:R_0805_2012Metric_Pad1.20x1.40mm_HandSolder" (id 2) (at 69.596 108.839 90)
+      (effects (font (size 1.27 1.27)) hide)
+    )
+    (property "Datasheet" "https://datasheet.lcsc.com/lcsc/2206010216_UNI-ROYAL-Uniroyal-Elec-0805W8F1002T5E_C17414.pdf" (id 3) (at 68.58 108.585 0)
+      (effects (font (size 1.27 1.27)) hide)
+    )
+    (property "Part Number" "0805W8F1200T5E" (id 4) (at 68.58 108.585 0)
       (effects (font (size 1.27 1.27)) hide)
     )
@@
       (effects (font (size 1.27 1.27)) (justify left))
     )
-    (property "Footprint" "Resistor_SMD:R_1206_3216Metric_Pad1.30x1.75mm_HandSolder" (id 2) (at 44.831 108.839 90)
-      (effects (font (size 1.27 1.27)) hide)
-    )
-    (property "Datasheet" "https://www.yageo.com/upload/media/product/productsearch/datasheet/rchip/PYu-RC_Group_51_RoHS_L_12.pdf" (id 3) (at 43.815 108.585 0)
-      (effects (font (size 1.27 1.27)) hide)
-    )
-    (property "Part Number" "RC1206FR-074K7L" (id 4) (at 43.815 108.585 0)
-      (effects (font (size 1.27 1.27)) hide)
-    )
+    (property "Footprint" "Resistor_SMD:R_0805_2012Metric_Pad1.20x1.40mm_HandSolder" (id 2) (at 44.831 108.839 90)
+      (effects (font (size 1.27 1.27)) hide)
+    )
+    (property "Datasheet" "https://datasheet.lcsc.com/lcsc/2206010216_UNI-ROYAL-Uniroyal-Elec-0805W8F1002T5E_C17414.pdf" (id 3) (at 43.815 108.585 0)
+      (effects (font (size 1.27 1.27)) hide)
+    )
+    (property "Part Number" "0805W8F1200T5E" (id 4) (at 43.815 108.585 0)
+      (effects (font (size 1.27 1.27)) hide)
+    )

Commit message: Fixed footprints 3D models orientation
Other:
- moved on the sheet: LD?, R?

Commit message: Update power supplies, symbols and footprint libs
Parts:
- U705: renamed from U?; Manufacturer (none) -> Texas Instruments
- gave numbers to parts that had none: 33
Connections:
- net ILCOK_21 is gone; now on net ILOCK_21: K701.21
