File: pcb/cad/quench-trigger.kicad_sch (KiCad schematic)
At the start: 34 parts, among them J701 Conn_Coaxial, J702 DB9_Female, K701 FINDER-30.22, Q701 BC846B, SW701 RST, SW702 TRIG, U701 74HCS08, U702 74HC574, U703 74LV132, U704 74LVC2G17, U705 74LVC2G17, U706 HFBR-1521Z

Commit message: Grouped 74HC123 into two IC's and updated BNC connector 3D model
Parts:
- J701: footprint Connector_Coaxial:BNC_Amphenol_B6252HB-NPP3G-50_Horizontal -> qds-cv-lib:Molex_0731375003
Changed lines of the file:
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@@
       (effects (font (size 1.27 1.27)) (justify left) hide)
     )
-    (property "Footprint" "Connector_Coaxial:BNC_Amphenol_B6252HB-NPP3G-50_Horizontal" (id 2) (at 256.54 78.74 0)
+    (property "Footprint" "qds-cv-lib:Molex_0731375003" (id 2) (at 256.54 78.74 0)
       (effects (font (size 1.27 1.27)) hide)
     )

Commit message: Replace schematic symbols and text fields for a better view
Other:
- moved on the sheet: R701, R702, R703, R704, R705

Commit message: Place components of validation and quench trigger circuits on PCB
Parts:
- added C705: 100n, Capacitor_SMD:C_0603_1608Metric_Pad1.08x0.95mm_HandSolder, symbol Device:C
- U702: footprint Package_SO:TSSOP-20_4.4x6.5mm_P0.65mm -> Package_SO:SO-20_12.8x7.5mm_P1.27mm
Connections:
- net +5V: now also U705.5 (VCC), C705.2; no longer U705.2 (GND)
- net Earth: now also U703.4, U703.5, U705.1, U705.2 (GND), C705.1; no longer U703.12, U703.13, U705.3, U705.5 (VCC)
- net REMOTE_RST+: now also U703.9; no longer U703.10
- net SW_TRIG-: now also U701.9, U702.6 (D4); no longer U701.13, U702.7 (D5)
- net TRIG-CH-A: now also U702.2 (D0); no longer U702.3 (D1)
- net TRIG-CH-B: now also U702.3 (D1); no longer U702.4 (D2)
- net TRIG-CH-C: now also U702.4 (D2); no longer U702.5 (D3)
- net TRIG-CH-D: now also U702.5 (D3); no longer U702.6 (D4)
- net at U705.4: now also R710.1
- net at U703.1, U703.2: now also U701.8, U702.7 (D5); no longer U701.11, U702.2 (D0)
- net at U703.3: now also U703.12; no longer U703.4
- net at U702.14 (Q5): now also U703.13, U704.1, U704.3, U705.3; no longer LD705.1 (K)
- net at U702.15 (Q4): now also LD705.1 (K); no longer LD704.1 (K)
- net at U702.16 (Q3): now also LD704.1 (K); no longer LD703.1 (K)
- net at U702.17 (Q2): now also LD703.1 (K); no longer LD702.1 (K)
- net at U702.18 (Q1): now also LD702.1 (K); no longer LD701.1 (K)
- net at U701.10: now also U701.11; no longer U701.6
- net at U701.12: now also U701.6; no longer U701.8
- net at U701.3: now also U701.13; no longer U701.9
- net at U703.11: now also U703.10
- net at U703.6: no longer U703.9
- net at U705.6: no longer R710.1
- new net: LD701.1 (K), U702.19 (Q0)
Other:
- moved on the sheet: LD701, LD702, LD703, LD704, LD705, R701, R702, R703, R704, R705, U701C, U701D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

Commit message: Include ISO-A power circuit, all connectors and test points on PCB
Parts:
- added TP701, TP702: TestPoint, qds-cv-lib:TestPoint_Keystone_5010-5014_Multipurpose, symbol Connector:TestPoint
Connections:
- net at U702.14 (Q5), U703.13, U704.1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: now also TP702.1
- net at U702.11 (Cp), U703.8: now also TP701.1
Changed lines of the file:
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@@
   (junction (at 110.49 69.85) (diameter 0) (color 0 0 0 0)
   )
+  (junction (at 204.47 64.77) (diameter 0) (color 0 0 0 0)
+  )
   (junction (at 251.46 34.925) (diameter 0) (color 0 0 0 0)
   )
@@
   (junction (at 231.14 101.6) (diameter 0) (color 0 0 0 0)
   )
-  (junction (at 171.45 64.77) (diameter 0) (color 0 0 0 0)
-  )
   (junction (at 43.815 116.205) (diameter 0) (color 0 0 0 0)
   )
@@
   (junction (at 68.58 132.715) (diameter 0) (color 0 0 0 0)
   )
+  (junction (at 163.83 74.93) (diameter 0) (color 0 0 0 0)
+  )
   (wire (pts (xy 228.6 34.925) (xy 236.22 34.925))
     (stroke (width 0) (type default) (color 0 0 0 0))
@@
     (stroke (width 0) (type default) (color 0 0 0 0))
   )
+  (wire (pts (xy 163.83 74.93) (xy 173.99 74.93))
+    (stroke (width 0) (type default) (color 0 0 0 0))
+  )
   (wire (pts (xy 233.68 78.74) (xy 241.3 78.74))
     (stroke (width 0) (type default) (color 0 0 0 0))
@@
     (stroke (width 0) (type default) (color 0 0 0 0))
   )
-  (wire (pts (xy 171.45 64.77) (xy 173.99 64.77))
-    (stroke (width 0) (type default) (color 0 0 0 0))
-  )
   (wire (pts (xy 95.25 69.85) (xy 110.49 69.85))
     (stroke (width 0) (type default) (color 0 0 0 0))
@@
     (stroke (width 0) (type default) (color 0 0 0 0))
   )
-  (wire (pts (xy 161.29 66.04) (xy 171.45 66.04))
-    (stroke (width 0) (type default) (color 0 0 0 0))
-  )
   (wire (pts (xy 121.92 158.75) (xy 134.62 158.75))
     (stroke (width 0) (type default) (color 0 0 0 0))
@@
     (stroke (width 0) (type default) (color 0 0 0 0))
   )
-  (wire (pts (xy 156.21 74.93) (xy 173.99 74.93))
+  (wire (pts (xy 156.21 74.93) (xy 163.83 74.93))
     (stroke (width 0) (type default) (color 0 0 0 0))
   )
@@
     (stroke (width 0) (type default) (color 0 0 0 0))
   )
-  (wire (pts (xy 171.45 64.77) (xy 171.45 66.04))
-    (stroke (width 0) (type default) (color 0 0 0 0))
-  )
   (wire (pts (xy 127 85.09) (xy 140.97 85.09))
     (stroke (width 0) (type default) (color 0 0 0 0))
@@
     (stroke (width 0) (type default) (color 0 0 0 0))
   )
-  (wire (pts (xy 171.45 64.77) (xy 153.67 64.77))
+  (wire (pts (xy 153.67 64.77) (xy 173.99 64.77))
     (stroke (width 0) (type default) (color 0 0 0 0))
   )
@@
     (pin "1")
   )
+  (symbol (lib_id "Connector:TestPoint") (at 163.83 74.93 180) (unit 1)
+    (in_bom yes) (on_board yes)
+    (property "Reference" "TP701" (id 0) (at 163.83 82.55 90))
+    (property "Value" "TestPoint" (id 1) (at 160.02 78.232 90)
+      (effects (font (size 1.27 1.27)) hide)
+    )
+    (property "Footprint" "qds-cv-lib:TestPoint_Keystone_5010-5014_Multipurpose" (id 2) (at 158.75 74.93 0)
+      (effects (font (size 1.27 1.27)) hide)
+    )
+    (property "Datasheet" "https://www.keyelco.com/product-pdf.cfm?p=1321" (id 3) (at 158.75 74.93 0)
+      (effects (font (size 1.27 1.27)) hide)
+    )
+    (pin "1")
+  )
   (symbol (lib_name "74LV132_4") (lib_id "qds-cv-lib-sym:74LV132") (at 148.59 74.93 0) (mirror x) (unit 3)
     (in_bom yes) (on_board yes) (fields_autoplaced)
@@
       (effects (font (size 1.27 1.27)) hide)
     )
+    (pin "1")
+  )
+  (symbol (lib_id "Connector:TestPoint") (at 204.47 64.77 270) (unit 1)
+    (in_bom yes) (on_board yes)
+    (property "Reference" "TP702" (id 0) (at 212.09 64.77 90))
+    (property "Value" "TestPoint" (id 1) (at 207.772 68.58 90)
+      (effects (font (size 1.27 1.27)) hide)
+    )
+    (property "Footprint" "qds-cv-lib:TestPoint_Keystone_5010-5014_Multipurpose" (id 2) (at 204.47 69.85 0)
+      (effects (font (size 1.27 1.27)) hide)
+    )
+    (property "Datasheet" "https://www.keyelco.com/product-pdf.cfm?p=1321" (id 3) (at 204.47 69.85 0)
+      (effects (font (size 1.27 1.27)) hide)
+    )

Commit message: Remake some logic connections and update PCB
Connections:
- net Earth: now also U703.12, U703.13; no longer U703.4, U703.5
- net REMOTE_RST+: now also U703.10; no longer U703.9
- net at TP702.1, U702.14 (Q5), U704.1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: now also U703.5; no longer U703.13
- net at U703.3: now also U703.4; no longer U703.12
- net at U703.11: no longer U703.10
- net at U703.6: now also U703.9
Other:
- moved on the sheet: U703B, U703D
Changed lines of the file:
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@@
   (junction (at 236.22 34.925) (diameter 0) (color 0 0 0 0)
   )
-  (junction (at 87.63 187.96) (diameter 0) (color 0 0 0 0)
-  )
   (junction (at 146.05 158.75) (diameter 0) (color 0 0 0 0)
   )
@@
   (junction (at 231.14 101.6) (diameter 0) (color 0 0 0 0)
   )
+  (junction (at 97.79 88.9) (diameter 0) (color 0 0 0 0)
+  )
   (junction (at 43.815 116.205) (diameter 0) (color 0 0 0 0)
   )
@@
     (stroke (width 0) (type default) (color 0 0 0 0))
   )
-  (wire (pts (xy 87.63 182.88) (xy 87.63 187.96))
+  (wire (pts (xy 97.79 83.82) (xy 97.79 88.9))
     (stroke (width 0) (type default) (color 0 0 0 0))
   )
@@
     (pin "2")
   )
-  (symbol (lib_id "power:Earth") (at 87.63 187.96 0) (unit 1)
-    (in_bom yes) (on_board yes) (fields_autoplaced)
-    (property "Reference" "#PWR0717" (id 0) (at 87.63 194.31 0)
-      (effects (font (size 1.27 1.27)) hide)
-    )
-    (property "Value" "Earth" (id 1) (at 87.63 191.77 0)
-      (effects (font (size 1.27 1.27)) hide)
-    )
-    (property "Footprint" "" (id 2) (at 87.63 187.96 0)
-      (effects (font (size 1.27 1.27)) hide)
-    )
-    (property "Datasheet" "~" (id 3) (at 87.63 187.96 0)
+  (symbol (lib_id "power:Earth") (at 97.79 88.9 0) (unit 1)
+    (in_bom yes) (on_board yes) (fields_autoplaced)
+    (property "Reference" "#PWR0717" (id 0) (at 97.79 95.25 0)
+      (effects (font (size 1.27 1.27)) hide)
+    )
+    (property "Value" "Earth" (id 1) (at 97.79 92.71 0)
+      (effects (font (size 1.27 1.27)) hide)
+    )
+    (property "Footprint" "" (id 2) (at 97.79 88.9 0)
+      (effects (font (size 1.27 1.27)) hide)
+    )
+    (property "Datasheet" "~" (id 3) (at 97.79 88.9 0)
       (effects (font (size 1.27 1.27)) hide)
     )
@@
     (pin "7")
   )
-  (symbol (lib_name "74LV132_2") (lib_id "qds-cv-lib-sym:74LV132") (at 133.35 72.39 0) (unit 4)
-    (in_bom yes) (on_board yes) (fields_autoplaced)
-    (property "Reference" "U703" (id 0) (at 133.35 63.5 0))
-    (property "Value" "74LV132" (id 1) (at 133.35 66.04 0))
-    (property "Footprint" "Package_SO:SO-14_3.9x8.65mm_P1.27mm" (id 2) (at 133.35 72.39 0)
-      (effects (font (size 1.27 1.27)) hide)
-    )
-    (property "Datasheet" "http://www.ti.com/lit/ds/symlink/sn74lv132a.pdf" (id 3) (at 133.35 72.39 0)
-      (effects (font (size 1.27 1.27)) hide)
-    )
-    (property "Part Number" "SN74LV132ADR" (id 4) (at 133.35 72.39 0)
+  (symbol (lib_name "74LV132_2") (lib_id "qds-cv-lib-sym:74LV132") (at 105.41 86.36 0) (unit 4)
+    (in_bom yes) (on_board yes) (fields_autoplaced)
+    (property "Reference" "U703" (id 0) (at 105.41 77.47 0))
+    (property "Value" "74LV132" (id 1) (at 105.41 80.01 0))
+    (property "Footprint" "Package_SO:SO-14_3.9x8.65mm_P1.27mm" (id 2) (at 105.41 86.36 0)
+      (effects (font (size 1.27 1.27)) hide)
+    )
+    (property "Datasheet" "http://www.ti.com/lit/ds/symlink/sn74lv132a.pdf" (id 3) (at 105.41 86.36 0)
+      (effects (font (size 1.27 1.27)) hide)
+    )
+    (property "Part Number" "SN74LV132ADR" (id 4) (at 105.41 86.36 0)
       (effects (font (size 1.27 1.27)) hide)
     )
@@
     (pin "1")
   )
-  (symbol (lib_name "74LV132_4") (lib_id "qds-cv-lib-sym:74LV132") (at 148.59 74.93 0) (mirror x) (unit 3)
+  (symbol (lib_name "74LV132_4") (lib_id "qds-cv-lib-sym:74LV132") (at 148.59 74.93 0) (unit 3)
     (in_bom yes) (on_board yes) (fields_autoplaced)
     (property "Reference" "U703" (id 0) (at 148.59 66.04 0))
@@
     (pin "3")
   )
-  (symbol (lib_id "qds-cv-lib-sym:74LV132") (at 95.25 185.42 0) (unit 2)
-    (in_bom yes) (on_board yes) (fields_autoplaced)
-    (property "Reference" "U703" (id 0) (at 95.25 176.53 0))
-    (property "Value" "74LV132" (id 1) (at 95.25 179.07 0))
-    (property "Footprint" "Package_SO:SO-14_3.9x8.65mm_P1.27mm" (id 2) (at 95.25 185.42 0)
-      (effects (font (size 1.27 1.27)) hide)
-    )
-    (property "Datasheet" "http://www.ti.com/lit/ds/symlink/sn74lv132a.pdf" (id 3) (at 95.25 185.42 0)
-      (effects (font (size 1.27 1.27)) hide)
-    )
-    (property "Part Number" "SN74LV132ADR" (id 4) (at 95.25 185.42 0)
-      (effects (font (size 1.27 1.27)) hide)
-    )
+  (symbol (lib_id "qds-cv-lib-sym:74LV132") (at 133.35 72.39 0) (unit 2)
+    (in_bom yes) (on_board yes) (fields_autoplaced)
+    (property "Reference" "U703" (id 0) (at 133.35 63.5 0))
+    (property "Value" "74LV132" (id 1) (at 133.35 66.04 0))
+    (property "Footprint" "Package_SO:SO-14_3.9x8.65mm_P1.27mm" (id 2) (at 133.35 72.39 0)
+      (effects (font (size 1.27 1.27)) hide)
+    )
+    (property "Datasheet" "http://www.ti.com/lit/ds/symlink/sn74lv132a.pdf" (id 3) (at 133.35 72.39 0)
+      (effects (font (size 1.27 1.27)) hide)
+    )
+    (property "Part Number" "SN74LV132ADR" (id 4) (at 133.35 72.39 0)
+      (effects (font (size 1.27 1.27)) hide)
+    )

Commit message: Update PCB layout
Parts:
- R708, R709: Manufacturer Yageo -> (none); Vendor Link https://www.digikey.com/en/products/detail/yageo/RC1206FR-0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 -> (none)
Connections:
- net +5V: now also LD701.2 (A), LD702.2 (A), LD703.2 (A), LD704.2 (A), LD705.2 (A); no longer R701.1, R702.1, R703.1, R704.1, R705.1
- net ILOCK_11: now also J702.5; no longer J702.3
- net ILOCK_12: now also J702.9; no longer J702.8
- net ILOCK_22: now also J702.8; no longer J702.9
- net REMOTE_RST+: now also J702.7; no longer J702.1
- net SW_TRIG+: now also J702.1; no longer J702.2
- net SW_TRIG-: now also J702.2; no longer J702.7
- net at R701.2: now also U702.19 (Q0); no longer LD701.2 (A)
- net at U702.15 (Q4): now also R705.2; no longer LD705.1 (K)
- net at U702.16 (Q3): now also R704.2; no longer LD704.1 (K)
- net at U702.17 (Q2): now also R703.2; no longer LD703.1 (K)
- net at U702.18 (Q1): now also R702.2; no longer LD702.1 (K)
- net at LD701.1 (K): now also R701.1; no longer U702.19 (Q0)
- new net: LD703.1 (K), R703.1
- new net: LD702.1 (K), R702.1
- new net: LD704.1 (K), R704.1
- new net: LD705.1 (K), R705.1
Other:
- moved on the sheet: LD701, LD702, LD703, LD704, LD705, R701, R702, R703, R704, R705

Commit message: Finish routing
Connections:
- net at U704.4: now also R710.1; no longer R712.1
- net at U705.4: now also R706.1; no longer R710.1
- net at U704.6: now also R712.1; no longer R706.1
Other:
- moved on the sheet: U704A, U704B, U705B
Changed lines of the file:
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@@
     (pin "5")
   )
-  (symbol (lib_id "qds-cv-lib-sym:74LVC2G17") (at 207.01 151.13 0) (unit 2)
-    (in_bom yes) (on_board yes)
-    (property "Reference" "U704" (id 0) (at 207.01 143.51 0))
-    (property "Value" "74LVC2G17" (id 1) (at 207.01 146.05 0))
-    (property "Footprint" "Package_TO_SOT_SMD:SOT-23-6_Handsoldering" (id 2) (at 207.01 138.43 0)
-      (effects (font (size 1.27 1.27)) hide)
-    )
-    (property "Datasheet" "https://www.ti.com/lit/ds/symlink/sn74lvc2g17.pdf" (id 3) (at 207.01 135.89 0)
-      (effects (font (size 1.27 1.27)) hide)
-    )
-    (property "Part Number" "SN74LVC2G17DBVR" (id 4) (at 207.01 151.13 0)
-      (effects (font (size 1.27 1.27)) hide)
-    )
-    (pin "1")
-    (pin "6")
-    (pin "3")
-    (pin "4")
-    (pin "2")
-    (pin "5")
-  )
-  (symbol (lib_name "74LVC2G17_4") (lib_id "qds-cv-lib-sym:74LVC2G17") (at 208.28 125.73 0) (unit 2)
-    (in_bom yes) (on_board yes) (fields_autoplaced)
-    (property "Reference" "U705" (id 0) (at 208.915 118.11 0))
-    (property "Value" "74LVC2G17" (id 1) (at 208.915 120.65 0))
+  (symbol (lib_id "qds-cv-lib-sym:74LVC2G17") (at 208.28 125.73 0) (unit 2)
+    (in_bom yes) (on_board yes)
+    (property "Reference" "U704" (id 0) (at 208.28 118.11 0))
+    (property "Value" "74LVC2G17" (id 1) (at 208.28 120.65 0))
     (property "Footprint" "Package_TO_SOT_SMD:SOT-23-6_Handsoldering" (id 2) (at 208.28 113.03 0)
       (effects (font (size 1.27 1.27)) hide)
@@
       (effects (font (size 1.27 1.27)) hide)
     )
-    (property "Manufacturer" "Texas Instruments" (id 5) (at 208.28 125.73 0)
+    (pin "1")
+    (pin "6")
+    (pin "3")
+    (pin "4")
+    (pin "2")
+    (pin "5")
+  )
+  (symbol (lib_name "74LVC2G17_4") (lib_id "qds-cv-lib-sym:74LVC2G17") (at 226.06 78.74 0) (unit 2)
+    (in_bom yes) (on_board yes) (fields_autoplaced)
+    (property "Reference" "U705" (id 0) (at 226.695 71.12 0))
+    (property "Value" "74LVC2G17" (id 1) (at 226.695 73.66 0))
+    (property "Footprint" "Package_TO_SOT_SMD:SOT-23-6_Handsoldering" (id 2) (at 226.06 66.04 0)
+      (effects (font (size 1.27 1.27)) hide)
+    )
+    (property "Datasheet" "https://www.ti.com/lit/ds/symlink/sn74lvc2g17.pdf" (id 3) (at 226.06 63.5 0)
+      (effects (font (size 1.27 1.27)) hide)
+    )
+    (property "Part Number" "SN74LVC2G17DBVR" (id 4) (at 226.06 78.74 0)
+      (effects (font (size 1.27 1.27)) hide)
+    )
+    (property "Manufacturer" "Texas Instruments" (id 5) (at 226.06 78.74 0)
       (effects (font (size 1.27 1.27)) hide)
     )
@@
     (pin "2")
   )
-  (symbol (lib_name "74LVC2G17_3") (lib_id "qds-cv-lib-sym:74LVC2G17") (at 226.06 78.74 0) (unit 1)
-    (in_bom yes) (on_board yes) (fields_autoplaced)
-    (property "Reference" "U704" (id 0) (at 226.695 71.12 0))
-    (property "Value" "74LVC2G17" (id 1) (at 226.695 73.66 0))
-    (property "Footprint" "Package_TO_SOT_SMD:SOT-23-6_Handsoldering" (id 2) (at 226.06 66.04 0)
-      (effects (font (size 1.27 1.27)) hide)
-    )
-    (property "Datasheet" "https://www.ti.com/lit/ds/symlink/sn74lvc2g17.pdf" (id 3) (at 226.06 63.5 0)
-      (effects (font (size 1.27 1.27)) hide)
-    )
-    (property "Part Number" "SN74LVC2G17DBVR" (id 4) (at 226.06 78.74 0)
-      (effects (font (size 1.27 1.27)) hide)
-    )
+  (symbol (lib_name "74LVC2G17_3") (lib_id "qds-cv-lib-sym:74LVC2G17") (at 207.01 151.13 0) (unit 1)
+    (in_bom yes) (on_board yes) (fields_autoplaced)
+    (property "Reference" "U704" (id 0) (at 207.645 143.51 0))
+    (property "Value" "74LVC2G17" (id 1) (at 207.645 146.05 0))
+    (property "Footprint" "Package_TO_SOT_SMD:SOT-23-6_Handsoldering" (id 2) (at 207.01 138.43 0)
+      (effects (font (size 1.27 1.27)) hide)
+    )
+    (property "Datasheet" "https://www.ti.com/lit/ds/symlink/sn74lvc2g17.pdf" (id 3) (at 207.01 135.89 0)
+      (effects (font (size 1.27 1.27)) hide)
+    )
+    (property "Part Number" "SN74LVC2G17DBVR" (id 4) (at 207.01 151.13 0)
+      (effects (font (size 1.27 1.27)) hide)
+    )
