File: pcb/cad/quench-trigger.kicad_sch (KiCad schematic)
At the start: 38 parts, among them J701 Conn_Coaxial, J702 DB9_Female, K701 FINDER-30.22, Q701 BC846B, SW701 RST, SW702 TRIG, U701 74HCS08, U702 74HC574, U703 74LV132, U704 74LVC2G17, U705 74LVC2G17, U706 HFBR-1521Z

Commit message: Preliminary placement of components from detection to validation stages
Parts:
- U702: footprint Package_SO:TSSOP-20_4.4x6.5mm_P0.65mm -> Package_SO:SO-20_12.8x7.5mm_P1.27mm; Manufacturer Texas -> NXP; Part Number SN74HCT574 -> 74HC574D
Changed lines of the file:
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@@
       (effects (font (size 1.27 1.27)) (justify left))
     )
-    (property "Footprint" "Package_SO:TSSOP-20_4.4x6.5mm_P0.65mm" (id 2) (at 186.69 64.77 0)
+    (property "Footprint" "Package_SO:SO-20_12.8x7.5mm_P1.27mm" (id 2) (at 186.69 64.77 0)
       (effects (font (size 1.27 1.27)) hide)
     )
-    (property "Datasheet" "https://www.ti.com/lit/ds/symlink/sn74hct574.pdf" (id 3) (at 186.69 64.77 0)
+    (property "Datasheet" "https://assets.nexperia.com/documents/data-sheet/74HC_HCT574.pdf" (id 3) (at 186.69 64.77 0)
       (effects (font (size 1.27 1.27)) hide)
     )
@@
       (effects (font (size 1.27 1.27)) hide)
     )
-    (property "Manufacturer" "Texas" (id 5) (at 186.69 64.77 0)
+    (property "Manufacturer" "NXP" (id 5) (at 186.69 64.77 0)
       (effects (font (size 1.27 1.27)) hide)
     )
-    (property "Part Number" "SN74HCT574" (id 6) (at 186.69 64.77 0)
+    (property "Part Number" "74HC574D" (id 6) (at 186.69 64.77 0)
       (effects (font (size 1.27 1.27)) hide)
     )

Commit message: Reposition of channels and connectors, place and route trigger and actuation circuit
Connections:
- net +5V: now also LD701.2 (A), LD702.2 (A), LD703.2 (A), LD704.2 (A), LD705.2 (A); no longer R701.1, R702.1, R703.1, R704.1, R705.1
- net Earth: now also J702.7, U703.4, U703.5, U704.3; no longer J702.6, U703.12, U703.13, U705.3
- net ILOCK_11: now also J702.5; no longer J702.3
- net ILOCK_12: now also J702.9; no longer J702.8
- net ILOCK_22: now also J702.8; no longer J702.9
- net REMOTE_RST+: now also U703.9; no longer U703.10
- net SW_TRIG+: now also J702.6; no longer J702.2
- net SW_TRIG-: now also J702.2, U701.9, U702.6 (D4); no longer J702.7, U701.13, U702.7 (D5)
- net TRIG-CH-A: now also U702.2 (D0); no longer U702.3 (D1)
- net TRIG-CH-B: now also U702.3 (D1); no longer U702.4 (D2)
- net TRIG-CH-C: now also U702.4 (D2); no longer U702.5 (D3)
- net TRIG-CH-D: now also U702.5 (D3); no longer U702.6 (D4)
- net at U704.4: no longer R712.1
- net at R706.1: now also U705.6; no longer U704.6
- net at R701.2: now also U702.19 (Q0); no longer LD701.2 (A)
- net at U703.1, U703.2: now also U701.8, U702.7 (D5); no longer U701.11, U702.2 (D0)
- net at U703.3: now also U703.13; no longer U703.4
- net at U702.14 (Q5): now also TP703.1, U703.12, U704.1, U705.1, U705.3; no longer LD705.1 (K)
- net at U702.15 (Q4): now also R705.2; no longer LD704.1 (K)
- net at U702.16 (Q3): now also R704.2; no longer LD703.1 (K)
- net at U702.17 (Q2): now also R703.2; no longer LD702.1 (K)
- net at LD701.1 (K): now also R701.1; no longer U702.18 (Q1)
- net at U701.10: now also U701.11; no longer U701.6
- net at U701.12: now also U701.6; no longer U701.8
- net at U701.3: now also U701.13; no longer U701.9
- net at R702.2: now also U702.18 (Q1); no longer LD702.2 (A)
- net at R710.1: now also U705.4; no longer U705.6
- new net: R712.1, U704.6
- new net: LD703.1 (K), R703.1
- new net: LD702.1 (K), R702.1
- new net: U703.10, U703.11
- new net: LD704.1 (K), R704.1
- new net: LD705.1 (K), R705.1
Other:
- moved on the sheet: LD701, LD702, LD703, LD704, LD705, R701, R702, R703, R704, R705, TP703, U701C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

Commit message: Replicate detection layout for all channels, place and route 5V-REF circuit
Connections:
- net REMOTE_RST+: now also J702.6; no longer J702.1
- net SW_TRIG+: now also J702.2; no longer J702.6
- net SW_TRIG-: now also J702.1; no longer J702.2
Changed lines of the file:
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@@
     (effects (font (size 1.27 1.27)) (justify right bottom))
   )
-  (label "REMOTE_RST+" (at 107.95 110.49 180)
+  (label "REMOTE_RST+" (at 107.95 113.03 180)
     (effects (font (size 1.27 1.27)) (justify right bottom))
   )
@@
     (effects (font (size 1.27 1.27)) (justify left bottom))
   )
-  (label "SW_TRIG+" (at 107.95 113.03 180)
+  (label "SW_TRIG+" (at 107.95 115.57 180)
     (effects (font (size 1.27 1.27)) (justify right bottom))
   )
@@
     (effects (font (size 1.27 1.27)) (justify right bottom))
   )
-  (label "SW_TRIG-" (at 107.95 115.57 180)
+  (label "SW_TRIG-" (at 107.95 110.49 180)
     (effects (font (size 1.27 1.27)) (justify right bottom))
   )

Commit message: Improve window comparator, +5V-REF and relay driver circuits close #19 close #20 close #22
Parts:
- added D702: SMBJ15A, Diode_SMD:D_SMB, symbol Diode:SM6T15A
Connections:
- net at K701.A1, R707.2: now also D702.2 (A2); no longer D701.1 (K)
- new net: D701.1 (K), D702.1 (A1)
Other:
- moved on the sheet: D701, K701, Q701, R707, R710, R712, U704A, U705B, U706

Commit message: Apply several changes based on test results - replace validation time 4k7 resistor by a 8k2, close #21 - remove pull-up resistor from AMC1200 positive input - split voltage taps pull-up/down resistors into 2 footprints each - change C204,304,404,504 footprints from 0603 to 0805 - include bypass switch for software trigger - remove test points from voltage taps - change window comparator input resistor to 4k7 - include footprint for a 0805 capacitor at the window comparator input
Parts:
- added SW703: SW_SPST, Button_Switch_THT:SW_DIP_SPSTx01_Slide_9.78x4.72mm_W7.62mm_P2.54mm, symbol Switch:SW_SPST
- R708, R709: Part Number 0805W8F1200T5E -> 0805W8F4701T5E
Connections:
- net SW_TRIG+: now also SW703.2 (B)
- net SW_TRIG-: now also SW703.1 (A)
Other:
- note added: "bypass"
- moved on the sheet: R709
Changed lines of the file:
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@@
   (junction (at 186.69 85.09) (diameter 0) (color 0 0 0 0)
+  )
+  (junction (at 68.58 108.585) (diameter 0) (color 0 0 0 0)
   )
   (junction (at 243.84 34.925) (diameter 0) (color 0 0 0 0)
@@
     (stroke (width 0) (type default) (color 0 0 0 0))
   )
+  (wire (pts (xy 68.58 119.38) (xy 68.58 120.015))
+    (stroke (width 0) (type default) (color 0 0 0 0))
+  )
   (wire (pts (xy 228.6 34.925) (xy 236.22 34.925))
     (stroke (width 0) (type default) (color 0 0 0 0))
@@
     (stroke (width 0) (type default) (color 0 0 0 0))
   )
-  (wire (pts (xy 68.58 112.395) (xy 68.58 116.205))
+  (wire (pts (xy 68.58 108.585) (xy 57.785 108.585))
     (stroke (width 0) (type default) (color 0 0 0 0))
   )
@@
     (stroke (width 0) (type default) (color 0 0 0 0))
   )
-  (wire (pts (xy 57.785 116.205) (xy 68.58 116.205))
-    (stroke (width 0) (type default) (color 0 0 0 0))
-  )
   (wire (pts (xy 191.77 104.14) (xy 217.17 104.14))
     (stroke (width 0) (type default) (color 0 0 0 0))
@@
     (stroke (width 0) (type default) (color 0 0 0 0))
   )
+  (wire (pts (xy 68.58 107.315) (xy 68.58 108.585))
+    (stroke (width 0) (type default) (color 0 0 0 0))
+  )
   (wire (pts (xy 230.505 126.365) (xy 239.395 126.365))
     (stroke (width 0) (type default) (color 0 0 0 0))
@@
     (stroke (width 0) (type default) (color 0 0 0 0))
   )
+  (wire (pts (xy 68.58 109.22) (xy 68.58 108.585))
+    (stroke (width 0) (type default) (color 0 0 0 0))
+  )
   (wire (pts (xy 138.43 158.115) (xy 149.86 158.115))
     (stroke (width 0) (type default) (color 0 0 0 0))
@@
     (stroke (width 0) (type default) (color 0 0 0 0))
   )
-  (wire (pts (xy 68.58 103.505) (xy 68.58 104.775))
-    (stroke (width 0) (type default) (color 0 0 0 0))
-  )
   (wire (pts (xy 138.43 183.515) (xy 149.86 183.515))
     (stroke (width 0) (type default) (color 0 0 0 0))
@@
   (wire (pts (xy 35.56 58.42) (xy 44.45 58.42))
     (stroke (width 0) (type default) (color 0 0 0 0))
+  )
+  (text "bypass" (at 69.85 117.475 0)
+    (effects (font (size 1.27 1.27)) (justify left bottom))
   )
   (text "Triggers aggregation, indication and actuation" (at 59.69 26.67 0)
@@
     (effects (font (size 1.27 1.27)) (justify right bottom))
   )
-  (label "SW_TRIG+" (at 57.785 116.205 0)
+  (label "SW_TRIG+" (at 57.785 108.585 0)
     (effects (font (size 1.27 1.27)) (justify left bottom))
   )
@@
     (pin "2")
   )
+  (symbol (lib_id "Switch:SW_SPST") (at 68.58 114.3 90) (unit 1)
+    (in_bom yes) (on_board yes) (fields_autoplaced)
+    (property "Reference" "SW703" (id 0) (at 69.85 114.2999 90)
+      (effects (font (size 1.27 1.27)) (justify right))
+    )
+    (property "Value" "SW_SPST" (id 1) (at 70.485 115.5699 90)
+      (effects (font (size 1.27 1.27)) (justify right) hide)
+    )
+    (property "Footprint" "Button_Switch_THT:SW_DIP_SPSTx01_Slide_9.78x4.72mm_W7.62mm_P2.54mm" (id 2) (at 68.58 114.3 0)
+      (effects (font (size 1.27 1.27)) hide)
+    )
+    (property "Datasheet" "~" (id 3) (at 68.58 114.3 0)
+      (effects (font (size 1.27 1.27)) hide)
+    )
+    (pin "1")
+    (pin "2")
+  )
   (symbol (lib_name "74LV132_1") (lib_id "qds-cv-lib-sym:74LV132") (at 125.73 170.815 180) (unit 5)
     (in_bom yes) (on_board yes)
@@
     (pin "2")
   )
-  (symbol (lib_id "Device:R_US") (at 68.58 108.585 0) (unit 1)
-    (in_bom yes) (on_board yes) (fields_autoplaced)
-    (property "Reference" "R709" (id 0) (at 70.485 107.3149 0)
-      (effects (font (size 1.27 1.27)) (justify left))
-    )
-    (property "Value" "4.7k" (id 1) (at 70.485 109.8549 0)
-      (effects (font (size 1.27 1.27)) (justify left))
-    )
-    (property "Footprint" "Resistor_SMD:R_0805_2012Metric_Pad1.20x1.40mm_HandSolder" (id 2) (at 69.596 108.839 90)
-      (effects (font (size 1.27 1.27)) hide)
-    )
-    (property "Datasheet" "https://datasheet.lcsc.com/lcsc/2206010216_UNI-ROYAL-Uniroyal-Elec-0805W8F1002T5E_C17414.pdf" (id 3) (at 68.58 108.585 0)
-      (effects (font (size 1.27 1.27)) hide)
-    )
-    (property "Part Number" "0805W8F1200T5E" (id 4) (at 68.58 108.585 0)
-      (effects (font (size 1.27 1.27)) hide)
-    )
-    (property "Description" "Resistor 4k7 1% 0.125W SMD 0805" (id 5) (at 68.58 108.585 0)
-      (effects (font (size 1.27 1.27)) hide)
-    )
-    (property "Manufacturer" "Royalohm" (id 6) (at 68.58 108.585 0)
-      (effects (font (size 1.27 1.27)) hide)
-    )
-    (property "Vendor Link" "" (id 7) (at 68.58 108.585 0)
+  (symbol (lib_id "Device:R_US") (at 68.58 103.505 0) (unit 1)
+    (in_bom yes) (on_board yes) (fields_autoplaced)
+    (property "Reference" "R709" (id 0) (at 70.485 102.2349 0)
+      (effects (font (size 1.27 1.27)) (justify left))
+    )
+    (property "Value" "4.7k" (id 1) (at 70.485 104.7749 0)
+      (effects (font (size 1.27 1.27)) (justify left))
+    )
+    (property "Footprint" "Resistor_SMD:R_0805_2012Metric_Pad1.20x1.40mm_HandSolder" (id 2) (at 69.596 103.759 90)
+      (effects (font (size 1.27 1.27)) hide)
+    )
+    (property "Datasheet" "https://datasheet.lcsc.com/lcsc/2206010216_UNI-ROYAL-Uniroyal-Elec-0805W8F1002T5E_C17414.pdf" (id 3) (at 68.58 103.505 0)
+      (effects (font (size 1.27 1.27)) hide)
+    )
+    (property "Part Number" "0805W8F4701T5E" (id 4) (at 68.58 103.505 0)
+      (effects (font (size 1.27 1.27)) hide)
+    )
+    (property "Description" "Resistor 4k7 1% 0.125W SMD 0805" (id 5) (at 68.58 103.505 0)
+      (effects (font (size 1.27 1.27)) hide)
+    )
+    (property "Manufacturer" "Royalohm" (id 6) (at 68.58 103.505 0)
+      (effects (font (size 1.27 1.27)) hide)
+    )
+    (property "Vendor Link" "" (id 7) (at 68.58 103.505 0)
       (effects (font (size 1.27 1.27)) hide)
     )
@@
     (pin "2")
   )
-  (symbol (lib_id "power:+5V") (at 68.58 103.505 0) (unit 1)
-    (in_bom yes) (on_board yes) (fields_autoplaced)
-    (property "Reference" "#PWR0709" (id 0) (at 68.58 107.315 0)
-      (effects (font (size 1.27 1.27)) hide)
-    )
-    (property "Value" "+5V" (id 1) (at 68.58 97.79 0))
-    (property "Footprint" "" (id 2) (at 68.58 103.505 0)
-      (effects (font (size 1.27 1.27)) hide)
-    )
-    (property "Datasheet" "" (id 3) (at 68.58 103.505 0)
+  (symbol (lib_id "power:+5V") (at 68.58 99.695 0) (unit 1)
+    (in_bom yes) (on_board yes) (fields_autoplaced)
+    (property "Reference" "#PWR0709" (id 0) (at 68.58 103.505 0)
+      (effects (font (size 1.27 1.27)) hide)
+    )
+    (property "Value" "+5V" (id 1) (at 68.58 93.98 0))
+    (property "Footprint" "" (id 2) (at 68.58 99.695 0)
+      (effects (font (size 1.27 1.27)) hide)
+    )
+    (property "Datasheet" "" (id 3) (at 68.58 99.695 0)
       (effects (font (size 1.27 1.27)) hide)
     )
@@
       (effects (font (size 1.27 1.27)) hide)
     )
-    (property "Part Number" "0805W8F1200T5E" (id 4) (at 43.815 108.585 0)
-      (effects (font (size 1.27 1.27)) hide)
-    )
+    (property "Part Number" "0805W8F4701T5E" (id 4) (at 43.815 108.585 0)
+      (effects (font (size 1.27 1.27)) hide)
+    )

Commit message: Add stitching capacitors to isolated supply circuits
Connections:
- net SW_TRIG+: now also J702.1; no longer J702.2
- net SW_TRIG-: now also J702.2; no longer J702.1
Changed lines of the file:
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@@
     (effects (font (size 1.27 1.27)) (justify left bottom))
   )
-  (label "SW_TRIG+" (at 107.95 115.57 180)
+  (label "SW_TRIG+" (at 107.95 110.49 180)
     (effects (font (size 1.27 1.27)) (justify right bottom))
   )
@@
     (effects (font (size 1.27 1.27)) (justify right bottom))
   )
-  (label "SW_TRIG-" (at 107.95 110.49 180)
+  (label "SW_TRIG-" (at 107.95 115.57 180)
     (effects (font (size 1.27 1.27)) (justify right bottom))
   )

Commit message: Place test-points, improve isolated circuit layout (channel D only)
Parts:
- C701, C702, C703, C704, C705: footprint Capacitor_SMD:C_0603_1608Metric_Pad1.08x0.95mm_HandSolder -> Capacitor_SMD:C_0805_2012Metric_Pad1.18x1.45mm_HandSolder; CNPEM Code AP107349 -> (none); Manufacturer TDK -> Kyocera; Part Number C1608X7R1H104K080AA -> 08055C104KAZ2A; Vendor Link https://br.mouser.com/ProductDetail/TDK/C1608X7R1H104K080AA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 -> (none)
- TP703: footprint (none) -> qds-cv-lib:TestPoint_Keystone_5010-5014_Multipurpose
Connections:
- net FF-CLK: now reaches TP702.1, U702.11 (Cp), U703.8

Commit message: Improve reset and sw_trigger circuits - add RC filter for reset signal (R713, C706) - change values of sw-trigger pull-up/down resistors (R709, R711) and add capacitor (C707)
Parts:
- added C706, C707: C, Capacitor_SMD:C_0805_2012Metric_Pad1.18x1.45mm_HandSolder, symbol Device:C
- added R713: R_US, Resistor_SMD:R_0805_2012Metric_Pad1.20x1.40mm_HandSolder, symbol Device:R_US
- R709: value 4.7k -> 270; Manufacturer Royalohm -> Fenghua Advance Technology; Part Number 0805W8F4701T5E -> RC-05K203JT
- R711: value 47k -> 4.7k; footprint Resistor_SMD:R_0603_1608Metric_Pad0.98x0.95mm_HandSolder -> Resistor_SMD:R_0805_2012Metric_Pad1.20x1.40mm_HandSolder; CNPEM Code AP107380 -> (none); Manufacturer Panasonic Electronic Components -> Royalohm; Part Number ERA-3AEB473V -> 0805W8F4701T5E; Vendor Link https://www.digikey.com/en/products/detail/ERA-3AEB473V/P47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 -> (none)
Connections:
- net Earth: now also C706.2, C707.2
- net REMOTE_RST+: now also R713.2; no longer U703.9
- net SW_TRIG-: now also C707.1
- new net RESET: C706.1, R713.1, U703.9
Other:
- moved on the sheet: J702, R709, SW702, SW703
