File: pcb/cad/detection-validation.kicad_sch (KiCad schematic)
At the start: 39 parts, among them SW401 SW_DIP_x05, U401 74HC123, U402 74HC123, U403 74HC123, U404 74HC123, U405 74HC32D, U406 74HC32D, U408 74HCS08

Commit message: update components specification
Parts:
- R401, R402, R403, R404: footprint (none) -> Resistor_SMD:R_0805_2012Metric_Pad1.20x1.40mm_HandSolder; Part Number (none) -> ERJ-6GEYJ102V
- R405, R406, R407, R408: Part Number (none) -> RC-05K203IT
- R409, R410, R411, R412: value 2k -> 2.2k; footprint (none) -> Resistor_SMD:R_0805_2012Metric_Pad1.20x1.40mm_HandSolder; Part Number (none) -> RC0805FR-072K2L
Changed lines of the file:
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@@
     (in_bom yes) (on_board yes)
     (property "Reference" "R409" (id 0) (at 246.888 45.339 0))
-    (property "Value" "2k" (id 1) (at 246.888 47.879 0))
-    (property "Footprint" "" (id 2) (at 243.332 46.355 90)
-      (effects (font (size 1.27 1.27)) hide)
-    )
-    (property "Datasheet" "~" (id 3) (at 244.348 46.609 0)
+    (property "Value" "2.2k" (id 1) (at 246.888 47.879 0))
+    (property "Footprint" "Resistor_SMD:R_0805_2012Metric_Pad1.20x1.40mm_HandSolder" (id 2) (at 243.332 46.355 90)
+      (effects (font (size 1.27 1.27)) hide)
+    )
+    (property "Datasheet" "https://www.yageo.com/upload/media/product/productsearch/datasheet/rchip/PYu-RC_Group_51_RoHS_L_12.pdf" (id 3) (at 244.348 46.609 0)
+      (effects (font (size 1.27 1.27)) hide)
+    )
+    (property "Part Number" "RC0805FR-072K2L" (id 4) (at 244.348 46.609 0)
       (effects (font (size 1.27 1.27)) hide)
     )
@@
     (property "Reference" "R401" (id 0) (at 33.02 31.115 90))
     (property "Value" "1k" (id 1) (at 33.02 33.655 90))
-    (property "Footprint" "" (id 2) (at 32.766 38.481 90)
-      (effects (font (size 1.27 1.27)) hide)
-    )
-    (property "Datasheet" "~" (id 3) (at 33.02 37.465 0)
+    (property "Footprint" "Resistor_SMD:R_0805_2012Metric_Pad1.20x1.40mm_HandSolder" (id 2) (at 32.766 38.481 90)
+      (effects (font (size 1.27 1.27)) hide)
+    )
+    (property "Datasheet" "https://industrial.panasonic.com/cdbs/www-data/pdf/RDA0000/AOA0000C301.pdf" (id 3) (at 33.02 37.465 0)
+      (effects (font (size 1.27 1.27)) hide)
+    )
+    (property "Part Number" "ERJ-6GEYJ102V" (id 4) (at 33.02 37.465 0)
       (effects (font (size 1.27 1.27)) hide)
     )
@@
       (effects (font (size 1.27 1.27)) hide)
     )
+    (property "Part Number" "RC-05K203IT" (id 4) (at 144.78 175.26 0)
+      (effects (font (size 1.27 1.27)) hide)
+    )
     (pin "1")
     (pin "2")
@@
     (in_bom yes) (on_board yes)
     (property "Reference" "R410" (id 0) (at 253.238 45.339 0))
-    (property "Value" "2k" (id 1) (at 253.238 47.879 0))
-    (property "Footprint" "" (id 2) (at 249.682 46.355 90)
-      (effects (font (size 1.27 1.27)) hide)
-    )
-    (property "Datasheet" "~" (id 3) (at 250.698 46.609 0)
+    (property "Value" "2.2k" (id 1) (at 253.238 47.879 0))
+    (property "Footprint" "Resistor_SMD:R_0805_2012Metric_Pad1.20x1.40mm_HandSolder" (id 2) (at 249.682 46.355 90)
+      (effects (font (size 1.27 1.27)) hide)
+    )
+    (property "Datasheet" "https://www.yageo.com/upload/media/product/productsearch/datasheet/rchip/PYu-RC_Group_51_RoHS_L_12.pdf" (id 3) (at 250.698 46.609 0)
+      (effects (font (size 1.27 1.27)) hide)
+    )
+    (property "Part Number" "RC0805FR-072K2L" (id 4) (at 250.698 46.609 0)
       (effects (font (size 1.27 1.27)) hide)
     )
@@
     (property "Reference" "R404" (id 0) (at 34.29 157.48 90))
     (property "Value" "1k" (id 1) (at 34.29 160.02 90))
-    (property "Footprint" "" (id 2) (at 34.036 164.846 90)
-      (effects (font (size 1.27 1.27)) hide)
-    )
-    (property "Datasheet" "~" (id 3) (at 34.29 163.83 0)
+    (property "Footprint" "Resistor_SMD:R_0805_2012Metric_Pad1.20x1.40mm_HandSolder" (id 2) (at 34.036 164.846 90)
+      (effects (font (size 1.27 1.27)) hide)
+    )
+    (property "Datasheet" "https://industrial.panasonic.com/cdbs/www-data/pdf/RDA0000/AOA0000C301.pdf" (id 3) (at 34.29 163.83 0)
+      (effects (font (size 1.27 1.27)) hide)
+    )
+    (property "Part Number" "ERJ-6GEYJ102V" (id 4) (at 34.29 163.83 0)
       (effects (font (size 1.27 1.27)) hide)
     )
@@
       (effects (font (size 1.27 1.27)) hide)
     )
+    (property "Part Number" "RC-05K203IT" (id 4) (at 144.78 90.17 0)
+      (effects (font (size 1.27 1.27)) hide)
+    )
     (pin "1")
     (pin "2")
@@
       (effects (font (size 1.27 1.27)) hide)
     )
+    (property "Part Number" "RC-05K203IT" (id 4) (at 143.51 48.895 0)
+      (effects (font (size 1.27 1.27)) hide)
+    )
     (pin "1")
     (pin "2")
@@
     (property "Reference" "R403" (id 0) (at 34.29 114.3 90))
     (property "Value" "1k" (id 1) (at 34.29 116.84 90))
-    (property "Footprint" "" (id 2) (at 34.036 121.666 90)
-      (effects (font (size 1.27 1.27)) hide)
-    )
-    (property "Datasheet" "~" (id 3) (at 34.29 120.65 0)
+    (property "Footprint" "Resistor_SMD:R_0805_2012Metric_Pad1.20x1.40mm_HandSolder" (id 2) (at 34.036 121.666 90)
+      (effects (font (size 1.27 1.27)) hide)
+    )
+    (property "Datasheet" "https://industrial.panasonic.com/cdbs/www-data/pdf/RDA0000/AOA0000C301.pdf" (id 3) (at 34.29 120.65 0)
+      (effects (font (size 1.27 1.27)) hide)
+    )
+    (property "Part Number" "ERJ-6GEYJ102V" (id 4) (at 34.29 120.65 0)
       (effects (font (size 1.27 1.27)) hide)
     )
@@
     (in_bom yes) (on_board yes)
     (property "Reference" "R411" (id 0) (at 259.588 45.339 0))
-    (property "Value" "2k" (id 1) (at 259.588 47.879 0))
-    (property "Footprint" "" (id 2) (at 256.032 46.355 90)
-      (effects (font (size 1.27 1.27)) hide)
-    )
-    (property "Datasheet" "~" (id 3) (at 257.048 46.609 0)
+    (property "Value" "2.2k" (id 1) (at 259.588 47.879 0))
+    (property "Footprint" "Resistor_SMD:R_0805_2012Metric_Pad1.20x1.40mm_HandSolder" (id 2) (at 256.032 46.355 90)
+      (effects (font (size 1.27 1.27)) hide)
+    )
+    (property "Datasheet" "https://www.yageo.com/upload/media/product/productsearch/datasheet/rchip/PYu-RC_Group_51_RoHS_L_12.pdf" (id 3) (at 257.048 46.609 0)
+      (effects (font (size 1.27 1.27)) hide)
+    )
+    (property "Part Number" "RC0805FR-072K2L" (id 4) (at 257.048 46.609 0)
       (effects (font (size 1.27 1.27)) hide)
     )
@@
     (property "Reference" "R402" (id 0) (at 34.29 72.39 90))
     (property "Value" "1k" (id 1) (at 34.29 74.93 90))
-    (property "Footprint" "" (id 2) (at 34.036 79.756 90)
-      (effects (font (size 1.27 1.27)) hide)
-    )
-    (property "Datasheet" "~" (id 3) (at 34.29 78.74 0)
+    (property "Footprint" "Resistor_SMD:R_0805_2012Metric_Pad1.20x1.40mm_HandSolder" (id 2) (at 34.036 79.756 90)
+      (effects (font (size 1.27 1.27)) hide)
+    )
+    (property "Datasheet" "https://industrial.panasonic.com/cdbs/www-data/pdf/RDA0000/AOA0000C301.pdf" (id 3) (at 34.29 78.74 0)
+      (effects (font (size 1.27 1.27)) hide)
+    )
+    (property "Part Number" "ERJ-6GEYJ102V" (id 4) (at 34.29 78.74 0)
       (effects (font (size 1.27 1.27)) hide)
     )
@@
       (effects (font (size 1.27 1.27)) hide)
     )
+    (property "Part Number" "RC-05K203IT" (id 4) (at 144.78 132.08 0)
+      (effects (font (size 1.27 1.27)) hide)
+    )
     (pin "1")
     (pin "2")
@@
     (in_bom yes) (on_board yes)
     (property "Reference" "R412" (id 0) (at 265.938 45.339 0))
-    (property "Value" "2k" (id 1) (at 265.938 47.879 0))
-    (property "Footprint" "" (id 2) (at 262.382 46.355 90)
-      (effects (font (size 1.27 1.27)) hide)
-    )
-    (property "Datasheet" "~" (id 3) (at 263.398 46.609 0)
-      (effects (font (size 1.27 1.27)) hide)
-    )
+    (property "Value" "2.2k" (id 1) (at 265.938 47.879 0))
+    (property "Footprint" "Resistor_SMD:R_0805_2012Metric_Pad1.20x1.40mm_HandSolder" (id 2) (at 262.382 46.355 90)
+      (effects (font (size 1.27 1.27)) hide)
+    )
+    (property "Datasheet" "https://www.yageo.com/upload/media/product/productsearch/datasheet/rchip/PYu-RC_Group_51_RoHS_L_12.pdf" (id 3) (at 263.398 46.609 0)
+      (effects (font (size 1.27 1.27)) hide)
+    )
+    (property "Part Number" "RC0805FR-072K2L" (id 4) (at 263.398 46.609 0)
+      (effects (font (size 1.27 1.27)) hide)
+    )

Commit message: Update componentes fields and reference circuit
Parts:
- R401, R402, R403, R404: CNPEM Code (none) -> AP110784; Manufacturer (none) -> Panasonic Electronic Components
- R405, R406, R407, R408: footprint (none) -> Resistor_SMD:R_0805_2012Metric_Pad1.20x1.40mm_HandSolder
- R409, R410, R411, R412: CNPEM Code (none) -> MT104237; Manufacturer (none) -> Yageo; Vendor Link (none) -> https://www.digikey.com/en/products/detail/yageo/RC0805FR-0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
- RV401, RV402, RV403, RV404: Vendor Link (none) -> https://br.mouser.com/ProductDetail/Bourns/3224X-1-503E?qs=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
Other:
- title: (none) -> Detection Validation Circuits
Changed lines of the file:
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@@
   (paper "A4")
   (title_block
+    (title "Detection Validation Circuits")
     (rev "v1.0.0")
     (company "CNPEM - Brazilian Center for Research in Energy and Materials")
@@
       (effects (font (size 1.27 1.27)) hide)
     )
+    (property "CNPEM Code" "MT104237" (id 5) (at 244.348 46.609 0)
+      (effects (font (size 1.27 1.27)) hide)
+    )
+    (property "Manufacturer" "Yageo" (id 6) (at 244.348 46.609 0)
+      (effects (font (size 1.27 1.27)) hide)
+    )
+    (property "Description" "Resistor 2.2k 1% 0.125W SMD 0805" (id 7) (at 244.348 46.609 0)
+      (effects (font (size 1.27 1.27)) hide)
+    )
+    (property "Vendor Link" "https://www.digikey.com/en/products/detail/yageo/RC0805FR-072K2L/727676?utm_adgroup=Resistors&utm_source=google&utm_medium=cpc&utm_campaign=Dynamic%20Search_PT_Product&utm_term=&utm_content=Resistors&gclid=Cj0KCQjwiZqhBhCJARIsACHHEH8v6oZGyHIjUrtn7TkF_AQuRcQJr-qTERqKybnCllzX-CPJhH9mu5EaAnnzEALw_wcB" (id 8) (at 244.348 46.609 0)
+      (effects (font (size 1.27 1.27)) hide)
+    )
     (pin "1")
     (pin "2")
@@
     )
     (property "Part Number" "ERJ-6GEYJ102V" (id 4) (at 33.02 37.465 0)
+      (effects (font (size 1.27 1.27)) hide)
+    )
+    (property "CNPEM Code" "AP110784" (id 5) (at 33.02 37.465 0)
+      (effects (font (size 1.27 1.27)) hide)
+    )
+    (property "Manufacturer" "Panasonic Electronic Components" (id 6) (at 33.02 37.465 0)
       (effects (font (size 1.27 1.27)) hide)
     )
@@
     (property "Reference" "R408" (id 0) (at 140.97 168.91 90))
     (property "Value" "20k" (id 1) (at 140.97 171.45 90))
-    (property "Footprint" "" (id 2) (at 141.224 174.244 90)
+    (property "Footprint" "Resistor_SMD:R_0805_2012Metric_Pad1.20x1.40mm_HandSolder" (id 2) (at 141.224 174.244 90)
       (effects (font (size 1.27 1.27)) hide)
     )
@@
       (effects (font (size 1.27 1.27)) hide)
     )
+    (property "Description" "Trimpot 50k, 12 turns, 10% tolerance, 4mm SMD Top Adjust" (id 6) (at 43.18 163.83 0)
+      (effects (font (size 1.27 1.27)) hide)
+    )
+    (property "Vendor Link" "https://br.mouser.com/ProductDetail/Bourns/3224X-1-503E?qs=A%2FVUe%2FMZWjw7UCYo8RtHVg%3D%3D" (id 7) (at 43.18 163.83 0)
+      (effects (font (size 1.27 1.27)) hide)
+    )
     (pin "1")
     (pin "2")
@@
     )
     (property "Part Number" "RC0805FR-072K2L" (id 4) (at 250.698 46.609 0)
+      (effects (font (size 1.27 1.27)) hide)
+    )
+    (property "CNPEM Code" "MT104237" (id 5) (at 250.698 46.609 0)
+      (effects (font (size 1.27 1.27)) hide)
+    )
+    (property "Manufacturer" "Yageo" (id 6) (at 250.698 46.609 0)
+      (effects (font (size 1.27 1.27)) hide)
+    )
+    (property "Description" "Resistor 2.2k 1% 0.125W SMD 0805" (id 7) (at 250.698 46.609 0)
+      (effects (font (size 1.27 1.27)) hide)
+    )
+    (property "Vendor Link" "https://www.digikey.com/en/products/detail/yageo/RC0805FR-072K2L/727676?utm_adgroup=Resistors&utm_source=google&utm_medium=cpc&utm_campaign=Dynamic%20Search_PT_Product&utm_term=&utm_content=Resistors&gclid=Cj0KCQjwiZqhBhCJARIsACHHEH8v6oZGyHIjUrtn7TkF_AQuRcQJr-qTERqKybnCllzX-CPJhH9mu5EaAnnzEALw_wcB" (id 8) (at 250.698 46.609 0)
       (effects (font (size 1.27 1.27)) hide)
     )
@@
       (effects (font (size 1.27 1.27)) hide)
     )
+    (property "CNPEM Code" "AP110784" (id 5) (at 34.29 163.83 0)
+      (effects (font (size 1.27 1.27)) hide)
+    )
+    (property "Manufacturer" "Panasonic Electronic Components" (id 6) (at 34.29 163.83 0)
+      (effects (font (size 1.27 1.27)) hide)
+    )
     (pin "1")
     (pin "2")
@@
     (property "Reference" "R406" (id 0) (at 140.97 83.82 90))
     (property "Value" "20k" (id 1) (at 140.97 86.36 90))
-    (property "Footprint" "" (id 2) (at 141.224 89.154 90)
+    (property "Footprint" "Resistor_SMD:R_0805_2012Metric_Pad1.20x1.40mm_HandSolder" (id 2) (at 141.224 89.154 90)
       (effects (font (size 1.27 1.27)) hide)
     )
@@
     (property "Reference" "R405" (id 0) (at 139.7 42.545 90))
     (property "Value" "20k" (id 1) (at 139.7 45.085 90))
-    (property "Footprint" "" (id 2) (at 139.954 47.879 90)
+    (property "Footprint" "Resistor_SMD:R_0805_2012Metric_Pad1.20x1.40mm_HandSolder" (id 2) (at 139.954 47.879 90)
       (effects (font (size 1.27 1.27)) hide)
     )
@@
       (effects (font (size 1.27 1.27)) hide)
     )
+    (property "CNPEM Code" "AP110784" (id 5) (at 34.29 120.65 0)
+      (effects (font (size 1.27 1.27)) hide)
+    )
+    (property "Manufacturer" "Panasonic Electronic Components" (id 6) (at 34.29 120.65 0)
+      (effects (font (size 1.27 1.27)) hide)
+    )
     (pin "1")
     (pin "2")
@@
     )
     (property "Part Number" "3224X-1-503E" (id 5) (at 43.18 78.74 0)
+      (effects (font (size 1.27 1.27)) hide)
+    )
+    (property "Description" "Trimpot 50k, 12 turns, 10% tolerance, 4mm SMD Top Adjust" (id 6) (at 43.18 78.74 0)
+      (effects (font (size 1.27 1.27)) hide)
+    )
+    (property "Vendor Link" "https://br.mouser.com/ProductDetail/Bourns/3224X-1-503E?qs=A%2FVUe%2FMZWjw7UCYo8RtHVg%3D%3D" (id 7) (at 43.18 78.74 0)
       (effects (font (size 1.27 1.27)) hide)
     )
@@
     )
     (property "Part Number" "3224X-1-503E" (id 5) (at 43.18 120.65 0)
+      (effects (font (size 1.27 1.27)) hide)
+    )
+    (property "Description" "Trimpot 50k, 12 turns, 10% tolerance, 4mm SMD Top Adjust" (id 6) (at 43.18 120.65 0)
+      (effects (font (size 1.27 1.27)) hide)
+    )
+    (property "Vendor Link" "https://br.mouser.com/ProductDetail/Bourns/3224X-1-503E?qs=A%2FVUe%2FMZWjw7UCYo8RtHVg%3D%3D" (id 7) (at 43.18 120.65 0)
       (effects (font (size 1.27 1.27)) hide)
     )
@@
       (effects (font (size 1.27 1.27)) hide)
     )
+    (property "CNPEM Code" "MT104237" (id 5) (at 257.048 46.609 0)
+      (effects (font (size 1.27 1.27)) hide)
+    )
+    (property "Manufacturer" "Yageo" (id 6) (at 257.048 46.609 0)
+      (effects (font (size 1.27 1.27)) hide)
+    )
+    (property "Description" "Resistor 2.2k 1% 0.125W SMD 0805" (id 7) (at 257.048 46.609 0)
+      (effects (font (size 1.27 1.27)) hide)
+    )
+    (property "Vendor Link" "https://www.digikey.com/en/products/detail/yageo/RC0805FR-072K2L/727676?utm_adgroup=Resistors&utm_source=google&utm_medium=cpc&utm_campaign=Dynamic%20Search_PT_Product&utm_term=&utm_content=Resistors&gclid=Cj0KCQjwiZqhBhCJARIsACHHEH8v6oZGyHIjUrtn7TkF_AQuRcQJr-qTERqKybnCllzX-CPJhH9mu5EaAnnzEALw_wcB" (id 8) (at 257.048 46.609 0)
+      (effects (font (size 1.27 1.27)) hide)
+    )
     (pin "1")
     (pin "2")
@@
       (effects (font (size 1.27 1.27)) hide)
     )
+    (property "Description" "Trimpot 50k, 12 turns, 10% tolerance, 4mm SMD Top Adjust" (id 6) (at 41.91 37.465 0)
+      (effects (font (size 1.27 1.27)) hide)
+    )
+    (property "Vendor Link" "https://br.mouser.com/ProductDetail/Bourns/3224X-1-503E?qs=A%2FVUe%2FMZWjw7UCYo8RtHVg%3D%3D" (id 7) (at 41.91 37.465 0)
+      (effects (font (size 1.27 1.27)) hide)
+    )
     (pin "1")
     (pin "2")
@@
       (effects (font (size 1.27 1.27)) hide)
     )
+    (property "CNPEM Code" "AP110784" (id 5) (at 34.29 78.74 0)
+      (effects (font (size 1.27 1.27)) hide)
+    )
+    (property "Manufacturer" "Panasonic Electronic Components" (id 6) (at 34.29 78.74 0)
+      (effects (font (size 1.27 1.27)) hide)
+    )
     (pin "1")
     (pin "2")
@@
     (property "Reference" "R407" (id 0) (at 140.97 125.73 90))
     (property "Value" "20k" (id 1) (at 140.97 128.27 90))
-    (property "Footprint" "" (id 2) (at 141.224 131.064 90)
+    (property "Footprint" "Resistor_SMD:R_0805_2012Metric_Pad1.20x1.40mm_HandSolder" (id 2) (at 141.224 131.064 90)
       (effects (font (size 1.27 1.27)) hide)
     )
@@
       (effects (font (size 1.27 1.27)) hide)
     )
+    (property "CNPEM Code" "MT104237" (id 5) (at 263.398 46.609 0)
+      (effects (font (size 1.27 1.27)) hide)
+    )
+    (property "Manufacturer" "Yageo" (id 6) (at 263.398 46.609 0)
+      (effects (font (size 1.27 1.27)) hide)
+    )
+    (property "Description" "Resistor 2.2k 1% 0.125W SMD 0805" (id 7) (at 263.398 46.609 0)
+      (effects (font (size 1.27 1.27)) hide)
+    )
+    (property "Vendor Link" "https://www.digikey.com/en/products/detail/yageo/RC0805FR-072K2L/727676?utm_adgroup=Resistors&utm_source=google&utm_medium=cpc&utm_campaign=Dynamic%20Search_PT_Product&utm_term=&utm_content=Resistors&gclid=Cj0KCQjwiZqhBhCJARIsACHHEH8v6oZGyHIjUrtn7TkF_AQuRcQJr-qTERqKybnCllzX-CPJhH9mu5EaAnnzEALw_wcB" (id 8) (at 263.398 46.609 0)
+      (effects (font (size 1.27 1.27)) hide)
+    )

Commit message: Fixed footprints 3D models orientation
Parts:
- RV401, RV402, RV403, RV404: footprint Potentiometer_SMD:Potentiometer_Bourns_3224X_Vertical -> qds-cv-lib:Potentiometer_Bourns_3224X_Vertical
Changed lines of the file:
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@@
     (property "Reference" "RV404" (id 0) (at 43.18 157.48 90))
     (property "Value" "50k" (id 1) (at 43.18 160.02 90))
-    (property "Footprint" "Potentiometer_SMD:Potentiometer_Bourns_3224X_Vertical" (id 2) (at 43.18 163.83 0)
+    (property "Footprint" "qds-cv-lib:Potentiometer_Bourns_3224X_Vertical" (id 2) (at 43.18 163.83 0)
       (effects (font (size 1.27 1.27)) hide)
     )
@@
     (property "Reference" "RV402" (id 0) (at 43.18 72.39 90))
     (property "Value" "50k" (id 1) (at 43.18 74.93 90))
-    (property "Footprint" "Potentiometer_SMD:Potentiometer_Bourns_3224X_Vertical" (id 2) (at 43.18 78.74 0)
+    (property "Footprint" "qds-cv-lib:Potentiometer_Bourns_3224X_Vertical" (id 2) (at 43.18 78.74 0)
       (effects (font (size 1.27 1.27)) hide)
     )
@@
     (property "Reference" "RV403" (id 0) (at 43.18 114.3 90))
     (property "Value" "50k" (id 1) (at 43.18 116.84 90))
-    (property "Footprint" "Potentiometer_SMD:Potentiometer_Bourns_3224X_Vertical" (id 2) (at 43.18 120.65 0)
+    (property "Footprint" "qds-cv-lib:Potentiometer_Bourns_3224X_Vertical" (id 2) (at 43.18 120.65 0)
       (effects (font (size 1.27 1.27)) hide)
     )
@@
     (property "Reference" "RV401" (id 0) (at 41.91 31.115 90))
     (property "Value" "50k" (id 1) (at 41.91 33.655 90))
-    (property "Footprint" "Potentiometer_SMD:Potentiometer_Bourns_3224X_Vertical" (id 2) (at 41.91 37.465 0)
-      (effects (font (size 1.27 1.27)) hide)
-    )
+    (property "Footprint" "qds-cv-lib:Potentiometer_Bourns_3224X_Vertical" (id 2) (at 41.91 37.465 0)
+      (effects (font (size 1.27 1.27)) hide)
+    )
