File: pcb/cad/detection-validation.kicad_sch (KiCad schematic)
At the start: 39 parts, among them SW601 SW_DIP_x05, U601 74HC32D, U602 74HC123, U603 74HCS08, U604 74HC32D, U605 74HC123, U606 74HC123, U607 74HC123

Commit message: Replace schematic symbols and text fields for a better view
Other:
- moved on the sheet: C607, C608, C609, C610, C611, C612, C613, R602, R603, R604, R605, SW601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

Commit message: Make modifications needed for single channel board
Parts:
- removed C603, C605, C614: 2.2u, Capacitor_SMD:C_0603_1608Metric_Pad1.08x0.95mm_HandSolder, symbol Device:C
- removed C604, C606, C615: 470p, Capacitor_SMD:C_0805_2012Metric_Pad1.18x1.45mm_HandSolder, symbol Device:C
- removed C608, C610, C611, C612: 100n, Capacitor_SMD:C_0603_1608Metric_Pad1.08x0.95mm_HandSolder, symbol Device:C
- removed R607, R609, R611: 1k, Resistor_SMD:R_0805_2012Metric_Pad1.20x1.40mm_HandSolder, symbol Device:R_US
- removed R608, R610, R612: 20k, Resistor_SMD:R_0805_2012Metric_Pad1.20x1.40mm_HandSolder, symbol Device:R_US
- removed RV602, RV603, RV604: 50k, qds-cv-lib:Potentiometer_Bourns_3224X_Vertical, symbol Device:R_Potentiometer_Trim_US
- removed U604: 74HC32D, Package_SO:SO-14_3.9x8.65mm_P1.27mm, symbol qds-cv-lib-sym:74HC32D
- removed U605, U606, U607: 74HC123, Package_SO:SOIC-16_3.9x9.9mm_P1.27mm, symbol qds-cv-lib-sym:74HC123
- added C? (x3): 470p, Capacitor_SMD:C_0805_2012Metric_Pad1.18x1.45mm_HandSolder, symbol Device:C
- added R? (x3): 20k, Resistor_SMD:R_0805_2012Metric_Pad1.20x1.40mm_HandSolder, symbol Device:R_US
Connections:
- net VAL-B is gone; now on net Earth: U601.13, U602.9 (A)
- net +5V: no longer U602.10 (B), U602.11 (Clr)
- net Earth: now also U601.10, U601.12, U601.9, U602.10 (B), U602.11 (Clr), U603.10, U603.12, U603.13, U603.4, U603.5, U603.9, C?.2, C?.2, C?.2, R?.1, R?.1, R?.1; no longer U602.6 (Cx)
- net TRIG-CH-B: now also C?.1, R?.2
- net TRIG-CH-C: now also C?.1, R?.2
- net TRIG-CH-D: now also C?.1, R?.2
- net at U602.12 (~{Q}): no longer U601.10
- net at U601.8: no longer U603.4
- net at U601.11: no longer U603.5
- now unconnected: U602.5 (Q)
Other:
- moved on the sheet: C607, C609, C613, U601E, U602C, U603E

Commit message: Add test points and extra resistors for temporary use. Remove power supplies
Parts:
- gave numbers to parts that had none: 6
Changed lines of the file:
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@@
   (symbol (lib_id "power:Earth") (at 117.475 127 0) (unit 1)
     (in_bom yes) (on_board yes) (fields_autoplaced)
-    (property "Reference" "#PWR?" (id 0) (at 117.475 133.35 0)
+    (property "Reference" "#PWR0108" (id 0) (at 117.475 133.35 0)
       (effects (font (size 1.27 1.27)) hide)
     )
@@
   (symbol (lib_id "Device:C") (at 161.925 85.725 0) (unit 1)
     (in_bom yes) (on_board yes) (fields_autoplaced)
-    (property "Reference" "C?" (id 0) (at 165.735 84.4549 0)
-      (effects (font (size 1.27 1.27)) (justify left))
-    )
-    (property "Value" "470p" (id 1) (at 165.735 86.9949 0)
+    (property "Reference" "C604" (id 0) (at 165.1 84.4549 0)
+      (effects (font (size 1.27 1.27)) (justify left))
+    )
+    (property "Value" "470p" (id 1) (at 165.1 86.9949 0)
       (effects (font (size 1.27 1.27)) (justify left))
     )
@@
   (symbol (lib_id "Device:R_US") (at 153.67 123.19 90) (unit 1)
     (in_bom yes) (on_board yes) (fields_autoplaced)
-    (property "Reference" "R?" (id 0) (at 153.67 116.84 90))
+    (property "Reference" "R612" (id 0) (at 153.67 116.84 90))
     (property "Value" "20k" (id 1) (at 153.67 119.38 90))
     (property "Footprint" "Resistor_SMD:R_0805_2012Metric_Pad1.20x1.40mm_HandSolder" (id 2) (at 153.924 122.174 90)
@@
   (symbol (lib_id "Device:C") (at 161.925 107.315 0) (unit 1)
     (in_bom yes) (on_board yes) (fields_autoplaced)
-    (property "Reference" "C?" (id 0) (at 165.735 106.0449 0)
-      (effects (font (size 1.27 1.27)) (justify left))
-    )
-    (property "Value" "470p" (id 1) (at 165.735 108.5849 0)
+    (property "Reference" "C606" (id 0) (at 165.1 106.0449 0)
+      (effects (font (size 1.27 1.27)) (justify left))
+    )
+    (property "Value" "470p" (id 1) (at 165.1 108.5849 0)
       (effects (font (size 1.27 1.27)) (justify left))
     )
@@
   (symbol (lib_id "Device:C") (at 161.925 128.27 0) (unit 1)
     (in_bom yes) (on_board yes) (fields_autoplaced)
-    (property "Reference" "C?" (id 0) (at 165.735 126.9999 0)
-      (effects (font (size 1.27 1.27)) (justify left))
-    )
-    (property "Value" "470p" (id 1) (at 165.735 129.5399 0)
+    (property "Reference" "C615" (id 0) (at 165.1 126.9999 0)
+      (effects (font (size 1.27 1.27)) (justify left))
+    )
+    (property "Value" "470p" (id 1) (at 165.1 129.5399 0)
       (effects (font (size 1.27 1.27)) (justify left))
     )
@@
   (symbol (lib_id "power:Earth") (at 95.885 102.235 0) (unit 1)
     (in_bom yes) (on_board yes) (fields_autoplaced)
-    (property "Reference" "#PWR?" (id 0) (at 95.885 108.585 0)
+    (property "Reference" "#PWR0111" (id 0) (at 95.885 108.585 0)
       (effects (font (size 1.27 1.27)) hide)
     )
@@
   (symbol (lib_id "power:Earth") (at 161.925 113.03 0) (unit 1)
     (in_bom yes) (on_board yes) (fields_autoplaced)
-    (property "Reference" "#PWR?" (id 0) (at 161.925 119.38 0)
+    (property "Reference" "#PWR0109" (id 0) (at 161.925 119.38 0)
       (effects (font (size 1.27 1.27)) hide)
     )
@@
   (symbol (lib_id "power:Earth") (at 161.925 91.44 0) (unit 1)
     (in_bom yes) (on_board yes) (fields_autoplaced)
-    (property "Reference" "#PWR?" (id 0) (at 161.925 97.79 0)
+    (property "Reference" "#PWR0113" (id 0) (at 161.925 97.79 0)
       (effects (font (size 1.27 1.27)) hide)
     )
@@
   (symbol (lib_id "power:Earth") (at 161.925 133.985 0) (unit 1)
     (in_bom yes) (on_board yes) (fields_autoplaced)
-    (property "Reference" "#PWR?" (id 0) (at 161.925 140.335 0)
+    (property "Reference" "#PWR0110" (id 0) (at 161.925 140.335 0)
       (effects (font (size 1.27 1.27)) hide)
     )
@@
   (symbol (lib_id "power:Earth") (at 59.055 100.33 0) (unit 1)
     (in_bom yes) (on_board yes) (fields_autoplaced)
-    (property "Reference" "#PWR?" (id 0) (at 59.055 106.68 0)
+    (property "Reference" "#PWR0112" (id 0) (at 59.055 106.68 0)
       (effects (font (size 1.27 1.27)) hide)
     )
@@
   (symbol (lib_id "Device:R_US") (at 153.67 80.645 90) (unit 1)
     (in_bom yes) (on_board yes) (fields_autoplaced)
-    (property "Reference" "R?" (id 0) (at 153.67 74.295 90))
-    (property "Value" "20k" (id 1) (at 153.67 76.835 90))
+    (property "Reference" "R608" (id 0) (at 153.67 74.93 90))
+    (property "Value" "20k" (id 1) (at 153.67 77.47 90))
     (property "Footprint" "Resistor_SMD:R_0805_2012Metric_Pad1.20x1.40mm_HandSolder" (id 2) (at 153.924 79.629 90)
       (effects (font (size 1.27 1.27)) hide)
@@
   (symbol (lib_id "Device:R_US") (at 153.67 102.235 90) (unit 1)
     (in_bom yes) (on_board yes) (fields_autoplaced)
-    (property "Reference" "R?" (id 0) (at 153.67 95.885 90))
-    (property "Value" "20k" (id 1) (at 153.67 98.425 90))
+    (property "Reference" "R610" (id 0) (at 153.67 96.52 90))
+    (property "Value" "20k" (id 1) (at 153.67 99.06 90))
     (property "Footprint" "Resistor_SMD:R_0805_2012Metric_Pad1.20x1.40mm_HandSolder" (id 2) (at 153.924 101.219 90)
       (effects (font (size 1.27 1.27)) hide)

Commit message: Place components of validation and quench trigger circuits on PCB
Connections:
- net at R601.1, RV601.2: now also RV601.1; no longer RV601.3
- net at C601.2, U602.15 (RCx): now also RV601.3; no longer RV601.1
Other:
- moved on the sheet: C604, C606, C615, R608, R610, R612, RV601, U603B, U603C, U603D

Commit message: Include ISO-A power circuit, all connectors and test points on PCB
Parts:
- added TP301: RCx, qds-cv-lib:TestPoint_Keystone_5010-5014_Multipurpose, symbol Connector:TestPoint
Connections:
- net TRIG-CH-A: now also SW601.5; no longer SW601.1
- net TRIG-CH-B: now also SW601.4; no longer SW601.2
- net TRIG-CH-D: now also SW601.2; no longer SW601.4
- net at R602.1: now also SW601.6; no longer SW601.10
- net at R603.1: now also SW601.7; no longer SW601.9
- net at C601.2, RV601.3, U602.15 (RCx): now also TP301.1
- net at R605.1: now also SW601.9; no longer SW601.7
Changed lines of the file:
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@@
   (junction (at 119.38 109.22) (diameter 0) (color 0 0 0 0)
+  )
+  (junction (at 46.99 43.815) (diameter 0) (color 0 0 0 0)
   )
   (junction (at 95.885 100.33) (diameter 0) (color 0 0 0 0)
@@
     (pin "7")
   )
-  (symbol (lib_id "Switch:SW_DIP_x05") (at 232.41 54.61 0) (unit 1)
+  (symbol (lib_id "Switch:SW_DIP_x05") (at 232.41 54.61 0) (mirror x) (unit 1)
     (in_bom yes) (on_board yes) (fields_autoplaced)
     (property "Reference" "SW601" (id 0) (at 232.41 41.91 0))
@@
       (effects (font (size 1.27 1.27)) hide)
     )
+    (pin "1")
+  )
+  (symbol (lib_id "Connector:TestPoint") (at 46.99 43.815 90) (unit 1)
+    (in_bom yes) (on_board yes)
+    (property "Reference" "TP301" (id 0) (at 39.37 43.815 90))
+    (property "Value" "RCx" (id 1) (at 43.688 40.005 90)
+      (effects (font (size 1.27 1.27)) hide)
+    )
+    (property "Footprint" "qds-cv-lib:TestPoint_Keystone_5010-5014_Multipurpose" (id 2) (at 46.99 38.735 0)
+      (effects (font (size 1.27 1.27)) hide)
+    )
+    (property "Datasheet" "https://www.keyelco.com/product-pdf.cfm?p=1321" (id 3) (at 46.99 38.735 0)
+      (effects (font (size 1.27 1.27)) hide)
+    )

Commit message: Remake some logic connections and update PCB
Changed lines of the file:
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@@
     (effects (font (size 1.27 1.27)) (justify left bottom))
   )
-  (label "TRIG-CH-B" (at 212.217 52.07 0)
+  (label "TRIG-CH-B" (at 212.09 52.07 0)
     (effects (font (size 1.27 1.27)) (justify left bottom))
   )
@@
     (effects (font (size 1.27 1.27)) (justify left bottom))
   )
-  (label "TRIG-CH-A" (at 212.217 49.53 0)
+  (label "TRIG-CH-A" (at 212.09 49.53 0)
     (effects (font (size 1.27 1.27)) (justify left bottom))
   )

Commit message: Last commit before flipping PTH components
Connections:
- net TRIG-CH-D: now also SW601.1
Changed lines of the file:
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@@
   (junction (at 58.42 53.975) (diameter 0) (color 0 0 0 0)
+  )
+  (junction (at 224.79 57.15) (diameter 0) (color 0 0 0 0)
   )
   (junction (at 256.54 40.005) (diameter 0) (color 0 0 0 0)
@@
     (stroke (width 0) (type default) (color 0 0 0 0))
   )
+  (wire (pts (xy 224.79 57.15) (xy 224.79 59.69))
+    (stroke (width 0) (type default) (color 0 0 0 0))
+  )

Commit message: Update PCB layout
Parts:
- R601: value 1k -> 4.7k; CNPEM Code AP110784 -> (none); Manufacturer Panasonic Electronic Components -> (none); Part Number ERJ-6GEYJ102V -> 0805W8F1200T5E
Changed lines of the file:
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@@
     (in_bom yes) (on_board yes)
     (property "Reference" "R601" (id 0) (at 33.02 31.115 90))
-    (property "Value" "1k" (id 1) (at 33.02 33.655 90))
+    (property "Value" "4.7k" (id 1) (at 33.02 33.655 90))
     (property "Footprint" "Resistor_SMD:R_0805_2012Metric_Pad1.20x1.40mm_HandSolder" (id 2) (at 32.766 38.481 90)
       (effects (font (size 1.27 1.27)) hide)
     )
-    (property "Datasheet" "https://industrial.panasonic.com/cdbs/www-data/pdf/RDA0000/AOA0000C301.pdf" (id 3) (at 33.02 37.465 0)
+    (property "Datasheet" "https://datasheet.lcsc.com/lcsc/2206010216_UNI-ROYAL-Uniroyal-Elec-0805W8F1002T5E_C17414.pdf" (id 3) (at 33.02 37.465 0)
       (effects (font (size 1.27 1.27)) hide)
     )
-    (property "Part Number" "ERJ-6GEYJ102V" (id 4) (at 33.02 37.465 0)
+    (property "Part Number" "0805W8F1200T5E" (id 4) (at 33.02 37.465 0)
       (effects (font (size 1.27 1.27)) hide)
     )
-    (property "CNPEM Code" "AP110784" (id 5) (at 33.02 37.465 0)
+    (property "CNPEM Code" "" (id 5) (at 33.02 37.465 0)
       (effects (font (size 1.27 1.27)) hide)
     )
-    (property "Manufacturer" "Panasonic Electronic Components" (id 6) (at 33.02 37.465 0)
+    (property "Manufacturer" "" (id 6) (at 33.02 37.465 0)
       (effects (font (size 1.27 1.27)) hide)
     )
+    (property "Description" "Resistor 4k7 1% 0.125W SMD 0805" (id 7) (at 33.02 37.465 0)
+      (effects (font (size 1.27 1.27)) hide)
+    )
