File: pcb/cad/detection-validation.kicad_sch (KiCad schematic)
At the start: 39 parts, among them SW601 SW_DIP_x04, U601 74HC32D, U602 74HC123, U603 74HCS08, U604 74HC32D, U605 74HC123

Commit message: Reposition of channels and connectors, place and route trigger and actuation circuit
Connections:
- net TRIG-CH-A: now also SW601.8; no longer SW601.1
- net TRIG-CH-B: now also SW601.7; no longer SW601.2
- net TRIG-CH-C: now also SW601.6; no longer SW601.3
- net TRIG-CH-D: now also SW601.5; no longer SW601.4
- net VAL-A: now also U601.13; no longer U601.5
- net VAL-B: now also U601.5; no longer U601.13
- net VAL-C: now also U604.13; no longer U604.5
- net VAL-D: now also U604.5; no longer U604.13
- net at R602.1: now also SW601.1; no longer SW601.8
- net at U601.1: now also U602.12 (~{Q}); no longer U602.4 (~{Q})
- net at U601.2, U601.4: now also U602.5 (Q); no longer U602.13 (Q)
- net at U601.3: now also U603.12; no longer U603.4
- net at R612.1: now also U603.6; no longer U603.8
- net at U605.12 (~{Q}): now also U604.1; no longer U604.9
- net at U604.10, U604.12: now also U605.13 (Q); no longer U605.5 (Q)
- net at R603.1: now also SW601.2; no longer SW601.7
- net at U601.6: now also U603.13; no longer U603.5
- net at R608.1: now also U603.11; no longer U603.3
- net at R606.1: now also U603.8; no longer U603.6
- net at U601.10, U601.12: now also U602.13 (Q); no longer U602.5 (Q)
- net at U601.8: now also U603.9; no longer U603.1
- net at U601.9: now also U602.4 (~{Q}); no longer U602.12 (~{Q})
- net at U603.2: now also U604.11; no longer U601.11
- net at U603.10: now also U601.11; no longer U604.11
- net at R605.1: now also SW601.4; no longer SW601.5
- net at R604.1: now also SW601.3; no longer SW601.6
- net at U604.2, U604.4: now also U605.5 (Q); no longer U605.13 (Q)
- net at U605.4 (~{Q}): now also U604.9; no longer U604.1
- net at U604.8: now also U603.1; no longer U603.9
- net at U604.6: now also U603.5; no longer U603.13
- net at R610.1: now also U603.3; no longer U603.11
- net at U604.3: now also U603.4; no longer U603.12
Other:
- moved on the sheet: U601A, U601B, U601C, U601D, U603A, U603B, U603C, U603D, U604A, U604B, U604C, U604D

Commit message: Replicate detection layout for all channels, place and route 5V-REF circuit
Connections:
- net at C605.2, U605.15 (RCx): now also RV603.3; no longer RV603.2
- net at R601.1: now also RV601.2; no longer RV601.3
- net at C601.2, U602.15 (RCx): now also RV601.3; no longer RV601.2
- net at R609.1: now also RV603.2; no longer RV603.3
- net at C603.2, U602.7 (RCx): now also RV602.3; no longer RV602.2
- net at R607.1: now also RV602.2; no longer RV602.3
Other:
- moved on the sheet: RV601, RV602, RV603

Commit message: Create +14V, -14V, +5V copper zones
Connections:
- net at C612.2, U605.7 (RCx): now also RV604.3; no longer RV604.2
- net at R611.1: now also RV604.2; no longer RV604.3
Other:
- moved on the sheet: RV604
Changed lines of the file:
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@@
   (junction (at 58.42 180.34) (diameter 0) (color 0 0 0 0)
   )
-  (junction (at 46.99 167.64) (diameter 0) (color 0 0 0 0)
-  )
   (junction (at 92.71 170.18) (diameter 0) (color 0 0 0 0)
   )
@@
   (junction (at 242.57 121.92) (diameter 0) (color 0 0 0 0)
   )
+  (junction (at 46.99 163.83) (diameter 0) (color 0 0 0 0)
+  )
   (junction (at 46.355 92.71) (diameter 0) (color 0 0 0 0)
   )
@@
     (stroke (width 0) (type default) (color 0 0 0 0))
   )
-  (wire (pts (xy 41.91 167.64) (xy 46.99 167.64))
-    (stroke (width 0) (type default) (color 0 0 0 0))
-  )
   (wire (pts (xy 37.465 41.275) (xy 37.465 37.465))
     (stroke (width 0) (type default) (color 0 0 0 0))
@@
     (stroke (width 0) (type default) (color 0 0 0 0))
   )
+  (wire (pts (xy 36.83 167.64) (xy 36.83 163.83))
+    (stroke (width 0) (type default) (color 0 0 0 0))
+  )
   (wire (pts (xy 205.105 154.94) (xy 205.105 157.48))
     (stroke (width 0) (type default) (color 0 0 0 0))
@@
     (stroke (width 0) (type default) (color 0 0 0 0))
   )
-  (wire (pts (xy 46.99 167.64) (xy 46.99 163.83))
+  (wire (pts (xy 46.99 163.83) (xy 46.99 170.18))
     (stroke (width 0) (type default) (color 0 0 0 0))
   )
@@
     (stroke (width 0) (type default) (color 0 0 0 0))
   )
+  (wire (pts (xy 43.18 167.64) (xy 36.83 167.64))
+    (stroke (width 0) (type default) (color 0 0 0 0))
+  )
   (wire (pts (xy 114.3 51.435) (xy 114.3 56.515))
     (stroke (width 0) (type default) (color 0 0 0 0))
@@
     (stroke (width 0) (type default) (color 0 0 0 0))
   )
-  (wire (pts (xy 46.99 170.18) (xy 46.99 167.64))
-    (stroke (width 0) (type default) (color 0 0 0 0))
-  )
   (wire (pts (xy 48.26 163.83) (xy 46.99 163.83))
     (stroke (width 0) (type default) (color 0 0 0 0))
@@
   )
   (wire (pts (xy 93.345 85.09) (xy 93.345 95.25))
-    (stroke (width 0) (type default) (color 0 0 0 0))
-  )
-  (wire (pts (xy 36.83 163.83) (xy 38.1 163.83))
     (stroke (width 0) (type default) (color 0 0 0 0))
   )
@@
     (pin "8")
   )
-  (symbol (lib_name "R_Potentiometer_Trim_US_1") (lib_id "Device:R_Potentiometer_Trim_US") (at 41.91 163.83 270) (unit 1)
+  (symbol (lib_name "R_Potentiometer_Trim_US_1") (lib_id "Device:R_Potentiometer_Trim_US") (at 43.18 163.83 90) (mirror x) (unit 1)
     (in_bom yes) (on_board yes) (fields_autoplaced)
-    (property "Reference" "RV604" (id 0) (at 41.91 157.48 90))
-    (property "Value" "50k" (id 1) (at 41.91 160.02 90))
-    (property "Footprint" "qds-cv-lib:Potentiometer_Bourns_3224X_Vertical" (id 2) (at 41.91 163.83 0)
-      (effects (font (size 1.27 1.27)) hide)
-    )
-    (property "Datasheet" "https://www.bourns.com/docs/Product-Datasheets/3224.pdf" (id 3) (at 41.91 163.83 0)
-      (effects (font (size 1.27 1.27)) hide)
-    )
-    (property "Manufacturer" "Bourns" (id 4) (at 41.91 163.83 0)
-      (effects (font (size 1.27 1.27)) hide)
-    )
-    (property "Part Number" "3224X-1-503E" (id 5) (at 41.91 163.83 0)
-      (effects (font (size 1.27 1.27)) hide)
-    )
-    (property "Description" "Trimpot 50k, 12 turns, 10% tolerance, 4mm SMD Top Adjust" (id 6) (at 41.91 163.83 0)
-      (effects (font (size 1.27 1.27)) hide)
-    )
-    (property "Vendor Link" "https://br.mouser.com/ProductDetail/Bourns/3224X-1-503E?qs=A%2FVUe%2FMZWjw7UCYo8RtHVg%3D%3D" (id 7) (at 41.91 163.83 0)
-      (effects (font (size 1.27 1.27)) hide)
-    )
+    (property "Reference" "RV604" (id 0) (at 43.18 157.48 90))
+    (property "Value" "50k" (id 1) (at 43.18 160.02 90))
+    (property "Footprint" "qds-cv-lib:Potentiometer_Bourns_3224X_Vertical" (id 2) (at 43.18 163.83 0)
+      (effects (font (size 1.27 1.27)) hide)
+    )
+    (property "Datasheet" "https://www.bourns.com/docs/Product-Datasheets/3224.pdf" (id 3) (at 43.18 163.83 0)
+      (effects (font (size 1.27 1.27)) hide)
+    )
+    (property "Manufacturer" "Bourns" (id 4) (at 43.18 163.83 0)
+      (effects (font (size 1.27 1.27)) hide)
+    )
+    (property "Part Number" "3224X-1-503E" (id 5) (at 43.18 163.83 0)
+      (effects (font (size 1.27 1.27)) hide)
+    )
+    (property "Description" "Trimpot 50k, 12 turns, 10% tolerance, 4mm SMD Top Adjust" (id 6) (at 43.18 163.83 0)
+      (effects (font (size 1.27 1.27)) hide)
+    )
+    (property "Vendor Link" "https://br.mouser.com/ProductDetail/Bourns/3224X-1-503E?qs=A%2FVUe%2FMZWjw7UCYo8RtHVg%3D%3D" (id 7) (at 43.18 163.83 0)
+      (effects (font (size 1.27 1.27)) hide)
+    )

Commit message: Apply several changes based on test results - replace validation time 4k7 resistor by a 8k2, close #21 - remove pull-up resistor from AMC1200 positive input - split voltage taps pull-up/down resistors into 2 footprints each - change C204,304,404,504 footprints from 0603 to 0805 - include bypass switch for software trigger - remove test points from voltage taps - change window comparator input resistor to 4k7 - include footprint for a 0805 capacitor at the window comparator input
Parts:
- R601, R607, R609, R611: value 4.7k -> 8.2k; Part Number 0805W8F1200T5E -> 0805W8F8201T5E
Changed lines of the file:
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@@
     (in_bom yes) (on_board yes)
     (property "Reference" "R601" (id 0) (at 33.02 31.115 90))
-    (property "Value" "4.7k" (id 1) (at 33.02 33.655 90))
+    (property "Value" "8.2k" (id 1) (at 33.02 33.655 90))
     (property "Footprint" "Resistor_SMD:R_0805_2012Metric_Pad1.20x1.40mm_HandSolder" (id 2) (at 32.766 38.481 90)
       (effects (font (size 1.27 1.27)) hide)
@@
       (effects (font (size 1.27 1.27)) hide)
     )
-    (property "Part Number" "0805W8F1200T5E" (id 4) (at 33.02 37.465 0)
+    (property "Part Number" "0805W8F8201T5E" (id 4) (at 33.02 37.465 0)
       (effects (font (size 1.27 1.27)) hide)
     )
@@
       (effects (font (size 1.27 1.27)) hide)
     )
-    (property "Description" "Resistor 4k7 1% 0.125W SMD 0805" (id 7) (at 33.02 37.465 0)
+    (property "Description" "Resistor 8k2 1% 0.125W SMD 0805" (id 7) (at 33.02 37.465 0)
       (effects (font (size 1.27 1.27)) hide)
     )
@@
     (in_bom yes) (on_board yes)
     (property "Reference" "R611" (id 0) (at 33.02 157.48 90))
-    (property "Value" "4.7k" (id 1) (at 33.02 160.02 90))
+    (property "Value" "8.2k" (id 1) (at 33.02 160.02 90))
     (property "Footprint" "Resistor_SMD:R_0805_2012Metric_Pad1.20x1.40mm_HandSolder" (id 2) (at 32.766 164.846 90)
       (effects (font (size 1.27 1.27)) hide)
@@
       (effects (font (size 1.27 1.27)) hide)
     )
-    (property "Part Number" "0805W8F1200T5E" (id 4) (at 33.02 163.83 0)
+    (property "Part Number" "0805W8F8201T5E" (id 4) (at 33.02 163.83 0)
       (effects (font (size 1.27 1.27)) hide)
     )
@@
       (effects (font (size 1.27 1.27)) hide)
     )
-    (property "Description" "Resistor 4k7 1% 0.125W SMD 0805" (id 7) (at 33.02 163.83 0)
+    (property "Description" "Resistor 8k2 1% 0.125W SMD 0805" (id 7) (at 33.02 163.83 0)
       (effects (font (size 1.27 1.27)) hide)
     )
@@
     (in_bom yes) (on_board yes)
     (property "Reference" "R609" (id 0) (at 33.02 114.3 90))
-    (property "Value" "4.7k" (id 1) (at 33.02 116.84 90))
+    (property "Value" "8.2k" (id 1) (at 33.02 116.84 90))
     (property "Footprint" "Resistor_SMD:R_0805_2012Metric_Pad1.20x1.40mm_HandSolder" (id 2) (at 32.766 121.666 90)
       (effects (font (size 1.27 1.27)) hide)
@@
       (effects (font (size 1.27 1.27)) hide)
     )
-    (property "Part Number" "0805W8F1200T5E" (id 4) (at 33.02 120.65 0)
-      (effects (font (size 1.27 1.27)) hide)
-    )
-    (property "CNPEM Code" "" (id 5) (at 33.02 120.65 0)
+    (property "Part Number" "0805W8F8201T5E" (id 4) (at 33.02 120.65 0)
       (effects (font (size 1.27 1.27)) hide)
     )
@@
       (effects (font (size 1.27 1.27)) hide)
     )
-    (property "Description" "Resistor 4k7 1% 0.125W SMD 0805" (id 7) (at 33.02 120.65 0)
+    (property "Description" "Resistor 8k2 1% 0.125W SMD 0805" (id 7) (at 33.02 120.65 0)
       (effects (font (size 1.27 1.27)) hide)
     )
@@
     (in_bom yes) (on_board yes)
     (property "Reference" "R607" (id 0) (at 33.655 72.39 90))
-    (property "Value" "4.7k" (id 1) (at 33.655 74.93 90))
+    (property "Value" "8.2k" (id 1) (at 33.655 74.93 90))
     (property "Footprint" "Resistor_SMD:R_0805_2012Metric_Pad1.20x1.40mm_HandSolder" (id 2) (at 33.401 79.756 90)
       (effects (font (size 1.27 1.27)) hide)
@@
       (effects (font (size 1.27 1.27)) hide)
     )
-    (property "Part Number" "0805W8F1200T5E" (id 4) (at 33.655 78.74 0)
+    (property "Part Number" "0805W8F8201T5E" (id 4) (at 33.655 78.74 0)
       (effects (font (size 1.27 1.27)) hide)
     )
@@
       (effects (font (size 1.27 1.27)) hide)
     )
-    (property "Description" "Resistor 4k7 1% 0.125W SMD 0805" (id 7) (at 33.655 78.74 0)
-      (effects (font (size 1.27 1.27)) hide)
-    )
+    (property "Description" "Resistor 8k2 1% 0.125W SMD 0805" (id 7) (at 33.655 78.74 0)
+      (effects (font (size 1.27 1.27)) hide)
+    )

Commit message: Replace protection flip-flop with latch, update components description generate HTML BOM list.
Parts:
- R606, R608, R610, R612: Part Number RC-05K203IT -> RC-05K203JT
Changed lines of the file:
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@@
+      (effects (font (size 1.27 1.27)) hide)
+    )
+    (property "Description" " Dual Retriggerable Monostable Multivibrators with Resets" (id 7) (at 254 134.62 0)
       (effects (font (size 1.27 1.27)) hide)
     )
@@
       (effects (font (size 1.27 1.27)) hide)
     )
+    (property "Description" "Quad 2-input OR gates" (id 7) (at 103.505 87.63 0)
+      (effects (font (size 1.27 1.27)) hide)
+    )
     (pin "1")
     (pin "2")
@@
       (effects (font (size 1.27 1.27)) hide)
     )
-    (property "Part Number" "RC-05K203IT" (id 4) (at 143.51 175.26 0)
+    (property "Part Number" "RC-05K203JT" (id 4) (at 143.51 175.26 0)
+      (effects (font (size 1.27 1.27)) hide)
+    )
+    (property "Description" "Resistor 20k 5% 0.1W SMD 0805" (id 5) (at 139.7 175.26 0)
       (effects (font (size 1.27 1.27)) hide)
     )
@@
     )
     (property "Manufacturer" "NXP" (id 6) (at 217.805 134.62 0)
+      (effects (font (size 1.27 1.27)) hide)
+    )
+    (property "Description" "Quad 2-input OR gates" (id 7) (at 217.805 134.62 0)
       (effects (font (size 1.27 1.27)) hide)
     )
@@
       (effects (font (size 1.27 1.27)) hide)
     )
+    (property "Description" " Dual Retriggerable Monostable Multivibrators with Resets" (id 7) (at 71.12 175.26 0)
+      (effects (font (size 1.27 1.27)) hide)
+    )
     (pin "1")
     (pin "13")
@@
       (effects (font (size 1.27 1.27)) hide)
     )
+    (property "Description" "Quad 2-input OR gates" (id 7) (at 103.505 97.79 0)
+      (effects (font (size 1.27 1.27)) hide)
+    )
     (pin "1")
     (pin "2")
@@
     )
     (property "Manufacturer" "NXP" (id 6) (at 229.235 134.62 0)
+      (effects (font (size 1.27 1.27)) hide)
+    )
+    (property "Description" "Quad 2-input OR gates" (id 7) (at 229.235 134.62 0)
       (effects (font (size 1.27 1.27)) hide)
     )
@@
       (effects (font (size 1.27 1.27)) hide)
     )
-    (property "Part Number" "RC-05K203IT" (id 4) (at 143.51 90.17 0)
+    (property "Part Number" "RC-05K203JT" (id 4) (at 143.51 90.17 0)
+      (effects (font (size 1.27 1.27)) hide)
+    )
+    (property "Description" "Resistor 20k 5% 0.1W SMD 0805" (id 5) (at 139.7 90.17 0)
       (effects (font (size 1.27 1.27)) hide)
     )
@@
       (effects (font (size 1.27 1.27)) hide)
     )
-    (property "Part Number" "RC-05K203IT" (id 4) (at 143.51 48.895 0)
+    (property "Part Number" "RC-05K203JT" (id 4) (at 143.51 48.895 0)
+      (effects (font (size 1.27 1.27)) hide)
+    )
+    (property "Description" "Resistor 20k 5% 0.1W SMD 0805" (id 5) (at 139.7 48.895 0)
       (effects (font (size 1.27 1.27)) hide)
     )
@@
       (effects (font (size 1.27 1.27)) hide)
     )
+    (property "Description" " Dual Retriggerable Monostable Multivibrators with Resets" (id 7) (at 71.12 48.895 0)
+      (effects (font (size 1.27 1.27)) hide)
+    )
     (pin "1")
     (pin "13")
@@
       (effects (font (size 1.27 1.27)) hide)
     )
+    (property "Description" "Quad 2-input OR gates" (id 7) (at 102.87 46.355 0)
+      (effects (font (size 1.27 1.27)) hide)
+    )
     (pin "1")
     (pin "2")
@@
       (effects (font (size 1.27 1.27)) hide)
     )
+    (property "Description" "Quad 2-Input AND Gates with Schmitt-Trigger Inputs" (id 7) (at 124.46 132.08 0)
+      (effects (font (size 1.27 1.27)) hide)
+    )
     (pin "1")
     (pin "2")
@@
       (effects (font (size 1.27 1.27)) hide)
     )
+    (property "Description" "Quad 2-input OR gates" (id 7) (at 102.87 139.7 0)
+      (effects (font (size 1.27 1.27)) hide)
+    )
     (pin "1")
     (pin "2")
@@
       (effects (font (size 1.27 1.27)) hide)
     )
+    (property "Description" "Switch slide DIP 4xSPST 25mA 24V" (id 6) (at 232.41 54.61 0)
+      (effects (font (size 1.27 1.27)) hide)
+    )
     (pin "1")
     (pin "2")
@@
     )
     (property "Part Number" "CD74HC123" (id 6) (at 242.57 134.62 0)
+      (effects (font (size 1.27 1.27)) hide)
+    )
+    (property "Description" " Dual Retriggerable Monostable Multivibrators with Resets" (id 7) (at 242.57 134.62 0)
       (effects (font (size 1.27 1.27)) hide)
     )
@@
       (effects (font (size 1.27 1.27)) hide)
     )
+    (property "Description" " Dual Retriggerable Monostable Multivibrators with Resets" (id 7) (at 71.12 132.08 0)
+      (effects (font (size 1.27 1.27)) hide)
+    )
     (pin "1")
     (pin "13")
@@
       (effects (font (size 1.27 1.27)) hide)
     )
+    (property "Description" "Quad 2-input OR gates" (id 7) (at 102.87 129.54 0)
+      (effects (font (size 1.27 1.27)) hide)
+    )
     (pin "1")
     (pin "2")
@@
       (effects (font (size 1.27 1.27)) hide)
     )
+    (property "Description" "Quad 2-Input AND Gates with Schmitt-Trigger Inputs" (id 7) (at 124.46 48.895 0)
+      (effects (font (size 1.27 1.27)) hide)
+    )
     (pin "1")
     (pin "2")
@@
       (effects (font (size 1.27 1.27)) hide)
     )
+    (property "Description" "Quad 2-input OR gates" (id 7) (at 102.87 182.88 0)
+      (effects (font (size 1.27 1.27)) hide)
+    )
     (pin "1")
     (pin "2")
@@
       (effects (font (size 1.27 1.27)) hide)
     )
+    (property "Description" "Quad 2-input OR gates" (id 7) (at 102.87 56.515 0)
+      (effects (font (size 1.27 1.27)) hide)
+    )
     (pin "1")
     (pin "2")
@@
       (effects (font (size 1.27 1.27)) hide)
     )
+    (property "Description" "Quad 2-Input AND Gates with Schmitt-Trigger Inputs" (id 7) (at 124.46 175.26 0)
+      (effects (font (size 1.27 1.27)) hide)
+    )
     (pin "1")
     (pin "2")
@@
       (effects (font (size 1.27 1.27)) hide)
     )
+    (property "Description" " Dual Retriggerable Monostable Multivibrators with Resets" (id 7) (at 71.755 90.17 0)
+      (effects (font (size 1.27 1.27)) hide)
+    )
     (pin "1")
     (pin "13")
@@
       (effects (font (size 1.27 1.27)) hide)
     )
+    (property "Description" "Quad 2-Input AND Gates with Schmitt-Trigger Inputs" (id 7) (at 125.095 90.17 0)
+      (effects (font (size 1.27 1.27)) hide)
+    )
     (pin "1")
     (pin "2")
@@
     )
     (property "Manufacturer" "Texas Instruments" (id 6) (at 205.105 134.62 0)
+      (effects (font (size 1.27 1.27)) hide)
+    )
+    (property "Description" "Quad 2-Input AND Gates with Schmitt-Trigger Inputs" (id 7) (at 205.105 134.62 0)
       (effects (font (size 1.27 1.27)) hide)
     )
@@
       (effects (font (size 1.27 1.27)) hide)
     )
-    (property "Part Number" "RC-05K203IT" (id 4) (at 143.51 132.08 0)
+    (property "Part Number" "RC-05K203JT" (id 4) (at 143.51 132.08 0)
+      (effects (font (size 1.27 1.27)) hide)
+    )
+    (property "Description" "Resistor 20k 5% 0.1W SMD 0805" (id 5) (at 139.7 132.08 0)
       (effects (font (size 1.27 1.27)) hide)
     )
@@
       (effects (font (size 1.27 1.27)) hide)
     )
+    (property "Description" "Quad 2-input OR gates" (id 7) (at 102.87 172.72 0)
+      (effects (font (size 1.27 1.27)) hide)
+    )
