File: pcb/cad/qds-cv.kicad_sch (KiCad schematic)
At the start: 1 part

Commit message: Created hierarchy connections, updates on analog-front-end and included 5V reference circuit
Connections:
- net VT4: now reaches J?.12
- net VT4: now also J?.24 (P24)
- net VT1: now reaches J?.15 (P15)
- net VT1: now also J?.2
- net VT2: now reaches J?.18 (P18)
- net VT2: now also J?.5
- net VT3: now reaches J?.21 (P21)
- net VT3: now also J?.9
Other:
- sheet Analog front-end renamed Isolated detection channel A
- sheet Detection & validation renamed Detection validation
- added sheet +5V reference (5v-reference.kicad_sch)
- sheet Detection validation ports: added TRIG-CH-A, TRIG-CH-B, TRIG-CH-C, TRIG-CH-D, VAL-A, VAL-B, VAL-C, VAL-D; removed TRIG, V-DET
- moved on the sheet: J?

Commit message: Update componentes fields and reference circuit
Parts:
- J?: value DB25_Male_MountingHoles -> DB25 Female; Manufacturer (none) -> Amphenol FCI
Other:
- added sheet Isolated detection channel B (analog-front-end.kicad_sch)
- added sheet Isolated detection channel C (analog-front-end.kicad_sch)
- added sheet Isolated detection channel D (analog-front-end.kicad_sch)
- sheet +5V reference ports: added +5VREF; removed none
- note added: "Quench detection system for vertical cryostat"

Commit message: Update power supplies, symbols and footprint libs
Parts:
- gave numbers to parts that had none: 1

Commit message: Make modifications needed for single channel board
Parts:
- removed J101: DB25 Female, Connector_Dsub:DSUB-25_Female_Horizontal_P2.77x2.84mm_EdgePinOffset7.70mm_Housed_MountingHolesOffset9.12mm, symbol Connector:DB25_Female_MountingHoles
- added J?: Conn_01x08, symbol Connector_Generic:Conn_01x08
- added TP? (x6): TestPoint, symbol Connector:TestPoint
Connections:
- net Detection validation/TRIG-CH-A: now also TP?.1
- net Detection validation/TRIG-CH-B: now also TP?.1
- net Detection validation/TRIG-CH-C: now also TP?.1
- net Detection validation/TRIG-CH-D: now also TP?.1
- net Earth: now also J?.4 (Pin_4)
- net VT1: now also TP?.1
- net VT2: now also TP?.1
- new net +14V: J?.1 (Pin_1)
- new net +5V: J?.3 (Pin_3)
- new net +5V-ISO-A: J?.5 (Pin_5)
- new net -14V: J?.2 (Pin_2)
- new net GND-ISO-A: J?.6 (Pin_6)
Other:
- removed sheet Isolated detection channel B
- removed sheet Isolated detection channel C
- removed sheet Isolated detection channel D
