File: pcb/cad/qds-cv.kicad_sch (KiCad schematic)
At the start: 7 parts

Commit message: Add test points and extra resistors for temporary use. Remove power supplies
Parts:
- gave numbers to parts that had none: 7
Other:
- removed sheet Power supplies

Commit message: Include ISO-A power circuit, all connectors and test points on PCB
Parts:
- added J101: DB25 Female, Connector_Dsub:DSUB-25_Female_Horizontal_P2.77x2.84mm_EdgePinOffset7.70mm_Housed_MountingHolesOffset9.12mm, symbol Connector:DB25_Female_MountingHoles
- added J301, J401, J501: Conn_Coaxial, qds-cv-lib:Molex_0731375003, symbol Connector:Conn_Coaxial
- added TP107, TP108, TP109, TP110, TP111, TP112, TP113, TP114, TP115, TP116, TP117, TP118, TP119: TestPoint, qds-cv-lib:TestPoint_Keystone_5010-5014_Multipurpose, symbol Connector:TestPoint
- J102: footprint (none) -> Connector_Phoenix_MC:PhoenixContact_MCV_1,5_6-GF-3.81_1x06_P3.81mm_Vertical_ThreadedFlange; symbol Connector_Generic:Conn_01x08 -> Connector_Generic:Conn_01x06
- TP101: value TestPoint -> VT1; footprint (none) -> qds-cv-lib:TestPoint_Keystone_5010-5014_Multipurpose
- TP102: value TestPoint -> VT2; footprint (none) -> qds-cv-lib:TestPoint_Keystone_5010-5014_Multipurpose
- TP103, TP104, TP105, TP106: footprint (none) -> qds-cv-lib:TestPoint_Keystone_5010-5014_Multipurpose
Connections:
- net +14V: now also TP107.1
- net +5V: now also TP109.1
- net +5V-ISO-A: now also TP111.1; no longer J102.5 (Pin_5)
- net -14V: now also TP108.1
- net Earth: now also J101.0 (PAD), TP116.1, TP117.1, TP118.1, TP119.1
- net GND-ISO-A: now also TP112.1, TP113.1, TP114.1, TP115.1; no longer J102.6 (Pin_6)
- net VT1: now also J101.12, J101.24 (P24)
- net VT2: now also J101.21 (P21), J101.9
- net VT3: now also J101.18 (P18), J101.5
- net VT4: now also J101.15 (P15), J101.2
- new net +15V: J102.5 (Pin_5), TP110.1
Other:
- added sheet Power supplies (power-supplies.kicad_sch)

Commit message: Last commit before flipping PTH components
Connections:
- net +15V: now also J102.6 (Pin_6); no longer J102.5 (Pin_5)
- net Earth: now also J102.5 (Pin_5)
Changed lines of the file:
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@@
   (junction (at 177.165 109.22) (diameter 0) (color 0 0 0 0)
   )
-  (junction (at 173.355 62.865) (diameter 0) (color 0 0 0 0)
+  (junction (at 173.355 65.405) (diameter 0) (color 0 0 0 0)
   )
   (junction (at 114.3 153.67) (diameter 0) (color 0 0 0 0)
@@
     (stroke (width 0) (type default) (color 0 0 0 0))
   )
-  (wire (pts (xy 173.355 48.26) (xy 173.355 62.865))
-    (stroke (width 0) (type default) (color 0 0 0 0))
-  )
   (wire (pts (xy 62.23 96.52) (xy 72.39 96.52))
     (stroke (width 0) (type default) (color 0 0 0 0))
@@
     (stroke (width 0) (type default) (color 0 0 0 0))
   )
+  (wire (pts (xy 173.355 48.26) (xy 173.355 65.405))
+    (stroke (width 0) (type default) (color 0 0 0 0))
+  )
   (wire (pts (xy 61.595 49.53) (xy 72.39 49.53))
     (stroke (width 0) (type default) (color 0 0 0 0))
@@
     (stroke (width 0) (type default) (color 0 0 0 0))
   )
+  (wire (pts (xy 161.925 62.865) (xy 178.435 62.865))
+    (stroke (width 0) (type default) (color 0 0 0 0))
+  )
   (wire (pts (xy 54.61 90.17) (xy 72.39 90.17))
     (stroke (width 0) (type default) (color 0 0 0 0))
@@
     (stroke (width 0) (type default) (color 0 0 0 0))
   )
-  (wire (pts (xy 161.925 62.865) (xy 173.355 62.865))
+  (wire (pts (xy 161.925 65.405) (xy 173.355 65.405))
     (stroke (width 0) (type default) (color 0 0 0 0))
   )
@@
     (stroke (width 0) (type default) (color 0 0 0 0))
   )
-  (wire (pts (xy 173.355 62.865) (xy 178.435 62.865))
+  (wire (pts (xy 173.355 65.405) (xy 178.435 65.405))
     (stroke (width 0) (type default) (color 0 0 0 0))
   )
@@
     (pin "1")
   )
+  (symbol (lib_id "power:Earth") (at 178.435 62.865 90) (unit 1)
+    (in_bom yes) (on_board yes) (fields_autoplaced)
+    (property "Reference" "#PWR0117" (id 0) (at 184.785 62.865 0)
+      (effects (font (size 1.27 1.27)) hide)
+    )
+    (property "Value" "Earth" (id 1) (at 182.245 62.865 0)
+      (effects (font (size 1.27 1.27)) hide)
+    )
+    (property "Footprint" "" (id 2) (at 178.435 62.865 0)
+      (effects (font (size 1.27 1.27)) hide)
+    )
+    (property "Datasheet" "~" (id 3) (at 178.435 62.865 0)
+      (effects (font (size 1.27 1.27)) hide)
+    )
+    (pin "1")
+  )
   (symbol (lib_id "Connector:TestPoint") (at 177.165 109.22 0) (unit 1)
     (in_bom yes) (on_board yes)
@@
     (pin "1")
   )
-  (symbol (lib_id "power:+15V") (at 178.435 62.865 270) (unit 1)
-    (in_bom yes) (on_board yes) (fields_autoplaced)
-    (property "Reference" "#PWR0106" (id 0) (at 174.625 62.865 0)
-      (effects (font (size 1.27 1.27)) hide)
-    )
-    (property "Value" "+15V" (id 1) (at 182.245 62.8649 90)
-      (effects (font (size 1.27 1.27)) (justify left))
-    )
-    (property "Footprint" "" (id 2) (at 178.435 62.865 0)
-      (effects (font (size 1.27 1.27)) hide)
-    )
-    (property "Datasheet" "" (id 3) (at 178.435 62.865 0)
+  (symbol (lib_id "power:+15V") (at 178.435 65.405 270) (unit 1)
+    (in_bom yes) (on_board yes) (fields_autoplaced)
+    (property "Reference" "#PWR0106" (id 0) (at 174.625 65.405 0)
+      (effects (font (size 1.27 1.27)) hide)
+    )
+    (property "Value" "+15V" (id 1) (at 182.245 65.4049 90)
+      (effects (font (size 1.27 1.27)) (justify left))
+    )
+    (property "Footprint" "" (id 2) (at 178.435 65.405 0)
+      (effects (font (size 1.27 1.27)) hide)
+    )
+    (property "Datasheet" "" (id 3) (at 178.435 65.405 0)
       (effects (font (size 1.27 1.27)) hide)
     )
@@
       (reference "#PWR0116") (unit 1) (value "Earth") (footprint "")
     )
+    (path "/da7b7fed-e089-4f9a-b121-597f1dede065"
+      (reference "#PWR0117") (unit 1) (value "Earth") (footprint "")
+    )
+    (path "/58dce8b4-330b-4018-9ad2-03758b5bcf64/b4085ae8-36cd-4942-9d92-5b9ca02250de"
+      (reference "#PWR0118") (unit 1) (value "GND-ISO-A") (footprint "")
+    )
     (path "/58dce8b4-330b-4018-9ad2-03758b5bcf64/0fb1d2f7-d6ac-499f-8b37-86a0baca3579"
       (reference "#PWR0201") (unit 1) (value "GND-ISO-A") (footprint "")
@@
       (reference "#PWR0929") (unit 1) (value "Earth") (footprint "")
     )
-    (path "/58dce8b4-330b-4018-9ad2-03758b5bcf64/b4085ae8-36cd-4942-9d92-5b9ca02250de"
-      (reference "#PWR?") (unit 1) (value "GND-ISO-A") (footprint "")
-    )
     (path "/58dce8b4-330b-4018-9ad2-03758b5bcf64/4acc0f00-f398-4825-bf6d-6f0cd46f9074"
       (reference "C201") (unit 1) (value "100n") (footprint "Capacitor_SMD:C_0603_1608Metric_Pad1.08x0.95mm_HandSolder")
@@
     )
     (path "/58dce8b4-330b-4018-9ad2-03758b5bcf64/38b5e452-8441-4b81-9620-131444429f1f"
-      (reference "C208") (unit 1) (value "100n") (footprint "Capacitor_SMD:C_0603_1608Metric_Pad1.08x0.95mm_HandSolder")
+      (reference "C208") (unit 1) (value "100n") (footprint "Capacitor_SMD:C_1206_3216Metric")
     )
     (path "/58dce8b4-330b-4018-9ad2-03758b5bcf64/6032a858-b0e2-4732-a382-a842e6bb8e5b"

Commit message: Update PCB layout
Parts:
- removed TP114, TP115: TestPoint, qds-cv-lib:TestPoint_Keystone_5010-5014_Multipurpose, symbol Connector:TestPoint
Connections:
- net VT1: now also TP102.1; no longer TP101.1
- net VT2: now also TP101.1; no longer TP102.1
Changed lines of the file:
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@@
   (junction (at 114.3 153.67) (diameter 0) (color 0 0 0 0)
   )
+  (junction (at 46.99 104.14) (diameter 0) (color 0 0 0 0)
+  )
   (junction (at 114.3 73.66) (diameter 0) (color 0 0 0 0)
   )
-  (junction (at 46.99 88.9) (diameter 0) (color 0 0 0 0)
-  )
   (junction (at 170.815 57.785) (diameter 0) (color 0 0 0 0)
   )
-  (junction (at 252.095 53.34) (diameter 0) (color 0 0 0 0)
-  )
   (junction (at 168.275 55.245) (diameter 0) (color 0 0 0 0)
   )
+  (junction (at 54.61 88.9) (diameter 0) (color 0 0 0 0)
+  )
   (junction (at 252.095 51.435) (diameter 0) (color 0 0 0 0)
   )
@@
   (junction (at 252.095 49.53) (diameter 0) (color 0 0 0 0)
   )
-  (junction (at 54.61 90.17) (diameter 0) (color 0 0 0 0)
-  )
   (junction (at 35.56 121.92) (diameter 0) (color 0 0 0 0)
   )
@@
     (stroke (width 0) (type default) (color 0 0 0 0))
   )
+  (wire (pts (xy 46.99 104.14) (xy 46.99 171.45))
+    (stroke (width 0) (type default) (color 0 0 0 0))
+  )
   (wire (pts (xy 168.275 48.26) (xy 168.275 55.245))
     (stroke (width 0) (type default) (color 0 0 0 0))
@@
     (stroke (width 0) (type default) (color 0 0 0 0))
   )
-  (wire (pts (xy 35.56 104.14) (xy 54.61 104.14))
-    (stroke (width 0) (type default) (color 0 0 0 0))
-  )
-  (wire (pts (xy 46.99 49.53) (xy 46.99 88.9))
+  (wire (pts (xy 35.56 104.14) (xy 46.99 104.14))
+    (stroke (width 0) (type default) (color 0 0 0 0))
+  )
+  (wire (pts (xy 46.99 49.53) (xy 46.99 104.14))
     (stroke (width 0) (type default) (color 0 0 0 0))
   )
@@
     (stroke (width 0) (type default) (color 0 0 0 0))
   )
-  (wire (pts (xy 35.56 88.9) (xy 46.99 88.9))
+  (wire (pts (xy 35.56 88.9) (xy 54.61 88.9))
     (stroke (width 0) (type default) (color 0 0 0 0))
   )
@@
     (stroke (width 0) (type default) (color 0 0 0 0))
   )
-  (wire (pts (xy 252.095 53.34) (xy 252.095 55.245))
-    (stroke (width 0) (type default) (color 0 0 0 0))
-  )
   (wire (pts (xy 161.925 62.865) (xy 178.435 62.865))
     (stroke (width 0) (type default) (color 0 0 0 0))
@@
     (stroke (width 0) (type default) (color 0 0 0 0))
   )
-  (wire (pts (xy 54.61 90.17) (xy 54.61 104.14))
-    (stroke (width 0) (type default) (color 0 0 0 0))
-  )
   (wire (pts (xy 104.14 165.1) (xy 104.14 153.67))
     (stroke (width 0) (type default) (color 0 0 0 0))
   )
-  (wire (pts (xy 54.61 90.17) (xy 54.61 55.88))
+  (wire (pts (xy 54.61 90.17) (xy 54.61 88.9))
     (stroke (width 0) (type default) (color 0 0 0 0))
   )
@@
     (stroke (width 0) (type default) (color 0 0 0 0))
   )
-  (wire (pts (xy 46.99 88.9) (xy 46.99 171.45))
+  (wire (pts (xy 54.61 88.9) (xy 54.61 55.88))
     (stroke (width 0) (type default) (color 0 0 0 0))
   )
@@
     )
     (property "Datasheet" "https://www.keyelco.com/product-pdf.cfm?p=1321" (id 3) (at 182.245 121.92 0)
-      (effects (font (size 1.27 1.27)) hide)
-    )
-    (pin "1")
-  )
-  (symbol (lib_id "Connector:TestPoint") (at 252.095 53.34 90) (unit 1)
-    (in_bom yes) (on_board yes)
-    (property "Reference" "TP114" (id 0) (at 244.475 53.34 90))
-    (property "Value" "TestPoint" (id 1) (at 248.793 49.53 90)
-      (effects (font (size 1.27 1.27)) hide)
-    )
-    (property "Footprint" "qds-cv-lib:TestPoint_Keystone_5010-5014_Multipurpose" (id 2) (at 252.095 48.26 0)
-      (effects (font (size 1.27 1.27)) hide)
-    )
-    (property "Datasheet" "https://www.keyelco.com/product-pdf.cfm?p=1321" (id 3) (at 252.095 48.26 0)
       (effects (font (size 1.27 1.27)) hide)
     )
@@
     (pin "1")
   )
-  (symbol (lib_id "Connector:TestPoint") (at 252.095 55.245 90) (unit 1)
-    (in_bom yes) (on_board yes)
-    (property "Reference" "TP115" (id 0) (at 244.475 55.245 90))
-    (property "Value" "TestPoint" (id 1) (at 248.793 51.435 90)
-      (effects (font (size 1.27 1.27)) hide)
-    )
-    (property "Footprint" "qds-cv-lib:TestPoint_Keystone_5010-5014_Multipurpose" (id 2) (at 252.095 50.165 0)
-      (effects (font (size 1.27 1.27)) hide)
-    )
-    (property "Datasheet" "https://www.keyelco.com/product-pdf.cfm?p=1321" (id 3) (at 252.095 50.165 0)
-      (effects (font (size 1.27 1.27)) hide)
-    )
-    (pin "1")
-  )
   (symbol (lib_id "power:Earth") (at 178.435 60.325 90) (unit 1)
     (in_bom yes) (on_board yes) (fields_autoplaced)
@@
     )
     (path "/9080f165-73ec-4038-a64c-5f7f77d629f0/0980d74d-7675-4a7f-95cf-ad0fc2222dd3"
-      (reference "R601") (unit 1) (value "1k") (footprint "Resistor_SMD:R_0805_2012Metric_Pad1.20x1.40mm_HandSolder")
+      (reference "R601") (unit 1) (value "4.7k") (footprint "Resistor_SMD:R_0805_2012Metric_Pad1.20x1.40mm_HandSolder")
     )
     (path "/9080f165-73ec-4038-a64c-5f7f77d629f0/0725f442-7b4f-4c23-8aca-7d56d49cc416"
@@
       (reference "TP113") (unit 1) (value "TestPoint") (footprint "qds-cv-lib:TestPoint_Keystone_5010-5014_Multipurpose")
     )
-    (path "/141ca897-0751-4f45-bae1-7eef20425b9c"
-      (reference "TP114") (unit 1) (value "TestPoint") (footprint "qds-cv-lib:TestPoint_Keystone_5010-5014_Multipurpose")
-    )
-    (path "/f0141e4a-7103-4848-bf0f-ffab9b9ebfda"
-      (reference "TP115") (unit 1) (value "TestPoint") (footprint "qds-cv-lib:TestPoint_Keystone_5010-5014_Multipurpose")
-    )
     (path "/024e8cff-bd14-487b-a98e-992b939de1a7"

Commit message: Finish routing
Connections:
- net +14V: now also J102.3 (Pin_3), TP109.1; no longer J102.1 (Pin_1), TP107.1
- net +15V: now also J102.1 (Pin_1), TP107.1; no longer J102.6 (Pin_6), TP110.1
- net +5V: now also J102.6 (Pin_6), TP110.1; no longer J102.3 (Pin_3), TP109.1
Changed lines of the file:
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@@
     (pin "1")
   )
-  (symbol (lib_id "qds-cv-lib-sym:+14V") (at 178.435 52.705 270) (unit 1)
-    (in_bom yes) (on_board yes) (fields_autoplaced)
-    (property "Reference" "#PWR0102" (id 0) (at 174.625 52.705 0)
-      (effects (font (size 1.27 1.27)) hide)
-    )
-    (property "Value" "+14V" (id 1) (at 181.61 52.7049 90)
-      (effects (font (size 1.27 1.27)) (justify left))
-    )
-    (property "Footprint" "" (id 2) (at 178.435 52.705 0)
-      (effects (font (size 1.27 1.27)) hide)
-    )
-    (property "Datasheet" "" (id 3) (at 178.435 52.705 0)
+  (symbol (lib_id "qds-cv-lib-sym:+14V") (at 178.435 57.785 270) (unit 1)
+    (in_bom yes) (on_board yes) (fields_autoplaced)
+    (property "Reference" "#PWR0102" (id 0) (at 174.625 57.785 0)
+      (effects (font (size 1.27 1.27)) hide)
+    )
+    (property "Value" "+14V" (id 1) (at 181.61 57.7849 90)
+      (effects (font (size 1.27 1.27)) (justify left))
+    )
+    (property "Footprint" "" (id 2) (at 178.435 57.785 0)
+      (effects (font (size 1.27 1.27)) hide)
+    )
+    (property "Datasheet" "" (id 3) (at 178.435 57.785 0)
       (effects (font (size 1.27 1.27)) hide)
     )
@@
     (pin "1")
   )
-  (symbol (lib_id "power:+15V") (at 178.435 65.405 270) (unit 1)
-    (in_bom yes) (on_board yes) (fields_autoplaced)
-    (property "Reference" "#PWR0106" (id 0) (at 174.625 65.405 0)
-      (effects (font (size 1.27 1.27)) hide)
-    )
-    (property "Value" "+15V" (id 1) (at 182.245 65.4049 90)
-      (effects (font (size 1.27 1.27)) (justify left))
-    )
-    (property "Footprint" "" (id 2) (at 178.435 65.405 0)
-      (effects (font (size 1.27 1.27)) hide)
-    )
-    (property "Datasheet" "" (id 3) (at 178.435 65.405 0)
+  (symbol (lib_id "power:+15V") (at 178.435 52.705 270) (unit 1)
+    (in_bom yes) (on_board yes) (fields_autoplaced)
+    (property "Reference" "#PWR0106" (id 0) (at 174.625 52.705 0)
+      (effects (font (size 1.27 1.27)) hide)
+    )
+    (property "Value" "+15V" (id 1) (at 182.245 52.7049 90)
+      (effects (font (size 1.27 1.27)) (justify left))
+    )
+    (property "Footprint" "" (id 2) (at 178.435 52.705 0)
+      (effects (font (size 1.27 1.27)) hide)
+    )
+    (property "Datasheet" "" (id 3) (at 178.435 52.705 0)
       (effects (font (size 1.27 1.27)) hide)
     )
@@
     (pin "1")
   )
-  (symbol (lib_id "power:+5V") (at 178.435 57.785 270) (unit 1)
-    (in_bom yes) (on_board yes) (fields_autoplaced)
-    (property "Reference" "#PWR0104" (id 0) (at 174.625 57.785 0)
-      (effects (font (size 1.27 1.27)) hide)
-    )
-    (property "Value" "+5V" (id 1) (at 181.61 57.7849 90)
-      (effects (font (size 1.27 1.27)) (justify left))
-    )
-    (property "Footprint" "" (id 2) (at 178.435 57.785 0)
-      (effects (font (size 1.27 1.27)) hide)
-    )
-    (property "Datasheet" "" (id 3) (at 178.435 57.785 0)
+  (symbol (lib_id "power:+5V") (at 178.435 65.405 270) (unit 1)
+    (in_bom yes) (on_board yes) (fields_autoplaced)
+    (property "Reference" "#PWR0104" (id 0) (at 174.625 65.405 0)
+      (effects (font (size 1.27 1.27)) hide)
+    )
+    (property "Value" "+5V" (id 1) (at 181.61 65.4049 90)
+      (effects (font (size 1.27 1.27)) (justify left))
+    )
+    (property "Footprint" "" (id 2) (at 178.435 65.405 0)
+      (effects (font (size 1.27 1.27)) hide)
+    )
+    (property "Datasheet" "" (id 3) (at 178.435 65.405 0)
       (effects (font (size 1.27 1.27)) hide)
     )
@@
     )
     (path "/9080f165-73ec-4038-a64c-5f7f77d629f0/885b0b11-1b27-42be-ab2d-d124a186fd45"
-      (reference "SW601") (unit 1) (value "SW_DIP_x05") (footprint "Button_Switch_SMD:SW_DIP_SPSTx05_Slide_6.7x14.26mm_W8.61mm_P2.54mm_LowProfile")
+      (reference "SW601") (unit 1) (value "SW_DIP_x04") (footprint "Button_Switch_SMD:SW_DIP_SPSTx04_Slide_6.7x11.72mm_W8.61mm_P2.54mm_LowProfile")
     )
     (path "/ad0bcf00-14ba-4be3-9e78-9e4ee2d714d5/bb451759-225a-4537-b020-f44335e01d55"

Commit message: Finish PCB layout including revision close #9 close #10 close #11 close #12 close #13 close #14 close #15 close #16
Parts:
- added TP120, TP121: TestPoint, qds-cv-lib:TestPoint_Keystone_5010-5014_Multipurpose, symbol Connector:TestPoint
Connections:
- net +14V: now also J102.4 (Pin_4); no longer J102.3 (Pin_3)
- net -14V: now also J102.3 (Pin_3); no longer J102.2 (Pin_2)
- net Earth: now also J102.2 (Pin_2), TP120.1, TP121.1; no longer J102.4 (Pin_4)
Other:
- moved on the sheet: TP116, TP117, TP118, TP119
