File: pcb/cad/qds-cv.kicad_sch (KiCad schematic)
At the start: 23 parts, among them J101 DB25 Female

Commit message: Start PCB design based on 1-channel version layout
Parts:
- added FID101, FID102, FID103, FID104: Fiducial, symbol Mechanical:Fiducial
Changed lines of the file:
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@@
     (pin "1")
+  )
+  (symbol (lib_id "Mechanical:Fiducial") (at 206.375 153.035 0) (unit 1)
+    (in_bom yes) (on_board yes)
+    (property "Reference" "FID101" (id 0) (at 197.485 153.035 0)
+      (effects (font (size 1.27 1.27)) (justify left))
+    )
+    (property "Value" "Fiducial" (id 1) (at 209.55 154.3049 0)
+      (effects (font (size 1.27 1.27)) (justify left) hide)
+    )
+    (property "Footprint" "" (id 2) (at 206.375 153.035 0)
+      (effects (font (size 1.27 1.27)) hide)
+    )
+    (property "Datasheet" "~" (id 3) (at 206.375 153.035 0)
+      (effects (font (size 1.27 1.27)) hide)
+    )
   )
   (symbol (lib_id "qds-cv-lib-sym:GND-ISO-D") (at 240.665 157.48 270) (unit 1)
@@
     (pin "1")
   )
+  (symbol (lib_id "Mechanical:Fiducial") (at 211.455 157.48 0) (unit 1)
+    (in_bom yes) (on_board yes)
+    (property "Reference" "FID104" (id 0) (at 213.36 157.48 0)
+      (effects (font (size 1.27 1.27)) (justify left))
+    )
+    (property "Value" "Fiducial" (id 1) (at 214.63 158.7499 0)
+      (effects (font (size 1.27 1.27)) (justify left) hide)
+    )
+    (property "Footprint" "" (id 2) (at 211.455 157.48 0)
+      (effects (font (size 1.27 1.27)) hide)
+    )
+    (property "Datasheet" "~" (id 3) (at 211.455 157.48 0)
+      (effects (font (size 1.27 1.27)) hide)
+    )
+  )
   (symbol (lib_id "power:Earth") (at 266.065 160.655 0) (unit 1)
     (in_bom yes) (on_board yes) (fields_autoplaced)
@@
     (pin "1")
   )
+  (symbol (lib_id "Mechanical:Fiducial") (at 211.455 153.035 0) (unit 1)
+    (in_bom yes) (on_board yes)
+    (property "Reference" "FID103" (id 0) (at 213.36 153.035 0)
+      (effects (font (size 1.27 1.27)) (justify left))
+    )
+    (property "Value" "Fiducial" (id 1) (at 214.63 154.3049 0)
+      (effects (font (size 1.27 1.27)) (justify left) hide)
+    )
+    (property "Footprint" "" (id 2) (at 211.455 153.035 0)
+      (effects (font (size 1.27 1.27)) hide)
+    )
+    (property "Datasheet" "~" (id 3) (at 211.455 153.035 0)
+      (effects (font (size 1.27 1.27)) hide)
+    )
+  )
   (symbol (lib_id "Connector:TestPoint") (at 240.665 137.795 270) (unit 1)
     (in_bom yes) (on_board yes) (fields_autoplaced)
@@
     )
     (pin "1")
+  )
+  (symbol (lib_id "Mechanical:Fiducial") (at 206.375 157.48 0) (unit 1)
+    (in_bom yes) (on_board yes)
+    (property "Reference" "FID102" (id 0) (at 197.485 157.48 0)
+      (effects (font (size 1.27 1.27)) (justify left))
+    )
+    (property "Value" "Fiducial" (id 1) (at 209.55 158.7499 0)
+      (effects (font (size 1.27 1.27)) (justify left) hide)
+    )
+    (property "Footprint" "" (id 2) (at 206.375 157.48 0)
+      (effects (font (size 1.27 1.27)) hide)
+    )
+    (property "Datasheet" "~" (id 3) (at 206.375 157.48 0)
+      (effects (font (size 1.27 1.27)) hide)
+    )
   )
   (symbol (lib_id "power:Earth") (at 27.94 139.7 0) (unit 1)
@@
       (reference "F901") (unit 1) (value "Fuse") (footprint "qds-cv-lib:ZH242")
     )
+    (path "/1a74589e-8294-4d5f-8ec5-103577a60293"
+      (reference "FID101") (unit 1) (value "Fiducial") (footprint "")
+    )
+    (path "/abe71458-5cd8-446f-9708-e78241464442"
+      (reference "FID102") (unit 1) (value "Fiducial") (footprint "")
+    )
+    (path "/63b58f54-de2f-47c2-88e2-fee7536fd8f1"
+      (reference "FID103") (unit 1) (value "Fiducial") (footprint "")
+    )
+    (path "/3bf8fc60-3967-4de7-9d3b-34dfb5d5e0a8"
+      (reference "FID104") (unit 1) (value "Fiducial") (footprint "")
+    )
     (path "/038aff54-beed-4c4d-80b5-b4a1c6c1a463"

Commit message: Reposition of channels and connectors, place and route trigger and actuation circuit
Connections:
- net VT1: now also J101.12, J101.24 (P24); no longer J101.15 (P15), J101.2
- net VT2: now also J101.21 (P21), J101.9; no longer J101.18 (P18), J101.5
- net VT3: now also J101.18 (P18), J101.5; no longer J101.21 (P21), J101.9
- net VT4: now also J101.15 (P15), J101.2; no longer J101.12, J101.24 (P24)
Other:
- moved on the sheet: J101
Changed lines of the file:
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@@
-    (stroke (width 0) (type default) (color 0 0 0 0))
-  )
-  (wire (pts (xy 29.21 139.7) (xy 27.94 139.7))
     (stroke (width 0) (type default) (color 0 0 0 0))
   )
@@
     (effects (font (size 1.27 1.27)) (justify left bottom))
   )
-  (symbol (lib_id "Connector:DB25_Female_MountingHoles") (at 29.21 104.14 0) (mirror y) (unit 1)
+  (symbol (lib_id "Connector:DB25_Female_MountingHoles") (at 29.21 104.14 180) (unit 1)
     (in_bom yes) (on_board yes)
-    (property "Reference" "J101" (id 0) (at 24.13 109.2201 0)
-      (effects (font (size 1.27 1.27)) (justify left))
-    )
-    (property "Value" "DB25 Female" (id 1) (at 22.86 106.68 90)
+    (property "Reference" "J101" (id 0) (at 24.13 99.0599 0)
+      (effects (font (size 1.27 1.27)) (justify left))
+    )
+    (property "Value" "DB25 Female" (id 1) (at 22.86 101.6 90)
       (effects (font (size 1.27 1.27)) (justify left))
     )
@@
     )
   )
-  (symbol (lib_id "power:Earth") (at 27.94 139.7 0) (unit 1)
-    (in_bom yes) (on_board yes) (fields_autoplaced)
-    (property "Reference" "#PWR0107" (id 0) (at 27.94 146.05 0)
-      (effects (font (size 1.27 1.27)) hide)
-    )
-    (property "Value" "Earth" (id 1) (at 27.94 143.51 0)
-      (effects (font (size 1.27 1.27)) hide)
-    )
-    (property "Footprint" "" (id 2) (at 27.94 139.7 0)
-      (effects (font (size 1.27 1.27)) hide)
-    )
-    (property "Datasheet" "~" (id 3) (at 27.94 139.7 0)
+  (symbol (lib_id "power:Earth") (at 29.21 68.58 270) (unit 1)
+    (in_bom yes) (on_board yes) (fields_autoplaced)
+    (property "Reference" "#PWR0107" (id 0) (at 22.86 68.58 0)
+      (effects (font (size 1.27 1.27)) hide)
+    )
+    (property "Value" "Earth" (id 1) (at 25.4 68.58 0)
+      (effects (font (size 1.27 1.27)) hide)
+    )
+    (property "Footprint" "" (id 2) (at 29.21 68.58 0)
+      (effects (font (size 1.27 1.27)) hide)
+    )
+    (property "Datasheet" "~" (id 3) (at 29.21 68.58 0)
       (effects (font (size 1.27 1.27)) hide)
     )
@@
       (reference "U703") (unit 1) (value "74LV132") (footprint "Package_SO:SO-14_3.9x8.65mm_P1.27mm")
     )
-    (path "/ad0bcf00-14ba-4be3-9e78-9e4ee2d714d5/cdade767-5111-4eca-b560-eccb92caa51a"
+    (path "/ad0bcf00-14ba-4be3-9e78-9e4ee2d714d5/662173bd-dda7-4715-8318-919e3602a656"
       (reference "U703") (unit 2) (value "74LV132") (footprint "Package_SO:SO-14_3.9x8.65mm_P1.27mm")
     )
@@
       (reference "U703") (unit 3) (value "74LV132") (footprint "Package_SO:SO-14_3.9x8.65mm_P1.27mm")
     )
-    (path "/ad0bcf00-14ba-4be3-9e78-9e4ee2d714d5/662173bd-dda7-4715-8318-919e3602a656"
+    (path "/ad0bcf00-14ba-4be3-9e78-9e4ee2d714d5/cdade767-5111-4eca-b560-eccb92caa51a"
       (reference "U703") (unit 4) (value "74LV132") (footprint "Package_SO:SO-14_3.9x8.65mm_P1.27mm")
     )
@@
       (reference "U704") (unit 3) (value "74LVC2G17") (footprint "Package_TO_SOT_SMD:SOT-23-6_Handsoldering")
     )
+    (path "/ad0bcf00-14ba-4be3-9e78-9e4ee2d714d5/08eb767d-dfe5-4b9c-b99b-a8c3913ca2c3"
+      (reference "U705") (unit 1) (value "74LVC2G17") (footprint "Package_TO_SOT_SMD:SOT-23-6_Handsoldering")
+    )
     (path "/ad0bcf00-14ba-4be3-9e78-9e4ee2d714d5/f1cb1b09-3a32-49c9-b31d-f3d3fc6082be"
-      (reference "U705") (unit 1) (value "74LVC2G17") (footprint "Package_TO_SOT_SMD:SOT-23-6_Handsoldering")
-    )
-    (path "/ad0bcf00-14ba-4be3-9e78-9e4ee2d714d5/08eb767d-dfe5-4b9c-b99b-a8c3913ca2c3"
       (reference "U705") (unit 2) (value "74LVC2G17") (footprint "Package_TO_SOT_SMD:SOT-23-6_Handsoldering")
     )

Commit message: Apply several changes based on test results - replace validation time 4k7 resistor by a 8k2, close #21 - remove pull-up resistor from AMC1200 positive input - split voltage taps pull-up/down resistors into 2 footprints each - change C204,304,404,504 footprints from 0603 to 0805 - include bypass switch for software trigger - remove test points from voltage taps - change window comparator input resistor to 4k7 - include footprint for a 0805 capacitor at the window comparator input
Parts:
- removed TP101: VT1, symbol Connector:TestPoint
- removed TP102: VT2, symbol Connector:TestPoint
- removed TP103: VT3, symbol Connector:TestPoint
- removed TP104: VT4, symbol Connector:TestPoint

Commit message: Place test-points, improve isolated circuit layout (channel D only)
Parts:
- TP105: value TestPoint -> +5V-ISO-A
- TP106: value TestPoint -> +5V-ISO-B
- TP107: value TestPoint -> +5V-ISO-C
- TP108: value TestPoint -> +5V-ISO-D
- TP109: value TestPoint -> GND-ISO-A; footprint (none) -> qds-cv-lib:TestPoint_Keystone_5010-5014_Multipurpose
- TP110: value TestPoint -> GND-ISO-B; footprint (none) -> qds-cv-lib:TestPoint_Keystone_5010-5014_Multipurpose
- TP111: value TestPoint -> GND-ISO-C; footprint (none) -> qds-cv-lib:TestPoint_Keystone_5010-5014_Multipurpose
- TP112: value TestPoint -> GND-ISO-D; footprint (none) -> qds-cv-lib:TestPoint_Keystone_5010-5014_Multipurpose
- TP113: value TestPoint -> +15V; footprint (none) -> qds-cv-lib:TestPoint_Keystone_5010-5014_Multipurpose
- TP114: value TestPoint -> +14V; footprint (none) -> qds-cv-lib:TestPoint_Keystone_5010-5014_Multipurpose
- TP115: value TestPoint -> -14V; footprint (none) -> qds-cv-lib:TestPoint_Keystone_5010-5014_Multipurpose
- TP116: value TestPoint -> +5V; footprint (none) -> qds-cv-lib:TestPoint_Keystone_5010-5014_Multipurpose
- TP117, TP118, TP119, TP120: value TestPoint -> GND; footprint (none) -> qds-cv-lib:TestPoint_Keystone_5010-5014_Multipurpose
- TP121, TP122: value TestPoint -> GND; footprint (none) -> TestPoint:TestPoint_Pad_D2.0mm
