File: pcb/cad/power-supplies.kicad_sch (KiCad schematic)
At the start: 0 parts

Commit message: Power supplies schematic created
Parts:
- added C? (x6): C, symbol Device:C
- added D?: SMBJ15A, Diode_SMD:D_SMB, symbol Diode:SM6T15A
- added F?: Fuse, qds-cv-lib:ZH242, symbol Device:Fuse
- added J?: Barrel_Jack_Switch, qds-cv-lib:CUI_PJ-002AH, symbol Connector:Barrel_Jack_Switch
- added PS?: JCM3012D15, qds-cv-lib:JCM30, symbol qds-cv-lib-sym:JCM3012D15
- added PS?: RI-1515S, qds-cv-lib:RI-1515S, symbol qds-cv-lib-sym:RI-1515S
- added R?: 47k, Resistor_SMD:R_0603_1608Metric_Pad0.98x0.95mm_HandSolder, symbol Device:R_US
- added R?: 4k42, Resistor_SMD:R_0603_1608Metric_Pad0.98x0.95mm_HandSolder, symbol Device:R_US
- added U?: R-78E5.0-0.5, Converter_DCDC:Converter_DCDC_RECOM_R-78E-0.5_THT, symbol Regulator_Switching:R-78E5.0-0.5
- added U?: LT1965EMS8E_PBF, SOP65P490X110-9N, symbol qds-cv-lib-sym:LT1965EMS8E_PBF
- added U?: LT1129-5.0_SOT223, Package_TO_SOT_SMD:SOT-223-3_TabPin2, symbol Regulator_Linear:LT1129-5.0_SOT223
Connections:
- new net: R?.1, R?.2, U?.3 (ADJ)
- new net: D?.1 (A1), F?.2, PS?.1 (+VIN), PS?.3 (REMOTE_ON/OFF)
- new net: D?.2 (A2), J?.2, PS?.2 (-VIN)
- new net: PS?.4 (+VOUT), U?.1 (VI)
- new net: F?.1, J?.1
- new net +14V: R?.1, U?.1 (OUT), U?.2 (OUT)
- new net +15V: C?.1, C?.1, PS?.2 (+VIN), PS?.4 (+VOUT), U?.1 (IN), U?.6 (~{SHDN}), U?.7 (IN), U?.8 (IN)
- new net +5V: U?.3 (OUT)
- new net +5V-ISO-A: U?.3 (VO)
- new net -15V: C?.2, C?.2, PS?.6 (-VOUT)
- new net GND: C?.1, C?.1, C?.2, C?.2, PS?.1 (-VIN), PS?.5 (COMMON), R?.2, U?.2 (GND), U?.4 (GND), U?.5 (GND), U?.9 (PAD)
- new net GND-ISO-A: PS?.3 (-VOUT), U?.2 (GND)
Other:
- title: (none) -> Power Supplies

Commit message: Included power supplies circuits and +5V-REF RC circuit in analog front-end
Parts:
- removed C? (x6): C, symbol Device:C
- added C? (x21): 10u, Capacitor_SMD:C_0805_2012Metric_Pad1.18x1.45mm_HandSolder, symbol Device:C_Small
- added C? (x8): 100n, Capacitor_SMD:C_0603_1608Metric_Pad1.08x0.95mm_HandSolder, symbol Device:C_Small
- added C? (x2): 1u, Capacitor_SMD:C_0805_2012Metric_Pad1.18x1.45mm_HandSolder, symbol Device:C_Small
- added C? (x2): 22u, symbol Device:C_Polarized_Small_US
- added LD?: Green, qds-cv-lib:LED_WP934CB_GD, symbol Device:LED
- added PS? (x3): RI-1515S, qds-cv-lib:RI-1515S, symbol qds-cv-lib-sym:RI-1515S
- added R? (x4): 1k3, Capacitor_SMD:C_0805_2012Metric_Pad1.18x1.45mm_HandSolder, symbol Device:R_US
- added R?: 127k, Resistor_SMD:R_0603_1608Metric_Pad0.98x0.95mm_HandSolder, symbol Device:R_US
- added R?: 270, Resistor_SMD:R_0805_2012Metric_Pad1.20x1.40mm_HandSolder, symbol Device:R_US
- added R?: 12k1, Resistor_SMD:R_0603_1608Metric_Pad0.98x0.95mm_HandSolder, symbol Device:R_US
- added U? (x3): LT1129CST-5, Package_TO_SOT_SMD:SOT-223-3_TabPin2, symbol Regulator_Linear:LT1129-5.0_SOT223
- added U?: LT3015EMSEPBF, MSOP-12_MSE, symbol qds-cv-lib-sym:LT3015EMSEPBF
- U?: MANUFACTURER Analog Devices -> (none); MAXIMUM_PACKAGE_HEIGHT 1.1 mm -> (none); PARTREV B -> (none); SNAPEDA_PN LT1965EMS8E#PBF -> (none); STANDARD IPC 7351B -> (none)
- U?: value LT1129-5.0_SOT223 -> LT1129CST-5; CNPEM Code (none) -> AR100794; Manufacturer (none) -> Analog Devices Inc.; Part Number (none) -> LT1129CST-5#TRPBF; Vendor Link (none) -> https://br.mouser.com/ProductDetail/Analog-Devices/LT1129CS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
Connections:
- net +14V: now also C?.1, C?.1, C?.1
- net +15V: now also C?.1, C?.1, C?.1, C?.1, C?.1, C?.1, C?.1, C?.1, C?.1, C?.1, PS?.2 (+VIN), PS?.2 (+VIN), PS?.2 (+VIN)
- net +5V: now also LD?.2 (A), R?.2; no longer U?.3 (OUT)
- net +5V-ISO-A: now also C?.1
- net -15V: now also U?.1 (IN_2), U?.13 (EPAD), U?.2 (IN_3), U?.3 (IN_4), U?.4 (IN), U?.5 (*SHDN)
- net GND-ISO-A: now also C?.2, C?.2, R?.2
- net at D?.1 (A1), F?.2, PS?.1 (+VIN)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: now also C?.1, C?.1, C?.1
- net at D?.2 (A2), J?.2, PS?.2 (-VIN): now also C?.2, C?.2, C?.2
- net at PS?.4 (+VOUT), U?.1 (VI): now also C?.1, R?.1
- net GND renamed Earth
- net Earth: now also C?.2, C?.2, C?.2, C?.2, C?.2, C?.2, C?.2, C?.2, C?.2, C?.2, C?.2, C?.2, C?.2, C?.2, C?.2, C?.2, C?.2, C?.2, LD?.1 (K), PS?.1 (-VIN), PS?.1 (-VIN), PS?.1 (-VIN), R?.2, U?.6 (GND_2), U?.7 (GND)
- new net: C?.1, PS?.4 (+VOUT), R?.1, U?.1 (VI) (x3)
- new net: C?.1, C?.1, R?.1, U?.3 (OUT)
- new net: R?.1, R?.2, U?.8 (SENSE/ADJ)
- new net +5V-ISO-B: C?.1, U?.3 (VO)
- new net +5V-ISO-C: C?.1, U?.3 (VO)
- new net +5V-ISO-D: C?.1, U?.3 (VO)
- new net -14V: C?.1, C?.1, C?.1, R?.1, U?.10 (OUT_3), U?.11 (OUT_4), U?.12 (OUT), U?.9 (OUT_2)
- new net GND-ISO-B: C?.2, C?.2, PS?.3 (-VOUT), R?.2, U?.2 (GND)
- new net GND-ISO-C: C?.2, C?.2, PS?.3 (-VOUT), R?.2, U?.2 (GND)
- new net GND-ISO-D: C?.2, C?.2, PS?.3 (-VOUT), R?.2, U?.2 (GND)
Other:
- note added: "+14V linear regulator"
- note added: "+5V DC-DC converter"
- note added: "-14V linear regulator"
- note added: "Isolated power supplies"
- note added: "Max capacitive load: 220 uF"
- note added: "Max capacitive load: 500 uF"
- note added: "Optional to provide minimum load"
- note added: "Switching freq: 330 kHz Noise: 60 mVpk-pk (Cout = 10 uF)"
- note added: "±15V main isolated DC-DC converter"
- moved on the sheet: D?, F?, J?, PS?, R?, U?

Commit message: specify components used in front-end, validation and power circuits, except resistors
Parts:
- C? (x21): Part Number C2012X5R1V106KT0J0E -> C2012X5R1V106K085AC
- C? (x2): footprint (none) -> Capacitor_Tantalum_SMD:CP_EIA-6032-28_Kemet-C_Pad2.25x2.35mm_HandSolder
- R?: Manufacturer Panasonic Electronic Components -> Panasonic
Changed lines of the file:
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@@
       (effects (font (size 1.27 1.27)) hide)
     )
-    (property "Manufacturer" "Panasonic Electronic Components" (id 6) (at 102.87 127 0)
+    (property "Manufacturer" "Panasonic" (id 6) (at 102.87 127 0)
       (effects (font (size 1.27 1.27)) hide)
     )
@@
       (effects (font (size 1.27 1.27)) hide)
     )
-    (property "Part Number" "C2012X5R1V106KT0J0E" (id 5) (at 64.77 53.34 0)
+    (property "Part Number" "C2012X5R1V106K085AC" (id 5) (at 64.77 53.34 0)
       (effects (font (size 1.27 1.27)) hide)
     )
@@
       (effects (font (size 1.27 1.27)) hide)
     )
-    (property "Part Number" "C2012X5R1V106KT0J0E" (id 5) (at 245.11 116.84 0)
+    (property "Part Number" "C2012X5R1V106K085AC" (id 5) (at 245.11 116.84 0)
       (effects (font (size 1.27 1.27)) hide)
     )
@@
       (effects (font (size 1.27 1.27)) hide)
     )
-    (property "Part Number" "C2012X5R1V106KT0J0E" (id 5) (at 54.61 91.44 0)
+    (property "Part Number" "C2012X5R1V106K085AC" (id 5) (at 54.61 91.44 0)
       (effects (font (size 1.27 1.27)) hide)
     )
@@
       (effects (font (size 1.27 1.27)) hide)
     )
-    (property "Part Number" "C2012X5R1V106KT0J0E" (id 5) (at 273.05 52.07 0)
+    (property "Part Number" "C2012X5R1V106K085AC" (id 5) (at 273.05 52.07 0)
       (effects (font (size 1.27 1.27)) hide)
     )
@@
       (effects (font (size 1.27 1.27)) hide)
     )
-    (property "Part Number" "C2012X5R1V106KT0J0E" (id 5) (at 99.06 91.44 0)
+    (property "Part Number" "C2012X5R1V106K085AC" (id 5) (at 99.06 91.44 0)
       (effects (font (size 1.27 1.27)) hide)
     )
@@
       (effects (font (size 1.27 1.27)) hide)
     )
-    (property "Part Number" "C2012X5R1V106KT0J0E" (id 5) (at 86.36 53.34 0)
+    (property "Part Number" "C2012X5R1V106K085AC" (id 5) (at 86.36 53.34 0)
       (effects (font (size 1.27 1.27)) hide)
     )
@@
       (effects (font (size 1.27 1.27)) hide)
     )
-    (property "Part Number" "C2012X5R1V106KT0J0E" (id 5) (at 76.2 53.34 0)
+    (property "Part Number" "C2012X5R1V106K085AC" (id 5) (at 76.2 53.34 0)
       (effects (font (size 1.27 1.27)) hide)
     )
@@
       (effects (font (size 1.27 1.27)) hide)
     )
-    (property "Part Number" "C2012X5R1V106KT0J0E" (id 5) (at 182.88 116.84 0)
+    (property "Part Number" "C2012X5R1V106K085AC" (id 5) (at 182.88 116.84 0)
       (effects (font (size 1.27 1.27)) hide)
     )
@@
       (effects (font (size 1.27 1.27)) hide)
     )
-    (property "Part Number" "C2012X5R1V106KT0J0E" (id 5) (at 182.88 52.07 0)
+    (property "Part Number" "C2012X5R1V106K085AC" (id 5) (at 182.88 52.07 0)
       (effects (font (size 1.27 1.27)) hide)
     )
@@
       (effects (font (size 1.27 1.27)) hide)
     )
-    (property "Part Number" "C2012X5R1V106KT0J0E" (id 5) (at 245.11 83.82 0)
+    (property "Part Number" "C2012X5R1V106K085AC" (id 5) (at 245.11 83.82 0)
       (effects (font (size 1.27 1.27)) hide)
     )
@@
       (effects (font (size 1.27 1.27)) (justify left))
     )
-    (property "Footprint" "" (id 2) (at 121.92 176.53 0)
+    (property "Footprint" "Capacitor_Tantalum_SMD:CP_EIA-6032-28_Kemet-C_Pad2.25x2.35mm_HandSolder" (id 2) (at 121.92 176.53 0)
       (effects (font (size 1.27 1.27)) hide)
     )
@@
       (effects (font (size 1.27 1.27)) hide)
     )
-    (property "Part Number" "C2012X5R1V106KT0J0E" (id 5) (at 142.24 57.15 0)
+    (property "Part Number" "C2012X5R1V106K085AC" (id 5) (at 142.24 57.15 0)
       (effects (font (size 1.27 1.27)) hide)
     )
@@
       (effects (font (size 1.27 1.27)) hide)
     )
-    (property "Part Number" "C2012X5R1V106KT0J0E" (id 5) (at 273.05 148.59 0)
+    (property "Part Number" "C2012X5R1V106K085AC" (id 5) (at 273.05 148.59 0)
       (effects (font (size 1.27 1.27)) hide)
     )
@@
       (effects (font (size 1.27 1.27)) hide)
     )
-    (property "Part Number" "C2012X5R1V106KT0J0E" (id 5) (at 273.05 116.84 0)
+    (property "Part Number" "C2012X5R1V106K085AC" (id 5) (at 273.05 116.84 0)
       (effects (font (size 1.27 1.27)) hide)
     )
@@
       (effects (font (size 1.27 1.27)) hide)
     )
-    (property "Part Number" "C2012X5R1V106KT0J0E" (id 5) (at 163.83 57.15 0)
+    (property "Part Number" "C2012X5R1V106K085AC" (id 5) (at 163.83 57.15 0)
       (effects (font (size 1.27 1.27)) hide)
     )
@@
       (effects (font (size 1.27 1.27)) hide)
     )
-    (property "Part Number" "C2012X5R1V106KT0J0E" (id 5) (at 245.11 52.07 0)
+    (property "Part Number" "C2012X5R1V106K085AC" (id 5) (at 245.11 52.07 0)
       (effects (font (size 1.27 1.27)) hide)
     )
@@
       (effects (font (size 1.27 1.27)) hide)
     )
-    (property "Part Number" "C2012X5R1V106KT0J0E" (id 5) (at 273.05 83.82 0)
+    (property "Part Number" "C2012X5R1V106K085AC" (id 5) (at 273.05 83.82 0)
       (effects (font (size 1.27 1.27)) hide)
     )
@@
       (effects (font (size 1.27 1.27)) hide)
     )
-    (property "Part Number" "C2012X5R1V106KT0J0E" (id 5) (at 245.11 148.59 0)
+    (property "Part Number" "C2012X5R1V106K085AC" (id 5) (at 245.11 148.59 0)
       (effects (font (size 1.27 1.27)) hide)
     )
@@
       (effects (font (size 1.27 1.27)) hide)
     )
-    (property "Part Number" "C2012X5R1V106KT0J0E" (id 5) (at 182.88 83.82 0)
+    (property "Part Number" "C2012X5R1V106K085AC" (id 5) (at 182.88 83.82 0)
       (effects (font (size 1.27 1.27)) hide)
     )
@@
       (effects (font (size 1.27 1.27)) hide)
     )
-    (property "Part Number" "C2012X5R1V106KT0J0E" (id 5) (at 163.83 49.53 0)
+    (property "Part Number" "C2012X5R1V106K085AC" (id 5) (at 163.83 49.53 0)
       (effects (font (size 1.27 1.27)) hide)
     )
@@
       (effects (font (size 1.27 1.27)) hide)
     )
-    (property "Part Number" "C2012X5R1V106KT0J0E" (id 5) (at 182.88 148.59 0)
+    (property "Part Number" "C2012X5R1V106K085AC" (id 5) (at 182.88 148.59 0)
       (effects (font (size 1.27 1.27)) hide)
     )
@@
       (effects (font (size 1.27 1.27)) hide)
     )
-    (property "Part Number" "C2012X5R1V106KT0J0E" (id 5) (at 152.4 57.15 0)
+    (property "Part Number" "C2012X5R1V106K085AC" (id 5) (at 152.4 57.15 0)
       (effects (font (size 1.27 1.27)) hide)
     )
@@
       (effects (font (size 1.27 1.27)) (justify left))
     )
-    (property "Footprint" "" (id 2) (at 121.92 132.08 0)
-      (effects (font (size 1.27 1.27)) hide)
-    )
+    (property "Footprint" "Capacitor_Tantalum_SMD:CP_EIA-6032-28_Kemet-C_Pad2.25x2.35mm_HandSolder" (id 2) (at 121.92 132.08 0)
+      (effects (font (size 1.27 1.27)) hide)
+    )

Commit message: Update componentes fields and reference circuit
Parts:
- PS? (x4): value RI-1515S -> RI-1515S/P; CNPEM Code (none) -> MT108486; Manufacturer (none) -> Recom Power; Part Number (none) -> RI-1515S/P; Vendor Link (none) -> https://www.digikey.com/en/products/detail/recom-power/RI-1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
- PS?: CNPEM Code (none) -> MT103202; Manufacturer (none) -> XP Power; Part Number (none) -> JCM3012D15; Vendor Link (none) -> https://www.digikey.com/en/products/detail/xp-power/JCM3012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
- R?: Manufacturer Panasonic -> Panasonic Electronic Components
- R? (x4): value 1k3 -> 1.3k; footprint Capacitor_SMD:C_0805_2012Metric_Pad1.18x1.45mm_HandSolder -> Resistor_SMD:R_0805_2012Metric_Pad1.20x1.40mm_HandSolder
- R?: value 4k42 -> 4.42k
- R?: CNPEM Code MT104052 -> (none); Manufacturer Yageo -> Fenghua Advance Technology; Part Number RC0805FR-07270RL -> RC-05K203JT; Vendor Link https://www.digikey.com/en/products/detail/yageo/RC0805FR-0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 -> (none)
- R?: value 12k1 -> 12.1k

Commit message: Update power supplies, symbols and footprint libs
Parts:
- removed C? (x7): 10u, Capacitor_SMD:C_0805_2012Metric_Pad1.18x1.45mm_HandSolder, symbol Device:C_Small
- removed D?: SMBJ15A, Diode_SMD:D_SMB, symbol Diode:SM6T15A
- added C901, C909: 22u, Capacitor_Tantalum_SMD:CP_EIA-6032-28_Kemet-C_Pad2.25x2.35mm_HandSolder, symbol Device:C_Polarized_Small_US
- added C902, C908, C910: 1u, Capacitor_SMD:C_0805_2012Metric_Pad1.18x1.45mm_HandSolder, symbol Device:C_Small
- added C907: 100u, Capacitor_SMD:C_Elec_6.3x7.7, symbol Device:C_Polarized_Small_US
- added C923, C932: 10u, Capacitor_SMD:C_0805_2012Metric_Pad1.18x1.45mm_HandSolder, symbol Device:C_Small
- added C924, C933: 100n, Capacitor_SMD:C_0603_1608Metric_Pad1.08x0.95mm_HandSolder, symbol Device:C_Small
- added D901: SMBJ15A, Diode_SMD:D_SMB, symbol Diode:SM6T15A
- U903: renamed from U?; Manufacturer (none) -> Recom Power; Part Number (none) -> R-78E5.0-0.5; Vendor Link (none) -> https://br.mouser.com/ProductDetail/RECOM-Power/R-78E50-05?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
- U905: renamed from U?; footprint SOP65P490X110-9N -> qds-cv-lib:SOP65P490X110-9N; Manufacturer (none) -> Analog Devices; Part Number (none) -> LT1965EMS8E; Vendor Link (none) -> https://www.digikey.com/en/products/detail/analog-devices-i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
- U907: renamed from U?; footprint MSOP-12_MSE -> qds-cv-lib:MSOP-12_MSE; Manufacturer (none) -> Analog Devices Inc.; Part Number (none) -> LT3015EMSEPBF; Vendor Link (none) -> https://www.digikey.com/en/products/detail/analog-devices-i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
- gave numbers to parts that had none: 47
Connections:
- net +15V: now also C901.1, C902.1, C923.1, C924.1
- net -15V: now also C909.2, C910.2, C932.1, C933.1
- net Earth: now also C901.2, C902.2, C909.1, C910.1, C923.2, C924.2, C932.2, C933.2
- net at F901.2, PS901.1 (+VIN), PS901.3 (REMOTE_ON/OFF): now also C907.1, C908.1, D901.1 (A1)
- net at J901.2, PS901.2 (-VIN): now also C907.2, C908.2, D901.2 (A2)
Other:
- moved on the sheet: F901, J901

Commit message: Fix +5V power reference so it is connected to R-78E5 output
Connections:
- net +5V: now also C917.1, C918.1, R903.1, U903.3 (OUT); no longer LD901.2 (A), R903.2
- new net: LD901.2 (A), R903.2
Changed lines of the file:
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@@
   (junction (at 137.16 53.34) (diameter 0) (color 0 0 0 0)
-  )
-  (junction (at 130.81 86.36) (diameter 0) (color 0 0 0 0)
   )
   (junction (at 273.05 46.99) (diameter 0) (color 0 0 0 0)
@@
     (pin "2")
   )
-  (symbol (lib_id "power:+5V") (at 130.81 86.36 0) (unit 1)
-    (in_bom yes) (on_board yes) (fields_autoplaced)
-    (property "Reference" "#PWR0911" (id 0) (at 130.81 90.17 0)
-      (effects (font (size 1.27 1.27)) hide)
-    )
-    (property "Value" "+5V" (id 1) (at 130.81 81.28 0))
-    (property "Footprint" "" (id 2) (at 130.81 86.36 0)
-      (effects (font (size 1.27 1.27)) hide)
-    )
-    (property "Datasheet" "" (id 3) (at 130.81 86.36 0)
-      (effects (font (size 1.27 1.27)) hide)
-    )
+  (symbol (lib_id "power:+5V") (at 111.76 86.36 0) (unit 1)
+    (in_bom yes) (on_board yes) (fields_autoplaced)
+    (property "Reference" "#PWR0911" (id 0) (at 111.76 90.17 0)
+      (effects (font (size 1.27 1.27)) hide)
+    )
+    (property "Value" "+5V" (id 1) (at 111.76 81.28 0))
+    (property "Footprint" "" (id 2) (at 111.76 86.36 0)
+      (effects (font (size 1.27 1.27)) hide)
+    )
+    (property "Datasheet" "" (id 3) (at 111.76 86.36 0)
+      (effects (font (size 1.27 1.27)) hide)
+    )
