File: pcb/cad/power-supplies.kicad_sch (KiCad schematic)
At the start: 61 parts, among them J901 Barrel_Jack_Switch, U901 LT1129CST-5, U902 LT1129CST-5, U903 R-78E5.0-0.5, U904 LT1129CST-5, U905 LT1965EMS8E_PBF, U906 LT1129CST-5, U907 LT3015EMSEPBF

Commit message: Plot gerber files, export schematic in PDF
Other:
- note added: "EXCLUDE FROM BOARD"
Changed lines of the file:
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@@
     (stroke (width 0) (type default) (color 0 0 0 0))
+  )
+  (polyline (pts (xy 20.955 29.21) (xy 20.955 194.31))
+    (stroke (width 1) (type default) (color 0 0 0 0))
   )
   (wire (pts (xy 182.88 86.36) (xy 182.88 88.9))
@@
     (stroke (width 0) (type default) (color 0 0 0 0))
   )
+  (polyline (pts (xy 20.955 194.31) (xy 165.735 194.31))
+    (stroke (width 1) (type default) (color 0 0 0 0))
+  )
   (wire (pts (xy 67.31 121.92) (xy 67.31 124.46))
     (stroke (width 0) (type default) (color 0 0 0 0))
@@
     (stroke (width 0) (type default) (color 0 0 0 0))
   )
+  (polyline (pts (xy 281.94 67.31) (xy 167.005 67.31))
+    (stroke (width 1) (type default) (color 0 0 0 0))
+  )
   (wire (pts (xy 95.25 46.99) (xy 95.25 53.34))
     (stroke (width 0) (type default) (color 0 0 0 0))
@@
     (stroke (width 0) (type default) (color 0 0 0 0))
   )
+  (polyline (pts (xy 165.735 163.83) (xy 281.94 163.83))
+    (stroke (width 1) (type default) (color 0 0 0 0))
+  )
   (wire (pts (xy 69.85 46.99) (xy 81.28 46.99))
     (stroke (width 0) (type default) (color 0 0 0 0))
@@
     (stroke (width 0) (type default) (color 0 0 0 0))
   )
+  (polyline (pts (xy 281.94 67.31) (xy 281.94 163.83))
+    (stroke (width 1) (type default) (color 0 0 0 0))
+  )
   (wire (pts (xy 228.6 57.15) (xy 236.22 57.15))
     (stroke (width 0) (type default) (color 0 0 0 0))
@@
     (stroke (width 0) (type default) (color 0 0 0 0))
   )
+  (polyline (pts (xy 167.005 67.31) (xy 167.005 29.21))
+    (stroke (width 1) (type default) (color 0 0 0 0))
+  )
   (wire (pts (xy 102.87 130.81) (xy 102.87 132.08))
     (stroke (width 0) (type default) (color 0 0 0 0))
@@
     (stroke (width 0) (type default) (color 0 0 0 0))
   )
+  (polyline (pts (xy 165.735 194.31) (xy 165.735 163.83))
+    (stroke (width 1) (type default) (color 0 0 0 0))
+  )
   (wire (pts (xy 99.06 93.98) (xy 99.06 96.52))
     (stroke (width 0) (type default) (color 0 0 0 0))
@@
   (wire (pts (xy 245.11 57.15) (xy 257.81 57.15))
     (stroke (width 0) (type default) (color 0 0 0 0))
+  )
+  (polyline (pts (xy 167.005 29.21) (xy 20.955 29.21))
+    (stroke (width 1) (type dash) (color 0 0 0 0))
   )
   (wire (pts (xy 132.08 143.51) (xy 140.97 143.51))
@@
     (effects (font (size 1 1)) (justify left bottom))
   )
+  (text "EXCLUDE FROM BOARD" (at 69.85 109.855 0)
+    (effects (font (size 10 10) (thickness 2) bold) (justify left bottom))
+  )
   (text "Optional\nto provide\nminimum\nload" (at 234.2263 87.2623 180)

Commit message: Rectify 74574 partnumber, generate HTML BOM list
Changed lines of the file:
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@@
     (effects (font (size 1 1)) (justify left bottom))
   )
-  (text "EXCLUDE FROM BOARD" (at 69.85 109.855 0)
+  (text "EXCLUDE FROM BOARD" (at 69.85 115.57 0)
     (effects (font (size 10 10) (thickness 2) bold) (justify left bottom))
   )

Commit message: Restore power supply circuit and make a separate board for it
Parts:
- added J402: Conn_01x02, TerminalBlock:TerminalBlock_bornier-2_P5.08mm, symbol Connector_Generic:Conn_01x02
- C904, C912, C916, C918, C920, C924, C927, C929, C933, C936: footprint Capacitor_SMD:C_0603_1608Metric_Pad1.08x0.95mm_HandSolder -> Capacitor_SMD:C_0805_2012Metric_Pad1.18x1.45mm_HandSolder
Connections:
- net at C907.2, C908.2, D901.2 (A2)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: now also J402.2 (Pin_2)
- net at F901.1, J901.1: now also J402.1 (Pin_1)
