File: pcb/cad/power-supplies.kicad_sch (KiCad schematic)
At the start: 61 parts, among them J901 Barrel_Jack_Switch, U901 LT1129CST-5, U902 LT1129CST-5, U903 R-78E5.0-0.5, U904 LT1129CST-5, U905 LT1965EMS8E_PBF, U906 LT1129CST-5, U907 LT3015EMSEPBF

Commit message: Add stitching capacitors to isolated supply circuits
Parts:
- added C937, C938, C939, C940, C941, C942, C943, C944: C, qds-cv-lib:C4532, symbol Device:C
- C904, C912, C916, C918, C920, C924, C927, C929, C933, C936: footprint Capacitor_SMD:C_0603_1608Metric_Pad1.08x0.95mm_HandSolder -> Capacitor_SMD:C_0805_2012Metric_Pad1.18x1.45mm_HandSolder; CNPEM Code AP107349 -> (none); Manufacturer TDK -> Kyocera; Part Number C1608X7R1H104K080AA -> 08055C104KAZ2A; Vendor Link https://br.mouser.com/ProductDetail/TDK/C1608X7R1H104K080AA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 -> (none)
Connections:
- net +15V: now also C937.1, C939.1, C941.1, C943.1
- net +15V-ISO-A: now also C937.2
- net +15V-ISO-B: now also C939.2
- net +15V-ISO-C: now also C941.2
- net +15V-ISO-D: now also C943.2
- net Earth: now also C938.1, C940.1, C942.1, C944.1
- net GND-ISO-A: now also C938.2
- net GND-ISO-B: now also C940.2
- net GND-ISO-C: now also C942.2
- net GND-ISO-D: now also C944.2

Commit message: Correct C934 polarization, rearrange JCM3012 Vin capacitors
Connections:
- net -14V: now also C934.2; no longer C934.1
- net Earth: now also C934.1; no longer C934.2
Other:
- moved on the sheet: C907, C908, C934, D901

Commit message: Replace protection flip-flop with latch, update components description generate HTML BOM list.
Parts:
- C937, C938, C939, C940, C941, C942, C943, C944: value C -> TBD
Changed lines of the file:
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@@
     (in_bom yes) (on_board yes)
     (property "Reference" "C938" (id 0) (at 216.535 65.405 90))
-    (property "Value" "C" (id 1) (at 216.535 67.945 90))
+    (property "Value" "TBD" (id 1) (at 216.535 67.945 90))
     (property "Footprint" "qds-cv-lib:C4532" (id 2) (at 217.17 62.5348 0)
       (effects (font (size 1.27 1.27)) hide)
@@
     (in_bom yes) (on_board yes)
     (property "Reference" "C941" (id 0) (at 210.82 100.965 90))
-    (property "Value" "C" (id 1) (at 210.82 103.505 90))
+    (property "Value" "TBD" (id 1) (at 210.82 103.505 90))
     (property "Footprint" "qds-cv-lib:C4532" (id 2) (at 217.17 103.8098 0)
       (effects (font (size 1.27 1.27)) hide)
@@
     (in_bom yes) (on_board yes)
     (property "Reference" "C943" (id 0) (at 210.82 132.715 90))
-    (property "Value" "C" (id 1) (at 210.82 135.255 90))
+    (property "Value" "TBD" (id 1) (at 210.82 135.255 90))
     (property "Footprint" "qds-cv-lib:C4532" (id 2) (at 217.17 135.5598 0)
       (effects (font (size 1.27 1.27)) hide)
@@
     (in_bom yes) (on_board yes)
     (property "Reference" "C939" (id 0) (at 210.82 67.945 90))
-    (property "Value" "C" (id 1) (at 210.82 70.485 90))
+    (property "Value" "TBD" (id 1) (at 210.82 70.485 90))
     (property "Footprint" "qds-cv-lib:C4532" (id 2) (at 217.17 70.7898 0)
       (effects (font (size 1.27 1.27)) hide)
@@
     (in_bom yes) (on_board yes)
     (property "Reference" "C937" (id 0) (at 210.82 36.195 90))
-    (property "Value" "C" (id 1) (at 210.82 38.735 90))
+    (property "Value" "TBD" (id 1) (at 210.82 38.735 90))
     (property "Footprint" "qds-cv-lib:C4532" (id 2) (at 217.17 39.0398 0)
       (effects (font (size 1.27 1.27)) hide)
@@
     (in_bom yes) (on_board yes)
     (property "Reference" "C940" (id 0) (at 216.535 97.155 90))
-    (property "Value" "C" (id 1) (at 216.535 99.695 90))
+    (property "Value" "TBD" (id 1) (at 216.535 99.695 90))
     (property "Footprint" "qds-cv-lib:C4532" (id 2) (at 217.17 94.2848 0)
       (effects (font (size 1.27 1.27)) hide)
@@
     (in_bom yes) (on_board yes)
     (property "Reference" "C944" (id 0) (at 216.535 161.925 90))
-    (property "Value" "C" (id 1) (at 216.535 164.465 90))
+    (property "Value" "TBD" (id 1) (at 216.535 164.465 90))
     (property "Footprint" "qds-cv-lib:C4532" (id 2) (at 217.17 159.0548 0)
       (effects (font (size 1.27 1.27)) hide)
@@
     (in_bom yes) (on_board yes)
     (property "Reference" "C942" (id 0) (at 216.535 130.175 90))
-    (property "Value" "C" (id 1) (at 216.535 132.715 90))
+    (property "Value" "TBD" (id 1) (at 216.535 132.715 90))
     (property "Footprint" "qds-cv-lib:C4532" (id 2) (at 217.17 127.3048 0)
       (effects (font (size 1.27 1.27)) hide)
