File: pcb/cad/5v-reference.kicad_sch (KiCad schematic)
At the start: 15 parts

Commit message: Update componentes fields and reference circuit
Parts:
- removed C? (x3): 100n, Capacitor_SMD:C_0603_1608Metric_Pad1.08x0.95mm_HandSolder, symbol Device:C
- added C? (x2): 1u, Capacitor_SMD:C_0805_2012Metric_Pad1.18x1.45mm_HandSolder, symbol Device:C
- added C?: 2.2u, qds-cv-lib:CP_EIA-3528-21_AVX-B_Pad1.65x2.4mm_HandSolder, symbol Device:C
- C?: value 100n -> 2.2u; footprint Capacitor_SMD:C_0603_1608Metric_Pad1.08x0.95mm_HandSolder -> qds-cv-lib:CP_EIA-3528-21_AVX-B_Pad1.65x2.4mm_HandSolder; CNPEM Code AP107349 -> AP107359; Manufacturer TDK -> Kyocera AVX; Part Number C1608X7R1H104K080AA -> TCJB225M035R0200; Vendor Link https://br.mouser.com/ProductDetail/TDK/C1608X7R1H104K080AA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 -> https://www.digikey.com/en/products/detail/TCJB225M035R0200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
- R? (x2): footprint (none) -> Resistor_SMD:R_0805_2012Metric_Pad1.20x1.40mm_HandSolder; Part Number (none) -> RC-05K203IT
- RV?: Vendor Link (none) -> https://br.mouser.com/ProductDetail/Bourns/3224X-1-502E?qs=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
- U?: value MAX6350 -> MAX6350CSA; footprint (none) -> Package_SO:SOIC-8_3.9x4.9mm_P1.27mm; CNPEM Code (none) -> AP104168; Manufacturer (none) -> Analog Devices; Part Number (none) -> Voltage References; Vendor Link (none) -> https://www.digikey.com/en/products/detail/analog-devices-i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
Connections:
- net +14V: now also C?.2
- net Earth: now also C?.1, C?.2, C?.2
- net at U?.3 (NR): now also C?.1
- net at R?.2, U?.3 (+): now also C?.1
Other:
- company: (none) -> CNPEM - Brazilian Center for Research in Energy and Materials

Commit message: Fixed footprints 3D models orientation
Parts:
- RV?: footprint Potentiometer_SMD:Potentiometer_Bourns_3224X_Vertical -> qds-cv-lib:Potentiometer_Bourns_3224X_Vertical
Other:
- moved on the sheet: R?
Changed lines of the file:
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@@
     (stroke (width 0) (type default) (color 0 0 0 0))
   )
-  (wire (pts (xy 97.79 97.79) (xy 104.14 97.79))
+  (wire (pts (xy 97.79 97.79) (xy 105.41 97.79))
     (stroke (width 0) (type default) (color 0 0 0 0))
   )
@@
     (stroke (width 0) (type default) (color 0 0 0 0))
   )
-  (wire (pts (xy 111.76 97.79) (xy 119.38 97.79))
+  (wire (pts (xy 113.03 97.79) (xy 119.38 97.79))
     (stroke (width 0) (type default) (color 0 0 0 0))
   )
@@
     (property "Reference" "RV?" (id 0) (at 90.17 71.12 90))
     (property "Value" "5k" (id 1) (at 90.17 73.66 90))
-    (property "Footprint" "Potentiometer_SMD:Potentiometer_Bourns_3224X_Vertical" (id 2) (at 90.17 77.47 0)
+    (property "Footprint" "qds-cv-lib:Potentiometer_Bourns_3224X_Vertical" (id 2) (at 90.17 77.47 0)
       (effects (font (size 1.27 1.27)) hide)
     )
@@
     (pin "3")
   )
-  (symbol (lib_id "Device:R_US") (at 107.95 97.79 90) (unit 1)
-    (in_bom yes) (on_board yes) (fields_autoplaced)
-    (property "Reference" "R?" (id 0) (at 107.95 91.44 90))
-    (property "Value" "620" (id 1) (at 107.95 93.98 90))
-    (property "Footprint" "Resistor_SMD:R_0805_2012Metric_Pad1.20x1.40mm_HandSolder" (id 2) (at 108.204 96.774 90)
-      (effects (font (size 1.27 1.27)) hide)
-    )
-    (property "Datasheet" "https://www.yageo.com/upload/media/product/productsearch/datasheet/rchip/PYu-RT_1-to-0.01_RoHS_L_13.pdf" (id 3) (at 107.95 97.79 0)
-      (effects (font (size 1.27 1.27)) hide)
-    )
-    (property "Part Number" "RT0805BRB07620RL" (id 4) (at 107.95 97.79 0)
-      (effects (font (size 1.27 1.27)) hide)
-    )
-    (property "Manufacturer" "Yageo" (id 5) (at 107.95 97.79 0)
-      (effects (font (size 1.27 1.27)) hide)
-    )
-    (property "CNPEM Code" "MC127962" (id 6) (at 107.95 97.79 0)
-      (effects (font (size 1.27 1.27)) hide)
-    )
-    (property "Vendor Link" "https://www.digikey.com/en/products/detail/yageo/RT0805BRB07620RL/5931645" (id 7) (at 107.95 97.79 0)
-      (effects (font (size 1.27 1.27)) hide)
-    )
-    (property "Description" "Resistor 620 0.1% 0.125W SMD 0805" (id 8) (at 107.95 97.79 0)
-      (effects (font (size 1.27 1.27)) hide)
-    )
+  (symbol (lib_id "Device:R_US") (at 109.22 97.79 90) (unit 1)
+    (in_bom yes) (on_board yes) (fields_autoplaced)
+    (property "Reference" "R?" (id 0) (at 109.22 91.44 90))
+    (property "Value" "620" (id 1) (at 109.22 93.98 90))
+    (property "Footprint" "Resistor_SMD:R_0805_2012Metric_Pad1.20x1.40mm_HandSolder" (id 2) (at 109.474 96.774 90)
+      (effects (font (size 1.27 1.27)) hide)
+    )
+    (property "Datasheet" "https://www.yageo.com/upload/media/product/productsearch/datasheet/rchip/PYu-RT_1-to-0.01_RoHS_L_13.pdf" (id 3) (at 109.22 97.79 0)
+      (effects (font (size 1.27 1.27)) hide)
+    )
+    (property "Part Number" "RT0805BRB07620RL" (id 4) (at 109.22 97.79 0)
+      (effects (font (size 1.27 1.27)) hide)
+    )
+    (property "Manufacturer" "Yageo" (id 5) (at 109.22 97.79 0)
+      (effects (font (size 1.27 1.27)) hide)
+    )
+    (property "CNPEM Code" "MC127962" (id 6) (at 109.22 97.79 0)
+      (effects (font (size 1.27 1.27)) hide)
+    )
+    (property "Vendor Link" "https://www.digikey.com/en/products/detail/yageo/RT0805BRB07620RL/5931645" (id 7) (at 109.22 97.79 0)
+      (effects (font (size 1.27 1.27)) hide)
+    )
+    (property "Description" "Resistor 620 0.1% 0.125W SMD 0805" (id 8) (at 109.22 97.79 0)
+      (effects (font (size 1.27 1.27)) hide)
+    )

Commit message: Update power supplies, symbols and footprint libs
Parts:
- gave numbers to parts that had none: 13
Changed lines of the file:
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@@
   (symbol (lib_id "qds-cv-lib-sym:OPA2227") (at 231.14 96.52 0) (mirror x) (unit 2)
     (in_bom yes) (on_board yes)
-    (property "Reference" "U?" (id 0) (at 233.68 100.33 0))
+    (property "Reference" "U801" (id 0) (at 233.68 100.33 0))
     (property "Value" "OPA2227" (id 1) (at 233.68 102.87 0))
     (property "Footprint" "Package_SO:SOIC-8_3.9x4.9mm_P1.27mm" (id 2) (at 231.14 96.52 0)
@@
   (symbol (lib_id "qds-cv-lib-sym:+14V") (at 195.58 88.9 0) (unit 1)
     (in_bom yes) (on_board yes) (fields_autoplaced)
-    (property "Reference" "#PWR?" (id 0) (at 195.58 92.71 0)
+    (property "Reference" "#PWR0802" (id 0) (at 195.58 92.71 0)
       (effects (font (size 1.27 1.27)) hide)
     )
@@
   (symbol (lib_id "qds-cv-lib-sym:+14V") (at 50.8 92.71 0) (unit 1)
     (in_bom yes) (on_board yes) (fields_autoplaced)
-    (property "Reference" "#PWR?" (id 0) (at 50.8 96.52 0)
+    (property "Reference" "#PWR0803" (id 0) (at 50.8 96.52 0)
       (effects (font (size 1.27 1.27)) hide)
     )
@@
   (symbol (lib_id "power:Earth") (at 195.58 109.22 0) (unit 1)
     (in_bom yes) (on_board yes) (fields_autoplaced)
-    (property "Reference" "#PWR?" (id 0) (at 195.58 115.57 0)
+    (property "Reference" "#PWR0804" (id 0) (at 195.58 115.57 0)
       (effects (font (size 1.27 1.27)) hide)
     )
@@
   (symbol (lib_id "Device:C") (at 201.93 99.06 0) (unit 1)
     (in_bom yes) (on_board yes) (fields_autoplaced)
-    (property "Reference" "C?" (id 0) (at 205.74 97.7899 0)
+    (property "Reference" "C801" (id 0) (at 205.74 97.7899 0)
       (effects (font (size 1.27 1.27)) (justify left))
     )
@@
   (symbol (lib_id "Device:R_US") (at 107.95 77.47 90) (unit 1)
     (in_bom yes) (on_board yes) (fields_autoplaced)
-    (property "Reference" "R?" (id 0) (at 107.95 71.12 90))
+    (property "Reference" "R801" (id 0) (at 107.95 71.12 90))
     (property "Value" "14k" (id 1) (at 107.95 73.66 90))
     (property "Footprint" "Resistor_SMD:R_0603_1608Metric_Pad0.98x0.95mm_HandSolder" (id 2) (at 108.204 76.454 90)
@@
   (symbol (lib_id "Device:R_US") (at 212.09 104.14 180) (unit 1)
     (in_bom yes) (on_board yes) (fields_autoplaced)
-    (property "Reference" "R?" (id 0) (at 214.63 102.8699 0)
+    (property "Reference" "R805" (id 0) (at 214.63 102.8699 0)
       (effects (font (size 1.27 1.27)) (justify right))
     )
@@
   (symbol (lib_id "power:Earth") (at 78.74 80.01 0) (unit 1)
     (in_bom yes) (on_board yes) (fields_autoplaced)
-    (property "Reference" "#PWR?" (id 0) (at 78.74 86.36 0)
+    (property "Reference" "#PWR0801" (id 0) (at 78.74 86.36 0)
       (effects (font (size 1.27 1.27)) hide)
     )
@@
   (symbol (lib_id "Reference_Voltage:MAX6350") (at 80.01 100.33 0) (unit 1)
     (in_bom yes) (on_board yes) (fields_autoplaced)
-    (property "Reference" "U?" (id 0) (at 82.0294 90.17 0)
+    (property "Reference" "U802" (id 0) (at 82.0294 90.17 0)
       (effects (font (size 1.27 1.27)) (justify left))
     )
@@
   (symbol (lib_id "Device:R_US") (at 134.62 77.47 90) (unit 1)
     (in_bom yes) (on_board yes) (fields_autoplaced)
-    (property "Reference" "R?" (id 0) (at 134.62 71.12 90))
+    (property "Reference" "R802" (id 0) (at 134.62 71.12 90))
     (property "Value" "620" (id 1) (at 134.62 73.66 90))
     (property "Footprint" "Resistor_SMD:R_0805_2012Metric_Pad1.20x1.40mm_HandSolder" (id 2) (at 134.874 76.454 90)
@@
   (symbol (lib_id "Device:C") (at 97.79 104.14 0) (mirror x) (unit 1)
     (in_bom yes) (on_board yes)
-    (property "Reference" "C?" (id 0) (at 104.14 102.87 0)
+    (property "Reference" "C804" (id 0) (at 104.14 102.87 0)
       (effects (font (size 1.27 1.27)) (justify right))
     )
@@
   (symbol (lib_id "Device:C") (at 61.595 104.14 0) (unit 1)
     (in_bom yes) (on_board yes) (fields_autoplaced)
-    (property "Reference" "C?" (id 0) (at 64.135 102.8762 0)
+    (property "Reference" "C803" (id 0) (at 64.135 102.8762 0)
       (effects (font (size 1.27 1.27)) (justify left))
     )
@@
   (symbol (lib_id "Device:R_Potentiometer_Trim_US") (at 90.17 77.47 90) (mirror x) (unit 1)
     (in_bom yes) (on_board yes) (fields_autoplaced)
-    (property "Reference" "RV?" (id 0) (at 90.17 71.12 90))
+    (property "Reference" "RV801" (id 0) (at 90.17 71.12 90))
     (property "Value" "5k" (id 1) (at 90.17 73.66 90))
     (property "Footprint" "qds-cv-lib:Potentiometer_Bourns_3224X_Vertical" (id 2) (at 90.17 77.47 0)
@@
   (symbol (lib_id "Device:R_US") (at 109.22 97.79 90) (unit 1)
     (in_bom yes) (on_board yes) (fields_autoplaced)
-    (property "Reference" "R?" (id 0) (at 109.22 91.44 90))
+    (property "Reference" "R804" (id 0) (at 109.22 91.44 90))
     (property "Value" "620" (id 1) (at 109.22 93.98 90))
     (property "Footprint" "Resistor_SMD:R_0805_2012Metric_Pad1.20x1.40mm_HandSolder" (id 2) (at 109.474 96.774 90)
@@
   (symbol (lib_id "Device:C") (at 119.38 104.14 0) (unit 1)
     (in_bom yes) (on_board yes) (fields_autoplaced)
-    (property "Reference" "C?" (id 0) (at 121.92 102.8762 0)
+    (property "Reference" "C805" (id 0) (at 121.92 102.8762 0)
       (effects (font (size 1.27 1.27)) (justify left))
     )
@@
   (symbol (lib_id "Device:R_US") (at 212.09 93.98 180) (unit 1)
     (in_bom yes) (on_board yes) (fields_autoplaced)
-    (property "Reference" "R?" (id 0) (at 214.63 92.7099 0)
+    (property "Reference" "R803" (id 0) (at 214.63 92.7099 0)
       (effects (font (size 1.27 1.27)) (justify right))
     )
@@
   (symbol (lib_id "Device:C") (at 50.8 104.14 0) (mirror x) (unit 1)
     (in_bom yes) (on_board yes)
-    (property "Reference" "C?" (id 0) (at 44.45 102.87 0)
+    (property "Reference" "C802" (id 0) (at 44.45 102.87 0)
       (effects (font (size 1.27 1.27)) (justify right))
     )
@@
   (symbol (lib_id "qds-cv-lib-sym:OPA2227") (at 193.04 99.06 0) (mirror y) (unit 3)
     (in_bom yes) (on_board yes)
-    (property "Reference" "U?" (id 0) (at 189.23 95.25 0))
+    (property "Reference" "U801" (id 0) (at 189.23 95.25 0))
     (property "Value" "OPA2227" (id 1) (at 189.23 99.06 0))
     (property "Footprint" "Package_SO:SOIC-8_3.9x4.9mm_P1.27mm" (id 2) (at 193.04 99.06 0)
@@
   (symbol (lib_id "power:Earth") (at 80.01 111.76 0) (unit 1)
     (in_bom yes) (on_board yes) (fields_autoplaced)
-    (property "Reference" "#PWR?" (id 0) (at 80.01 118.11 0)
+    (property "Reference" "#PWR0805" (id 0) (at 80.01 118.11 0)
       (effects (font (size 1.27 1.27)) hide)
     )
@@
   (symbol (lib_id "qds-cv-lib-sym:OPA2227") (at 134.62 95.25 0) (mirror x) (unit 1)
     (in_bom yes) (on_board yes)
-    (property "Reference" "U?" (id 0) (at 137.16 99.06 0))
+    (property "Reference" "U801" (id 0) (at 137.16 99.06 0))
     (property "Value" "OPA2227" (id 1) (at 137.16 101.6 0))
     (property "Footprint" "Package_SO:SOIC-8_3.9x4.9mm_P1.27mm" (id 2) (at 134.62 95.25 0)

Commit message: Add test points and extra resistors for temporary use. Remove power supplies
Parts:
- added TP501: TestPoint, symbol Connector:TestPoint
Connections:
- net +5VREF: now also TP501.1
Changed lines of the file:
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@@
   (junction (at 201.93 107.95) (diameter 0) (color 0 0 0 0)
   )
+  (junction (at 153.035 95.25) (diameter 0) (color 0 0 0 0)
+  )
   (junction (at 97.79 97.79) (diameter 0) (color 0 0 0 0)
   )
@@
     (stroke (width 0) (type default) (color 0 0 0 0))
   )
-  (wire (pts (xy 146.05 95.25) (xy 157.48 95.25))
+  (wire (pts (xy 146.05 95.25) (xy 153.035 95.25))
     (stroke (width 0) (type default) (color 0 0 0 0))
   )
@@
   )
   (wire (pts (xy 90.17 97.79) (xy 97.79 97.79))
+    (stroke (width 0) (type default) (color 0 0 0 0))
+  )
+  (wire (pts (xy 153.035 95.25) (xy 157.48 95.25))
     (stroke (width 0) (type default) (color 0 0 0 0))
   )
@@
     (pin "2")
   )
+  (symbol (lib_id "Connector:TestPoint") (at 153.035 95.25 180) (unit 1)
+    (in_bom yes) (on_board yes) (fields_autoplaced)
+    (property "Reference" "TP501" (id 0) (at 154.94 97.2819 0)
+      (effects (font (size 1.27 1.27)) (justify right))
+    )
+    (property "Value" "TestPoint" (id 1) (at 154.94 99.8219 0)
+      (effects (font (size 1.27 1.27)) (justify right))
+    )
+    (property "Footprint" "" (id 2) (at 147.955 95.25 0)
+      (effects (font (size 1.27 1.27)) hide)
+    )
+    (property "Datasheet" "~" (id 3) (at 147.955 95.25 0)
+      (effects (font (size 1.27 1.27)) hide)
+    )
+    (pin "1")
+  )
   (symbol (lib_id "Device:R_Potentiometer_Trim_US") (at 90.17 77.47 90) (mirror x) (unit 1)

Commit message: Include ISO-A power circuit, all connectors and test points on PCB
Parts:
- TP501: value TestPoint -> 5V-REF; footprint (none) -> qds-cv-lib:TestPoint_Keystone_5010-5014_Multipurpose
Changed lines of the file:
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@@
   (symbol (lib_id "Connector:TestPoint") (at 153.035 95.25 180) (unit 1)
     (in_bom yes) (on_board yes) (fields_autoplaced)
-    (property "Reference" "TP501" (id 0) (at 154.94 97.2819 0)
+    (property "Reference" "TP501" (id 0) (at 154.94 98.5519 0)
       (effects (font (size 1.27 1.27)) (justify right))
     )
-    (property "Value" "TestPoint" (id 1) (at 154.94 99.8219 0)
-      (effects (font (size 1.27 1.27)) (justify right))
+    (property "Value" "5V-REF" (id 1) (at 154.94 99.8219 0)
+      (effects (font (size 1.27 1.27)) (justify right) hide)
     )
-    (property "Footprint" "" (id 2) (at 147.955 95.25 0)
+    (property "Footprint" "qds-cv-lib:TestPoint_Keystone_5010-5014_Multipurpose" (id 2) (at 147.955 95.25 0)
       (effects (font (size 1.27 1.27)) hide)
     )
-    (property "Datasheet" "~" (id 3) (at 147.955 95.25 0)
+    (property "Datasheet" "https://www.keyelco.com/product-pdf.cfm?p=1321" (id 3) (at 147.955 95.25 0)
       (effects (font (size 1.27 1.27)) hide)
     )

Commit message: Last commit before flipping PTH components
Connections:
- net Earth: now also RV801.2, RV801.3; no longer RV801.1
- new net: R801.1, RV801.1
Other:
- moved on the sheet: RV801
Changed lines of the file:
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@@
   (junction (at 61.595 110.49) (diameter 0) (color 0 0 0 0)
   )
-  (junction (at 95.25 77.47) (diameter 0) (color 0 0 0 0)
-  )
   (junction (at 201.93 90.17) (diameter 0) (color 0 0 0 0)
   )
@@
   (junction (at 201.93 107.95) (diameter 0) (color 0 0 0 0)
   )
+  (junction (at 86.36 77.47) (diameter 0) (color 0 0 0 0)
+  )
   (junction (at 153.035 95.25) (diameter 0) (color 0 0 0 0)
   )
@@
     (stroke (width 0) (type default) (color 0 0 0 0))
   )
+  (wire (pts (xy 90.17 81.28) (xy 86.36 81.28))
+    (stroke (width 0) (type default) (color 0 0 0 0))
+  )
   (wire (pts (xy 119.38 110.49) (xy 97.79 110.49))
     (stroke (width 0) (type default) (color 0 0 0 0))
@@
     (stroke (width 0) (type default) (color 0 0 0 0))
   )
-  (wire (pts (xy 95.25 77.47) (xy 104.14 77.47))
+  (wire (pts (xy 93.98 77.47) (xy 104.14 77.47))
     (stroke (width 0) (type default) (color 0 0 0 0))
   )
@@
     (stroke (width 0) (type default) (color 0 0 0 0))
   )
-  (wire (pts (xy 90.17 81.28) (xy 95.25 81.28))
-    (stroke (width 0) (type default) (color 0 0 0 0))
-  )
   (wire (pts (xy 195.58 107.95) (xy 195.58 106.68))
     (stroke (width 0) (type default) (color 0 0 0 0))
@@
     (stroke (width 0) (type default) (color 0 0 0 0))
   )
-  (wire (pts (xy 93.98 77.47) (xy 95.25 77.47))
-    (stroke (width 0) (type default) (color 0 0 0 0))
-  )
   (wire (pts (xy 111.76 77.47) (xy 120.65 77.47))
     (stroke (width 0) (type default) (color 0 0 0 0))
@@
     (stroke (width 0) (type default) (color 0 0 0 0))
   )
+  (wire (pts (xy 86.36 81.28) (xy 86.36 77.47))
+    (stroke (width 0) (type default) (color 0 0 0 0))
+  )
   (wire (pts (xy 195.58 90.17) (xy 201.93 90.17))
     (stroke (width 0) (type default) (color 0 0 0 0))
@@
   )
   (wire (pts (xy 146.05 95.25) (xy 153.035 95.25))
-    (stroke (width 0) (type default) (color 0 0 0 0))
-  )
-  (wire (pts (xy 95.25 81.28) (xy 95.25 77.47))
     (stroke (width 0) (type default) (color 0 0 0 0))
   )
@@
     (pin "1")
   )
-  (symbol (lib_id "Device:R_Potentiometer_Trim_US") (at 90.17 77.47 90) (mirror x) (unit 1)
+  (symbol (lib_id "Device:R_Potentiometer_Trim_US") (at 90.17 77.47 270) (unit 1)
     (in_bom yes) (on_board yes) (fields_autoplaced)
     (property "Reference" "RV801" (id 0) (at 90.17 71.12 90))
