File: pcb/cad/5v-reference.kicad_sch (KiCad schematic)
At the start: 14 parts, among them U801 OPA2227, U802 MAX6350CSA

Commit message: Preliminary placement of components from detection to validation stages
Connections:
- net Earth: now also RV801.2, RV801.3; no longer RV801.1
- new net: R801.1, RV801.1
Other:
- moved on the sheet: RV801
Changed lines of the file:
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@@
   (junction (at 61.595 110.49) (diameter 0) (color 0 0 0 0)
   )
-  (junction (at 95.25 77.47) (diameter 0) (color 0 0 0 0)
-  )
   (junction (at 201.93 90.17) (diameter 0) (color 0 0 0 0)
   )
@@
   )
   (junction (at 50.8 92.71) (diameter 0) (color 0 0 0 0)
+  )
+  (junction (at 85.725 77.47) (diameter 0) (color 0 0 0 0)
   )
   (junction (at 120.65 77.47) (diameter 0) (color 0 0 0 0)
@@
     (stroke (width 0) (type default) (color 0 0 0 0))
   )
-  (wire (pts (xy 78.74 77.47) (xy 86.36 77.47))
+  (wire (pts (xy 78.74 77.47) (xy 85.725 77.47))
     (stroke (width 0) (type default) (color 0 0 0 0))
   )
@@
     (stroke (width 0) (type default) (color 0 0 0 0))
   )
-  (wire (pts (xy 95.25 77.47) (xy 104.14 77.47))
+  (wire (pts (xy 93.98 77.47) (xy 104.14 77.47))
     (stroke (width 0) (type default) (color 0 0 0 0))
   )
@@
     (stroke (width 0) (type default) (color 0 0 0 0))
   )
-  (wire (pts (xy 90.17 81.28) (xy 95.25 81.28))
-    (stroke (width 0) (type default) (color 0 0 0 0))
-  )
   (wire (pts (xy 195.58 107.95) (xy 195.58 106.68))
     (stroke (width 0) (type default) (color 0 0 0 0))
@@
     (stroke (width 0) (type default) (color 0 0 0 0))
   )
-  (wire (pts (xy 93.98 77.47) (xy 95.25 77.47))
-    (stroke (width 0) (type default) (color 0 0 0 0))
-  )
   (wire (pts (xy 111.76 77.47) (xy 120.65 77.47))
     (stroke (width 0) (type default) (color 0 0 0 0))
@@
     (stroke (width 0) (type default) (color 0 0 0 0))
   )
+  (wire (pts (xy 85.725 81.28) (xy 85.725 77.47))
+    (stroke (width 0) (type default) (color 0 0 0 0))
+  )
+  (wire (pts (xy 85.725 77.47) (xy 86.36 77.47))
+    (stroke (width 0) (type default) (color 0 0 0 0))
+  )
+  (wire (pts (xy 90.17 81.28) (xy 85.725 81.28))
+    (stroke (width 0) (type default) (color 0 0 0 0))
+  )
   (wire (pts (xy 195.58 90.17) (xy 201.93 90.17))
     (stroke (width 0) (type default) (color 0 0 0 0))
@@
   )
   (wire (pts (xy 146.05 95.25) (xy 152.4 95.25))
-    (stroke (width 0) (type default) (color 0 0 0 0))
-  )
-  (wire (pts (xy 95.25 81.28) (xy 95.25 77.47))
     (stroke (width 0) (type default) (color 0 0 0 0))
   )
@@
     (pin "2")
   )
-  (symbol (lib_id "Device:R_Potentiometer_Trim_US") (at 90.17 77.47 90) (mirror x) (unit 1)
+  (symbol (lib_id "Device:R_Potentiometer_Trim_US") (at 90.17 77.47 270) (unit 1)
     (in_bom yes) (on_board yes) (fields_autoplaced)
     (property "Reference" "RV801" (id 0) (at 90.17 71.12 90))

Commit message: Replicate detection layout for all channels, place and route 5V-REF circuit
Connections:
- net Earth: no longer RV801.2
- net at R801.1: now also RV801.2; no longer RV801.1
Changed lines of the file:
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@@
   (junction (at 50.8 92.71) (diameter 0) (color 0 0 0 0)
-  )
-  (junction (at 85.725 77.47) (diameter 0) (color 0 0 0 0)
   )
   (junction (at 120.65 77.47) (diameter 0) (color 0 0 0 0)
@@
   (no_connect (at 90.17 105.41))
   (wire (pts (xy 61.595 100.33) (xy 69.85 100.33))
+    (stroke (width 0) (type default) (color 0 0 0 0))
+  )
+  (wire (pts (xy 96.52 77.47) (xy 104.14 77.47))
     (stroke (width 0) (type default) (color 0 0 0 0))
   )
@@
     (stroke (width 0) (type default) (color 0 0 0 0))
   )
+  (wire (pts (xy 90.17 81.28) (xy 96.52 81.28))
+    (stroke (width 0) (type default) (color 0 0 0 0))
+  )
   (wire (pts (xy 80.01 111.76) (xy 80.01 110.49))
     (stroke (width 0) (type default) (color 0 0 0 0))
   )
-  (wire (pts (xy 78.74 77.47) (xy 85.725 77.47))
-    (stroke (width 0) (type default) (color 0 0 0 0))
-  )
   (wire (pts (xy 201.93 90.17) (xy 212.09 90.17))
-    (stroke (width 0) (type default) (color 0 0 0 0))
-  )
-  (wire (pts (xy 93.98 77.47) (xy 104.14 77.47))
     (stroke (width 0) (type default) (color 0 0 0 0))
   )
@@
     (stroke (width 0) (type default) (color 0 0 0 0))
   )
-  (wire (pts (xy 85.725 81.28) (xy 85.725 77.47))
-    (stroke (width 0) (type default) (color 0 0 0 0))
-  )
-  (wire (pts (xy 85.725 77.47) (xy 86.36 77.47))
-    (stroke (width 0) (type default) (color 0 0 0 0))
-  )
-  (wire (pts (xy 90.17 81.28) (xy 85.725 81.28))
+  (wire (pts (xy 78.74 77.47) (xy 86.36 77.47))
     (stroke (width 0) (type default) (color 0 0 0 0))
   )
@@
     (stroke (width 0) (type default) (color 0 0 0 0))
   )
+  (wire (pts (xy 96.52 81.28) (xy 96.52 77.47))
+    (stroke (width 0) (type default) (color 0 0 0 0))
+  )

Commit message: Improve window comparator, +5V-REF and relay driver circuits close #19 close #20 close #22
Parts:
- R801: value 14k -> 12.1k; Part Number ERA-3AEB1402V -> ERA-3AEB1212V; Vendor Link https://www.digikey.com/en/products/detail/panasonic-electronic-components/ERA-3AEB1402V/2026850 -> https://www.digikey.com/en/products/detail/panasonic-electronic-components/ERA-3AEB1212V/2026845
- R802, R804: value 620 -> 1.5k; CNPEM Code MC127962 -> AP104196; Manufacturer Yageo -> Panasonic; Part Number RT0805BRB07620RL -> ERA-6AEB152V; Vendor Link https://www.digikey.com/en/products/detail/yageo/RT0805BRB0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 -> (none)
- RV801: value 5k -> 50k; Part Number 3224X-1-502E -> 3224X-1-503E; Vendor Link https://br.mouser.com/ProductDetail/Bourns/3224X-1-502E?qs=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 -> https://br.mouser.com/ProductDetail/Bourns/3224X-1-503E?qs=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
Changed lines of the file:
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@@
     (in_bom yes) (on_board yes) (fields_autoplaced)
     (property "Reference" "R801" (id 0) (at 107.95 71.12 90))
-    (property "Value" "14k" (id 1) (at 107.95 73.66 90))
+    (property "Value" "12.1k" (id 1) (at 107.95 73.66 90))
     (property "Footprint" "Resistor_SMD:R_0603_1608Metric_Pad0.98x0.95mm_HandSolder" (id 2) (at 108.204 76.454 90)
       (effects (font (size 1.27 1.27)) hide)
@@
       (effects (font (size 1.27 1.27)) hide)
     )
-    (property "Part Number" "ERA-3AEB1402V" (id 4) (at 107.95 77.47 0)
+    (property "Part Number" "ERA-3AEB1212V" (id 4) (at 107.95 77.47 0)
       (effects (font (size 1.27 1.27)) hide)
     )
@@
       (effects (font (size 1.27 1.27)) hide)
     )
-    (property "Vendor Link" "https://www.digikey.com/en/products/detail/panasonic-electronic-components/ERA-3AEB1402V/2026850" (id 7) (at 107.95 77.47 0)
-      (effects (font (size 1.27 1.27)) hide)
-    )
-    (property "Description" "Resistor 14k 0.1% 0.1W SMD 0603" (id 8) (at 107.95 77.47 0)
+    (property "Vendor Link" "https://www.digikey.com/en/products/detail/panasonic-electronic-components/ERA-3AEB1212V/2026845" (id 7) (at 107.95 77.47 0)
+      (effects (font (size 1.27 1.27)) hide)
+    )
+    (property "Description" "Resistor 12k1 0.1% 0.1W SMD 0603" (id 8) (at 107.95 77.47 0)
       (effects (font (size 1.27 1.27)) hide)
     )
@@
     (in_bom yes) (on_board yes) (fields_autoplaced)
     (property "Reference" "R802" (id 0) (at 134.62 71.12 90))
-    (property "Value" "620" (id 1) (at 134.62 73.66 90))
+    (property "Value" "1.5k" (id 1) (at 134.62 73.66 90))
     (property "Footprint" "Resistor_SMD:R_0805_2012Metric_Pad1.20x1.40mm_HandSolder" (id 2) (at 134.874 76.454 90)
       (effects (font (size 1.27 1.27)) hide)
     )
-    (property "Datasheet" "https://www.yageo.com/upload/media/product/productsearch/datasheet/rchip/PYu-RT_1-to-0.01_RoHS_L_13.pdf" (id 3) (at 134.62 77.47 0)
-      (effects (font (size 1.27 1.27)) hide)
-    )
-    (property "Part Number" "RT0805BRB07620RL" (id 4) (at 134.62 77.47 0)
-      (effects (font (size 1.27 1.27)) hide)
-    )
-    (property "Manufacturer" "Yageo" (id 5) (at 134.62 77.47 0)
-      (effects (font (size 1.27 1.27)) hide)
-    )
-    (property "CNPEM Code" "MC127962" (id 6) (at 134.62 77.47 0)
-      (effects (font (size 1.27 1.27)) hide)
-    )
-    (property "Vendor Link" "https://www.digikey.com/en/products/detail/yageo/RT0805BRB07620RL/5931645" (id 7) (at 134.62 77.47 0)
-      (effects (font (size 1.27 1.27)) hide)
-    )
-    (property "Description" "Resistor 620 0.1% 0.125W SMD 0805" (id 8) (at 134.62 77.47 0)
+    (property "Datasheet" "https://industrial.panasonic.com/cdbs/www-data/pdf/RDM0000/AOA0000C307.pdf" (id 3) (at 134.62 77.47 0)
+      (effects (font (size 1.27 1.27)) hide)
+    )
+    (property "Part Number" "ERA-6AEB152V" (id 4) (at 134.62 77.47 0)
+      (effects (font (size 1.27 1.27)) hide)
+    )
+    (property "Manufacturer" "Panasonic" (id 5) (at 134.62 77.47 0)
+      (effects (font (size 1.27 1.27)) hide)
+    )
+    (property "CNPEM Code" "AP104196" (id 6) (at 134.62 77.47 0)
+      (effects (font (size 1.27 1.27)) hide)
+    )
+    (property "Vendor Link" "" (id 7) (at 134.62 77.47 0)
+      (effects (font (size 1.27 1.27)) hide)
+    )
+    (property "Description" "Resistor 1.5k 0.1% 0.125W SMD 0805" (id 8) (at 134.62 77.47 0)
       (effects (font (size 1.27 1.27)) hide)
     )
@@
     (in_bom yes) (on_board yes) (fields_autoplaced)
     (property "Reference" "RV801" (id 0) (at 90.17 71.12 90))
-    (property "Value" "5k" (id 1) (at 90.17 73.66 90))
+    (property "Value" "50k" (id 1) (at 90.17 73.66 90))
     (property "Footprint" "qds-cv-lib:Potentiometer_Bourns_3224X_Vertical" (id 2) (at 90.17 77.47 0)
       (effects (font (size 1.27 1.27)) hide)
@@
       (effects (font (size 1.27 1.27)) hide)
     )
-    (property "Part Number" "3224X-1-502E" (id 5) (at 90.17 77.47 0)
-      (effects (font (size 1.27 1.27)) hide)
-    )
-    (property "Description" "Trimpot 5k, 12 turns, 10% tolerance, 4mm SMD Top Adjust" (id 6) (at 90.17 77.47 0)
-      (effects (font (size 1.27 1.27)) hide)
-    )
-    (property "Vendor Link" "https://br.mouser.com/ProductDetail/Bourns/3224X-1-502E?qs=A%2FVUe%2FMZWjxlruRNznslvQ%3D%3D" (id 7) (at 90.17 77.47 0)
+    (property "Part Number" "3224X-1-503E" (id 5) (at 90.17 77.47 0)
+      (effects (font (size 1.27 1.27)) hide)
+    )
+    (property "Description" "Trimpot 50k, 12 turns, 10% tolerance, 4mm SMD Top Adjust" (id 6) (at 90.17 77.47 0)
+      (effects (font (size 1.27 1.27)) hide)
+    )
+    (property "Vendor Link" "https://br.mouser.com/ProductDetail/Bourns/3224X-1-503E?qs=A%2FVUe%2FMZWjw7UCYo8RtHVg%3D%3D" (id 7) (at 90.17 77.47 0)
       (effects (font (size 1.27 1.27)) hide)
     )
@@
     (in_bom yes) (on_board yes) (fields_autoplaced)
     (property "Reference" "R804" (id 0) (at 109.22 91.44 90))
-    (property "Value" "620" (id 1) (at 109.22 93.98 90))
+    (property "Value" "1.5k" (id 1) (at 109.22 93.98 90))
     (property "Footprint" "Resistor_SMD:R_0805_2012Metric_Pad1.20x1.40mm_HandSolder" (id 2) (at 109.474 96.774 90)
       (effects (font (size 1.27 1.27)) hide)
     )
-    (property "Datasheet" "https://www.yageo.com/upload/media/product/productsearch/datasheet/rchip/PYu-RT_1-to-0.01_RoHS_L_13.pdf" (id 3) (at 109.22 97.79 0)
-      (effects (font (size 1.27 1.27)) hide)
-    )
-    (property "Part Number" "RT0805BRB07620RL" (id 4) (at 109.22 97.79 0)
-      (effects (font (size 1.27 1.27)) hide)
-    )
-    (property "Manufacturer" "Yageo" (id 5) (at 109.22 97.79 0)
-      (effects (font (size 1.27 1.27)) hide)
-    )
-    (property "CNPEM Code" "MC127962" (id 6) (at 109.22 97.79 0)
-      (effects (font (size 1.27 1.27)) hide)
-    )
-    (property "Vendor Link" "https://www.digikey.com/en/products/detail/yageo/RT0805BRB07620RL/5931645" (id 7) (at 109.22 97.79 0)
-      (effects (font (size 1.27 1.27)) hide)
-    )
-    (property "Description" "Resistor 620 0.1% 0.125W SMD 0805" (id 8) (at 109.22 97.79 0)
-      (effects (font (size 1.27 1.27)) hide)
-    )
+    (property "Datasheet" "https://industrial.panasonic.com/cdbs/www-data/pdf/RDM0000/AOA0000C307.pdf" (id 3) (at 109.22 97.79 0)
+      (effects (font (size 1.27 1.27)) hide)
+    )
+    (property "Part Number" "ERA-6AEB152V" (id 4) (at 109.22 97.79 0)
+      (effects (font (size 1.27 1.27)) hide)
+    )
+    (property "Manufacturer" "Panasonic" (id 5) (at 109.22 97.79 0)
+      (effects (font (size 1.27 1.27)) hide)
+    )
+    (property "CNPEM Code" "AP104196" (id 6) (at 109.22 97.79 0)
+      (effects (font (size 1.27 1.27)) hide)
+    )
+    (property "Vendor Link" "" (id 7) (at 109.22 97.79 0)
+      (effects (font (size 1.27 1.27)) hide)
+    )
+    (property "Description" "Resistor 1.5k 0.1% 0.125W SMD 0805" (id 8) (at 109.22 97.79 0)
+      (effects (font (size 1.27 1.27)) hide)
+    )

Commit message: Place test-points, improve isolated circuit layout (channel D only)
Parts:
- C801: footprint Capacitor_SMD:C_0603_1608Metric_Pad1.08x0.95mm_HandSolder -> Capacitor_SMD:C_0805_2012Metric_Pad1.18x1.45mm_HandSolder; CNPEM Code AP107349 -> (none); Manufacturer TDK -> Kyocera; Part Number C1608X7R1H104K080AA -> 08055C104KAZ2A; Vendor Link https://br.mouser.com/ProductDetail/TDK/C1608X7R1H104K080AA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 -> (none)
- TP801: footprint (none) -> qds-cv-lib:TestPoint_Keystone_5010-5014_Multipurpose
Changed lines of the file:
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@@
       (effects (font (size 1.27 1.27)) (justify left))
     )
-    (property "Footprint" "Capacitor_SMD:C_0603_1608Metric_Pad1.08x0.95mm_HandSolder" (id 2) (at 202.8952 102.87 0)
-      (effects (font (size 1.27 1.27)) hide)
-    )
-    (property "Datasheet" "https://product.tdk.com/system/files/dam/doc/product/capacitor/ceramic/mlcc/catalog/mlcc_commercial_general_en.pdf" (id 3) (at 201.93 99.06 0)
-      (effects (font (size 1.27 1.27)) hide)
-    )
-    (property "CNPEM Code" "AP107349" (id 4) (at 201.93 99.06 0)
-      (effects (font (size 1.27 1.27)) hide)
-    )
-    (property "Description" "Ceramic Capacitor 100nF 50V 10% SMD 0603 X7R" (id 5) (at 201.93 99.06 0)
-      (effects (font (size 1.27 1.27)) hide)
-    )
-    (property "Manufacturer" "TDK" (id 6) (at 201.93 99.06 0)
-      (effects (font (size 1.27 1.27)) hide)
-    )
-    (property "Part Number" "C1608X7R1H104K080AA" (id 7) (at 201.93 99.06 0)
-      (effects (font (size 1.27 1.27)) hide)
-    )
-    (property "Vendor Link" "https://br.mouser.com/ProductDetail/TDK/C1608X7R1H104K080AA?qs=NRhsANhppD8dEJli2CDBHA%3D%3D" (id 8) (at 201.93 99.06 0)
+    (property "Footprint" "Capacitor_SMD:C_0805_2012Metric_Pad1.18x1.45mm_HandSolder" (id 2) (at 202.8952 102.87 0)
+      (effects (font (size 1.27 1.27)) hide)
+    )
+    (property "Datasheet" "https://spicat.kyocera-avx.com/product/mlcc/chartview/08055C104KAZ2A/DataSheet/X7R" (id 3) (at 201.93 99.06 0)
+      (effects (font (size 1.27 1.27)) hide)
+    )
+    (property "CNPEM Code" "" (id 4) (at 201.93 99.06 0)
+      (effects (font (size 1.27 1.27)) hide)
+    )
+    (property "Description" "Ceramic Capacitor 100nF 50V 10% SMD 0805 X7R" (id 5) (at 201.93 99.06 0)
+      (effects (font (size 1.27 1.27)) hide)
+    )
+    (property "Manufacturer" "Kyocera" (id 6) (at 201.93 99.06 0)
+      (effects (font (size 1.27 1.27)) hide)
+    )
+    (property "Part Number" "08055C104KAZ2A" (id 7) (at 201.93 99.06 0)
+      (effects (font (size 1.27 1.27)) hide)
+    )
+    (property "Vendor Link" "" (id 8) (at 201.93 99.06 0)
       (effects (font (size 1.27 1.27)) hide)
     )
@@
       (effects (font (size 1.27 1.27)) (justify left) hide)
     )
-    (property "Footprint" "" (id 2) (at 147.32 95.25 0)
-      (effects (font (size 1.27 1.27)) hide)
-    )
+    (property "Footprint" "qds-cv-lib:TestPoint_Keystone_5010-5014_Multipurpose" (id 2) (at 147.32 95.25 0)
+      (effects (font (size 1.27 1.27)) hide)
+    )
