File: pcb/cad/5v-reference.kicad_sch (KiCad schematic)
At the start: 14 parts, among them U801 OPA2227, U802 MAX6350CSA

Commit message: Replace protection flip-flop with latch, update components description generate HTML BOM list.
Parts:
- R803, R805: Part Number RC-05K203IT -> RC-05K203JT
- TP801: Part Number (none) -> 5012
Changed lines of the file:
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@@
       (effects (font (size 1.27 1.27)) hide)
     )
-    (property "Part Number" "RC-05K203IT" (id 4) (at 212.09 104.14 0)
+    (property "Part Number" "RC-05K203JT" (id 4) (at 212.09 104.14 0)
+      (effects (font (size 1.27 1.27)) hide)
+    )
+    (property "Description" "Resistor 20k 5% 0.1W SMD 0805" (id 5) (at 212.09 104.14 0)
       (effects (font (size 1.27 1.27)) hide)
     )
@@
       (effects (font (size 1.27 1.27)) hide)
     )
-    (property "Part Number" "RC-05K203IT" (id 4) (at 212.09 93.98 0)
+    (property "Part Number" "RC-05K203JT" (id 4) (at 212.09 93.98 0)
+      (effects (font (size 1.27 1.27)) hide)
+    )
+    (property "Description" "Resistor 20k 5% 0.1W SMD 0805" (id 5) (at 212.09 93.98 0)
       (effects (font (size 1.27 1.27)) hide)
     )
@@
       (effects (font (size 1.27 1.27)) hide)
     )
+    (property "Part Number" "5012" (id 4) (at 152.4 95.25 0)
+      (effects (font (size 1.27 1.27)) hide)
+    )

Commit message: Update component properties
Parts:
- R801: CNPEM Code AP107375 -> AP107374
Changed lines of the file:
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@@
       (effects (font (size 1.27 1.27)) hide)
     )
-    (property "CNPEM Code" "AP107375" (id 6) (at 107.95 77.47 0)
+    (property "CNPEM Code" "AP107374" (id 6) (at 107.95 77.47 0)
       (effects (font (size 1.27 1.27)) hide)
     )

Commit message: Replace tantalum capacitor symbols with polarized version close #51
Parts:
- C802, C804: symbol Device:C -> Device:C_Polarized_US
Connections:
- net +14V: now also C802.1; no longer C802.2
- net Earth: now also C802.2, C804.2; no longer C802.1, C804.1
- net at R804.1, U802.6 (OUT): now also C804.1; no longer C804.2
Changed lines of the file:
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@@
     (pin "2")
   )
-  (symbol (lib_id "Device:C") (at 97.79 104.14 0) (mirror x) (unit 1)
+  (symbol (lib_id "Device:C_Polarized_US") (at 97.79 104.14 0) (unit 1)
     (in_bom yes) (on_board yes)
-    (property "Reference" "C804" (id 0) (at 104.14 102.87 0)
+    (property "Reference" "C804" (id 0) (at 106.68 105.41 0)
       (effects (font (size 1.27 1.27)) (justify right))
     )
-    (property "Value" "2.2u" (id 1) (at 106.68 105.41 0)
+    (property "Value" "2.2u" (id 1) (at 106.045 102.87 0)
       (effects (font (size 1.27 1.27)) (justify right))
     )
-    (property "Footprint" "qds-cv-lib:CP_EIA-3528-21_AVX-B_Pad1.65x2.4mm_HandSolder" (id 2) (at 98.7552 100.33 0)
+    (property "Footprint" "qds-cv-lib:CP_EIA-3528-21_AVX-B_Pad1.65x2.4mm_HandSolder" (id 2) (at 97.79 104.14 0)
       (effects (font (size 1.27 1.27)) hide)
     )
-    (property "Datasheet" "https://datasheets.kyocera-avx.com/TCJ.pdf" (id 3) (at 97.79 104.14 0)
+    (property "Datasheet" "~" (id 3) (at 97.79 104.14 0)
       (effects (font (size 1.27 1.27)) hide)
     )
@@
     (pin "2")
   )
-  (symbol (lib_id "Device:C") (at 50.8 104.14 0) (mirror x) (unit 1)
+  (symbol (lib_id "Device:C_Polarized_US") (at 50.8 104.14 0) (unit 1)
     (in_bom yes) (on_board yes)
-    (property "Reference" "C802" (id 0) (at 44.45 102.87 0)
+    (property "Reference" "C802" (id 0) (at 46.355 105.41 0)
       (effects (font (size 1.27 1.27)) (justify right))
     )
-    (property "Value" "2.2u" (id 1) (at 46.355 105.41 0)
+    (property "Value" "2.2u" (id 1) (at 46.355 102.87 0)
       (effects (font (size 1.27 1.27)) (justify right))
     )
-    (property "Footprint" "qds-cv-lib:CP_EIA-3528-21_AVX-B_Pad1.65x2.4mm_HandSolder" (id 2) (at 51.7652 100.33 0)
+    (property "Footprint" "qds-cv-lib:CP_EIA-3528-21_AVX-B_Pad1.65x2.4mm_HandSolder" (id 2) (at 50.8 104.14 0)
       (effects (font (size 1.27 1.27)) hide)
     )
-    (property "Datasheet" "https://datasheets.kyocera-avx.com/TCJ.pdf" (id 3) (at 50.8 104.14 0)
+    (property "Datasheet" "~" (id 3) (at 50.8 104.14 0)
       (effects (font (size 1.27 1.27)) hide)
     )
