File: pcb/cad/qds-cv.kicad_pcb (KiCad board)
At the start: 2 copper layers, 219 x 159 mm, 156 parts, among them J101 DB25 Female, J102 Conn_01x08, J201 Conn_Coaxial, J301 Conn_Coaxial, J401 Conn_Coaxial, J501 Conn_Coaxial, J701 Conn_Coaxial, J702 DB9_Female, J901 Barrel_Jack_Switch, K701 FINDER-30.22, Q701 BC846B, SW601 SW_DIP_x05, SW701 RST, SW702 TRIG, U201 OPA2227, U202 AMC1200, U203 AD8421, U204 LM393-N, U601 74HC32D, U602 74HC123, U603 74HCS08, U701 74HCS08, U702 74HC574, U703 74LV132, U704 74LVC2G17, U705 74LVC2G17, U706 HFBR-1521Z, U801 OPA2227, U802 MAX6350CSA, U901 LT1129CST-5

Commit message: Update PCB layout
Parts:
- removed TP114, TP115: TestPoint, qds-cv-lib:TestPoint_Keystone_5010-5014_Multipurpose
- R601: value 1k -> 4.7k
- moved TP117 168.4 mm to (285.0, 52.4)
- moved TP116 168.4 mm to (276.9, 52.6)
- moved TP118 168.4 mm to (285.0, 62.5)
- moved R711 165.3 mm to (121.4, 141.7), turned to 0 degrees
- moved TP110 112.6 mm to (167.2, 155.4), turned to 180 degrees
- moved TP109 107.5 mm to (174.5, 155.4), turned to 180 degrees
- moved TP108 104.3 mm to (181.7, 155.4), turned to 180 degrees
- moved TP107 103.1 mm to (188.5, 155.4), turned to 180 degrees
- moved TP103 102.6 mm to (228.9, 86.1)
- moved TP119 99.0 mm to (226.7, 111.3)
- moved J102 69.3 mm to (193.9, 130.4), turned to 180 degrees
- moved TP104 67.3 mm to (247.1, 111.3)
- moved TP105 65.7 mm to (242.1, 111.3)
- moved TP106 65.2 mm to (237.0, 111.3), turned to 180 degrees
- moved R602 51.7 mm to (232.5, 124.1), turned to 180 degrees
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Connections:
- D701 pad 1: Net-(LD702-Pad1) -> Net-(D701-Pad1)
- J702 pad 1: /Quench trigger/REMOTE_RST+ -> /Quench trigger/SW_TRIG+
- J702 pad 2: /Quench trigger/SW_TRIG+ -> /Quench trigger/SW_TRIG-
- J702 pad 3: /Quench trigger/ILOCK_11 -> unconnected-(J702-Pad3)
- J702 pad 5: unconnected-(J702-Pad5) -> /Quench trigger/ILOCK_11
- J702 pad 7: /Quench trigger/SW_TRIG- -> /Quench trigger/REMOTE_RST+
- J702 pad 8: /Quench trigger/ILOCK_12 -> /Quench trigger/ILOCK_22
- J702 pad 9: /Quench trigger/ILOCK_22 -> /Quench trigger/ILOCK_12
- K701 pad A1: Net-(LD702-Pad1) -> Net-(D701-Pad1)
- LD701 pad 1: Net-(LD701-Pad1) -> Net-(R701-Pad1)
- LD701 pad 2: Net-(LD701-Pad2) -> +5V
- LD702 pad 1: Net-(LD702-Pad1) -> Net-(R702-Pad1)
- LD702 pad 2: Net-(LD702-Pad2) -> +5V
- LD703 pad 1: Net-(LD703-Pad1) -> Net-(R703-Pad1)
- LD703 pad 2: Net-(LD703-Pad2) -> +5V
- LD704 pad 1: Net-(LD704-Pad1) -> Net-(R704-Pad1)
- LD704 pad 2: Net-(LD704-Pad2) -> +5V
- LD705 pad 1: Net-(LD705-Pad1) -> Net-(R705-Pad1)
- LD705 pad 2: Net-(LD705-Pad2) -> +5V
- Q701 pad 3: Net-(LD702-Pad1) -> Net-(D701-Pad2)
- R204 pad 1: /VT1 -> /VT2
- R210 pad 1: /VT2 -> /VT1
- R701 pad 1: +5V -> Net-(R701-Pad1)
- R701 pad 2: Net-(LD701-Pad2) -> Net-(U702-Pad19)
- R702 pad 1: +5V -> Net-(R702-Pad1)
- R702 pad 2: Net-(LD702-Pad2) -> Net-(U702-Pad18)
- R703 pad 1: +5V -> Net-(R703-Pad1)
- R703 pad 2: Net-(LD703-Pad2) -> Net-(U702-Pad17)
- R704 pad 1: +5V -> Net-(R704-Pad1)
- R704 pad 2: Net-(LD704-Pad2) -> Net-(U702-Pad16)
- R705 pad 1: +5V -> Net-(R705-Pad1)
- R705 pad 2: Net-(LD705-Pad2) -> Net-(U702-Pad15)
- R707 pad 2: Net-(D701-Pad2) -> Net-(D701-Pad1)
- TP101 pad 1: /VT1 -> /VT2
- TP102 pad 1: /VT2 -> /VT1
- U702 pad 15: Net-(LD705-Pad1) -> Net-(U702-Pad15)
- U702 pad 16: Net-(LD704-Pad1) -> Net-(U702-Pad16)
- U702 pad 17: Net-(LD703-Pad1) -> Net-(U702-Pad17)
- U702 pad 18: Net-(LD702-Pad1) -> Net-(U702-Pad18)
- U702 pad 19: Net-(LD701-Pad1) -> Net-(U702-Pad19)
Routing:
- net /Quench trigger/REMOTE_RST+: track 3.50 -> 252.8 mm
- net /Quench trigger/SW_TRIG-: track 22.0 -> 177.0 mm
- net Net-(Q701-Pad1): track 0.00 -> 118.4 mm
- net Net-(U702-Pad15): track 0.00 -> 50.9 mm
- net Net-(U702-Pad16): track 0.00 -> 49.2 mm
- net Net-(U702-Pad17): track 0.00 -> 47.5 mm
- net Net-(U702-Pad18): track 0.00 -> 45.6 mm
- net Net-(U702-Pad19): track 0.00 -> 43.8 mm
- net +5V: track 29.5 -> 73.1 mm
- net Net-(U601-Pad3): track 0.00 -> 30.0 mm, vias 0 -> 2
- net +15V: track 5.69 -> 32.9 mm
- net /VT1: track 3.91 -> 26.5 mm
- net /VT2: track 3.41 -> 24.7 mm
- net /Detection validation/TRIG-CH-D: track 31.6 -> 49.5 mm
- net Net-(TP702-Pad1): track 36.9 -> 50.8 mm
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- added copper zone on B.Cu, net GND-ISO-A
- added copper zone on F.Cu, net GND-ISO-A

Commit message: Finish routing
Parts:
- added ?: , , F.Cu at (229.1, 105.9)
- added ?: , , F.Cu at (158.5, 87.1)
- SW601: value SW_DIP_x05 -> SW_DIP_x04; footprint Button_Switch_SMD:SW_DIP_SPSTx05_Slide_6.7x14.26mm_W8.61mm_P2.54mm_LowProfile -> Button_Switch_SMD:SW_DIP_SPSTx04_Slide_6.7x11.72mm_W8.61mm_P2.54mm_LowProfile
- moved TP116 124.6 mm to (176.5, 126.5)
- moved R709 105.4 mm to (223.3, 139.7), turned to 0 degrees
- moved TP117 86.1 mm to (274.8, 137.9)
- moved TP118 83.1 mm to (205.5, 86.6)
- moved TP110 46.2 mm to (203.2, 126.5)
- moved TP109 33.6 mm to (191.8, 126.5)
- moved TP119 33.2 mm to (197.4, 126.7)
- moved TP107 29.7 mm to (181.6, 126.5)
- moved TP108 29.3 mm to (186.7, 126.5)
- moved TP103 24.5 mm to (243.3, 105.9)
- moved TP111 22.7 mm to (142.8, 90.9)
- moved TP501 21.4 mm to (193.3, 86.4)
- moved C602 16.3 mm to (243.8, 101.6), turned to 0 degrees
- moved TP201 15.6 mm to (191.0, 114.3)
- moved R706 13.9 mm to (238.5, 141.5), turned to 180 degrees
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Connections:
- J102 pad 1: +14V -> +15V
- J102 pad 3: +5V -> +14V
- J102 pad 6: +15V -> +5V
- R605 pad 1: Net-(R605-Pad1) -> Net-(SW601-Pad8)
- RV201 pad 1: Net-(C212-Pad1) -> unconnected-(RV201-Pad1)
- SW601 pad 2: /Detection validation/TRIG-CH-D -> /Detection validation/TRIG-CH-C
- SW601 pad 3: /Detection validation/TRIG-CH-C -> /Detection validation/TRIG-CH-B
- SW601 pad 4: /Detection validation/TRIG-CH-B -> /Detection validation/TRIG-CH-A
- SW601 pad 5: /Detection validation/TRIG-CH-A -> Net-(R602-Pad1)
- SW601 pad 6: Net-(R602-Pad1) -> Net-(R603-Pad1)
- SW601 pad 7: Net-(R603-Pad1) -> Net-(R604-Pad1)
- SW601 pad 8: Net-(R604-Pad1) -> Net-(SW601-Pad8)
- TP107 pad 1: +14V -> +15V
- TP109 pad 1: +5V -> +14V
- TP110 pad 1: +15V -> +5V
- U704 pad 4: Net-(R712-Pad1) -> Net-(R710-Pad1)
- U704 pad 6: Net-(R706-Pad1) -> Net-(R712-Pad1)
- U705 pad 4: Net-(R710-Pad1) -> Net-(R706-Pad1)
Routing:
- net +5V: track 73.1 -> 515.1 mm, vias 0 -> 12
- net +14V: track 19.8 -> 184.8 mm, vias 0 -> 5
- net Net-(J701-Pad1): track 0.00 -> 137.8 mm, vias 0 -> 2
- net Net-(R712-Pad2): track 0.00 -> 137.6 mm, vias 0 -> 2
- net Net-(J201-Pad1): track 0.00 -> 134.1 mm, vias 0 -> 2
- net /Quench trigger/SW_TRIG+: track 9.55 -> 125.3 mm
- net /Quench trigger/SW_TRIG-: track 177.0 -> 266.6 mm, vias 0 -> 2
- net GND-ISO-A: track 90.7 -> 12.0 mm
- net -14V: track 5.75 -> 64.8 mm, vias 0 -> 2
- net +15V: track 32.9 -> 55.9 mm
- net Net-(U601-Pad3): track 30.0 -> 13.7 mm
- net Net-(Q701-Pad1): track 118.4 -> 103.6 mm
- net /+5V reference/+5VREF: track 14.3 -> 28.8 mm
- net Net-(R209-Pad1): track 11.9 -> 24.2 mm
- net Net-(TP206-Pad1): track 8.65 -> 19.7 mm
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