File: pcb/cad/qds-cv.kicad_pcb (KiCad board)
At the start: 2 copper layers, 219 x 159 mm, 156 parts, among them J101 DB25 Female, J102 Conn_01x08, J201 Conn_Coaxial, J301 Conn_Coaxial, J401 Conn_Coaxial, J501 Conn_Coaxial, J701 Conn_Coaxial, J702 DB9_Female, J901 Barrel_Jack_Switch, K701 FINDER-30.22, Q701 BC846B, SW601 SW_DIP_x04, SW701 RST, SW702 TRIG, U201 OPA2227, U202 AMC1200, U203 AD8421, U204 LM393-N, U601 74HC32D, U602 74HC123, U603 74HCS08, U701 74HCS08, U702 74HC574, U703 74LV132, U704 74LVC2G17, U705 74LVC2G17, U706 HFBR-1521Z, U801 OPA2227, U802 MAX6350CSA, U901 LT1129CST-5

Commit message: Restore power supply circuit and make a separate board for it
Parts:
- added C901: 22u, Capacitor_Tantalum_SMD:CP_EIA-6032-28_Kemet-C_Pad2.25x2.35mm_HandSolder, F.Cu at (167.7, 244.4)
- added C902: 1u, Capacitor_SMD:C_0805_2012Metric_Pad1.18x1.45mm_HandSolder, F.Cu at (164.2, 242.9)
- added C907: 100u, Capacitor_SMD:C_Elec_6.3x7.7, F.Cu at (208.1, 252.0)
- added C908: 1u, Capacitor_SMD:C_0805_2012Metric_Pad1.18x1.45mm_HandSolder, F.Cu at (213.7, 252.0)
- added C909: 22u, Capacitor_Tantalum_SMD:CP_EIA-6032-28_Kemet-C_Pad2.25x2.35mm_HandSolder, F.Cu at (167.7, 259.8)
- added C910: 1u, Capacitor_SMD:C_0805_2012Metric_Pad1.18x1.45mm_HandSolder, F.Cu at (164.2, 261.3)
- added C915: 10u, Capacitor_SMD:C_0805_2012Metric_Pad1.18x1.45mm_HandSolder, F.Cu at (172.9, 232.4)
- added C916: 100n, Capacitor_SMD:C_0805_2012Metric_Pad1.18x1.45mm_HandSolder, F.Cu at (172.9, 229.6)
- added C917: 10u, Capacitor_SMD:C_0805_2012Metric_Pad1.18x1.45mm_HandSolder, F.Cu at (172.9, 221.8)
- added C918: 100n, Capacitor_SMD:C_0805_2012Metric_Pad1.18x1.45mm_HandSolder, F.Cu at (172.9, 224.6)
- added C923: 10u, Capacitor_SMD:C_0805_2012Metric_Pad1.18x1.45mm_HandSolder, F.Cu at (151.7, 237.7)
- added C924: 100n, Capacitor_SMD:C_0805_2012Metric_Pad1.18x1.45mm_HandSolder, F.Cu at (151.7, 235.2)
- added C925: 22u, Capacitor_Tantalum_SMD:CP_EIA-6032-28_Kemet-C_Pad2.25x2.35mm_HandSolder, F.Cu at (156.8, 230.5)
- added C926: 1u, Capacitor_SMD:C_0805_2012Metric_Pad1.18x1.45mm_HandSolder, F.Cu at (152.1, 223.3)
- added C927: 100n, Capacitor_SMD:C_0805_2012Metric_Pad1.18x1.45mm_HandSolder, F.Cu at (152.1, 220.7)
- added C932: 10u, Capacitor_SMD:C_0805_2012Metric_Pad1.18x1.45mm_HandSolder, F.Cu at (141.0, 237.7)
- added C933: 100n, Capacitor_SMD:C_0805_2012Metric_Pad1.18x1.45mm_HandSolder, F.Cu at (141.0, 235.2)
- added C934: 22u, Capacitor_Tantalum_SMD:CP_EIA-6032-28_Kemet-C_Pad2.25x2.35mm_HandSolder, F.Cu at (135.7, 230.7)
- added C935: 1u, Capacitor_SMD:C_0805_2012Metric_Pad1.18x1.45mm_HandSolder, F.Cu at (140.6, 223.7)
- added C936: 100n, Capacitor_SMD:C_0805_2012Metric_Pad1.18x1.45mm_HandSolder, F.Cu at (140.6, 221.1)
- added D901: SMBJ15A, Diode_SMD:D_SMB, F.Cu at (201.0, 252.0)
- added F901: Fuse, qds-cv-lib:ZH242, F.Cu at (223.3, 252.0)
- added J103: Conn_01x08, qds-cv-lib:Edge_Pads-3.81_1x06_P3.81mm, F.Cu at (144.2, 211.5)
- added J402: Conn_01x02, TerminalBlock:TerminalBlock_bornier-2_P5.08mm, F.Cu at (236.8, 263.0)
- added PS901: JCM3012D15, qds-cv-lib:JCM30, F.Cu at (184.4, 252.0)
- added R905: 47k, Resistor_SMD:R_0603_1608Metric_Pad0.98x0.95mm_HandSolder, F.Cu at (152.1, 225.7)
- added R906: 4.42k, Resistor_SMD:R_0603_1608Metric_Pad0.98x0.95mm_HandSolder, F.Cu at (148.7, 227.4)
- added R908: 127k, Resistor_SMD:R_0603_1608Metric_Pad0.98x0.95mm_HandSolder, F.Cu at (140.4, 226.1)
- added R909: 12.1k, Resistor_SMD:R_0603_1608Metric_Pad0.98x0.95mm_HandSolder, F.Cu at (144.0, 227.4)
- added U903: R-78E5.0-0.5, Converter_DCDC:Converter_DCDC_RECOM_R-78E-0.5_THT, F.Cu at (168.0, 229.5)
- added U905: LT1965EMS8E_PBF, qds-cv-lib:SOP65P490X110-9N, F.Cu at (152.1, 230.6)
- added U907: LT3015EMSEPBF, qds-cv-lib:MSOP-12_MSE, F.Cu at (140.4, 230.6)
- C904: footprint Capacitor_SMD:C_0603_1608Metric_Pad1.08x0.95mm_HandSolder -> Capacitor_SMD:C_0805_2012Metric_Pad1.18x1.45mm_HandSolder
- moved TP701 40.0 mm to (224.5, 137.9)
- moved C202 40.0 mm to (101.2, 100.3)
- moved C208 40.0 mm to (104.5, 100.3)
- moved C903 40.0 mm to (115.4, 114.8)
- moved Q701 40.0 mm to (94.4, 151.5)
- moved R201 40.0 mm to (101.2, 95.6)
- moved R208 40.0 mm to (121.6, 100.5)
- moved TP113 40.0 mm to (109.1, 90.9)
- moved TP120 40.0 mm to (118.5, 87.1)
- moved TP206 40.0 mm to (124.6, 87.1)
- moved TP207 40.0 mm to (124.6, 108.7)
- moved C201 40.0 mm to (129.1, 96.4)
- moved C203 40.0 mm to (129.0, 104.7)
- moved C204 40.0 mm to (141.4, 93.6)
- moved C205 40.0 mm to (146.8, 106.7)
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Routing:
- net +15V: track 101.6 -> 179.4 mm, vias 1 -> 2
- net -15V: track 0.00 -> 48.3 mm, vias 0 -> 1
- net Net-(C907-Pad1): track 0.00 -> 48.2 mm
- net Net-(C907-Pad2): track 0.00 -> 44.0 mm
- net +5V: track 520.4 -> 540.9 mm
- net -14V: track 69.3 -> 88.1 mm
- net Net-(F901-Pad1): track 0.00 -> 13.5 mm
- net +14V: track 125.9 -> 137.6 mm
- net Earth: track 3.00 -> 10.2 mm, vias 24 -> 25
- net Net-(R905-Pad2): track 0.00 -> 5.73 mm
- net Net-(R908-Pad2): track 0.00 -> 5.22 mm
- added copper zone on B.Cu, net (none)
- added copper zone on F.Cu, net (none)
- added copper zone on F.Cu, net +14V
- added copper zone on F.Cu, net +15V
- added copper zone on F.Cu, net -14V
- added copper zone on B.Cu, net -15V
- added copper zone on F.Cu, net -15V
Other:
- board size 219 x 159 mm -> 219 x 229 mm
