File: pcb/cad/qds-cv.kicad_pcb (KiCad board)
At the start: 2 copper layers, 219 x 229 mm, 188 parts, among them J101 DB25 Female, J102 Conn_01x08, J103 Conn_01x08, J201 Conn_Coaxial, J301 Conn_Coaxial, J401 Conn_Coaxial, J402 Conn_01x02, J501 Conn_Coaxial, J701 Conn_Coaxial, J702 DB9_Female, J901 Barrel_Jack_Switch, K701 FINDER-30.22, Q701 BC846B, SW601 SW_DIP_x04, SW701 RST, SW702 TRIG, U201 OPA2227, U202 AMC1200, U203 AD8421, U204 LM393-N, U601 74HC32D, U602 74HC123, U603 74HCS08, U701 74HCS08, U702 74HC574, U703 74LV132, U704 74LVC2G17, U705 74LVC2G17, U706 HFBR-1521Z, U801 OPA2227, U802 MAX6350CSA, U901 LT1129CST-5, U903 R-78E5.0-0.5, U905 LT1965EMS8E_PBF, U907 LT3015EMSEPBF

Commit message: Replace tantalum capacitor symbols with polarized version
Parts:
- turned C802 to 180 degrees
- turned C804 to 0 degrees
Connections:
- C802 pad 1: Earth -> +14V
- C802 pad 2: +14V -> Earth
- C804 pad 1: Earth -> Net-(C804-Pad1)
- C804 pad 2: Net-(C804-Pad2) -> Earth
- R804 pad 1: Net-(C804-Pad2) -> Net-(C804-Pad1)
- U802 pad 6: Net-(C804-Pad2) -> Net-(C804-Pad1)
Routing:
- net Net-(C804-Pad2): track 8.57 -> 0.00 mm
- net Net-(C804-Pad1): track 0.00 -> 8.57 mm
Changed lines of the file:
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@@
   (net 16 "/Detection validation/TRIG-CH-D")
   (net 17 "Net-(C803-Pad1)")
-  (net 18 "Net-(C804-Pad2)")
+  (net 18 "Net-(C804-Pad1)")
   (net 19 "Net-(C805-Pad1)")
   (net 20 "Net-(D701-Pad2)")
@@
   )
   (footprint "qds-cv-lib:CP_EIA-3528-21_AVX-B_Pad1.65x2.4mm_HandSolder" (layer "F.Cu")
-    (at 141.8226 71.448 180)
+    (at 141.8226 71.448)
     (descr "Tantalum Capacitor SMD Kemet-B (3528-21 Metric), IPC_7351 nominal, (Body size from: http://www.kemet.com/Lists/ProductCatalog/Attachments/253/KEM_TC101_STD.pdf), generated with kicad-footprint-generator")
     (tags "capacitor tantalum")
@@
     (fp_line (start 1.75 -1.4) (end -1.05 -1.4) (layer "F.Fab") (width 0.1))
     (fp_line (start -1.75 -0.7) (end -1.75 1.4) (layer "F.Fab") (width 0.1))
-    (pad "1" smd roundrect (at -1.725 0 180) (size 1.65 2.4) (layers "F.Cu" "F.Paste" "F.Mask") (roundrect_rratio 0.1666672727)
+    (pad "1" smd roundrect (at -1.725 0) (size 1.65 2.4) (layers "F.Cu" "F.Paste" "F.Mask") (roundrect_rratio 0.1666672727)
+      (net 18 "Net-(C804-Pad1)") (pintype "passive"))
+    (pad "2" smd roundrect (at 1.725 0) (size 1.65 2.4) (layers "F.Cu" "F.Paste" "F.Mask") (roundrect_rratio 0.1666672727)
       (net 2 "Earth") (pintype "passive"))
-    (pad "2" smd roundrect (at 1.725 0 180) (size 1.65 2.4) (layers "F.Cu" "F.Paste" "F.Mask") (roundrect_rratio 0.1666672727)
-      (net 18 "Net-(C804-Pad2)") (pintype "passive"))
     (model "${KICAD6_3DMODEL_DIR}/Capacitor_Tantalum_SMD.3dshapes/CP_EIA-3528-21_Kemet-B.wrl"
       (offset (xyz 0 0 0))
@@
     (fp_line (start 1 -0.625) (end 1 0.625) (layer "F.Fab") (width 0.1))
     (pad "1" smd roundrect (at -1 0 180) (size 1.2 1.4) (layers "F.Cu" "F.Paste" "F.Mask") (roundrect_rratio 0.2083333333)
-      (net 18 "Net-(C804-Pad2)") (pintype "passive"))
+      (net 18 "Net-(C804-Pad1)") (pintype "passive"))
     (pad "2" smd roundrect (at 1 0 180) (size 1.2 1.4) (layers "F.Cu" "F.Paste" "F.Mask") (roundrect_rratio 0.2083333333)
       (net 19 "Net-(C805-Pad1)") (pintype "passive"))
@@
   )
   (footprint "qds-cv-lib:CP_EIA-3528-21_AVX-B_Pad1.65x2.4mm_HandSolder" (layer "F.Cu")
-    (at 126.3071 71.194)
+    (at 126.3071 71.194 180)
     (descr "Tantalum Capacitor SMD Kemet-B (3528-21 Metric), IPC_7351 nominal, (Body size from: http://www.kemet.com/Lists/ProductCatalog/Attachments/253/KEM_TC101_STD.pdf), generated with kicad-footprint-generator")
     (tags "capacitor tantalum")
@@
     (fp_line (start -1.75 -0.7) (end -1.75 1.4) (layer "F.Fab") (width 0.1))
     (fp_line (start 1.75 1.4) (end 1.75 -1.4) (layer "F.Fab") (width 0.1))
-    (pad "1" smd roundrect (at -1.725 0) (size 1.65 2.4) (layers "F.Cu" "F.Paste" "F.Mask") (roundrect_rratio 0.1666672727)
-      (net 2 "Earth") (pintype "passive"))
-    (pad "2" smd roundrect (at 1.725 0) (size 1.65 2.4) (layers "F.Cu" "F.Paste" "F.Mask") (roundrect_rratio 0.1666672727)
+    (pad "1" smd roundrect (at -1.725 0 180) (size 1.65 2.4) (layers "F.Cu" "F.Paste" "F.Mask") (roundrect_rratio 0.1666672727)
       (net 1 "+14V") (pintype "passive"))
+    (pad "2" smd roundrect (at 1.725 0 180) (size 1.65 2.4) (layers "F.Cu" "F.Paste" "F.Mask") (roundrect_rratio 0.1666672727)
+      (net 2 "Earth") (pintype "passive"))
     (model "${KICAD6_3DMODEL_DIR}/Capacitor_Tantalum_SMD.3dshapes/CP_EIA-3528-21_Kemet-B.wrl"
       (offset (xyz 0 0 0))
@@
       (net 92 "unconnected-(U802-Pad5)") (pinfunction "TRIM") (pintype "passive"))
     (pad "6" smd roundrect (at 2.475 0.635) (size 1.95 0.6) (layers "F.Cu" "F.Paste" "F.Mask") (roundrect_rratio 0.25)
-      (net 18 "Net-(C804-Pad2)") (pinfunction "OUT") (pintype "power_out"))
+      (net 18 "Net-(C804-Pad1)") (pinfunction "OUT") (pintype "power_out"))
     (pad "7" smd roundrect (at 2.475 -0.635) (size 1.95 0.6) (layers "F.Cu" "F.Paste" "F.Mask") (roundrect_rratio 0.25)
       (net 93 "unconnected-(U802-Pad7)") (pinfunction "NC") (pintype "no_connect"))

Commit message: Replace 74574 flip-flop with 74573 latch close #48
Parts:
- U702: value 74HC574 -> 74HC573
Changed lines of the file:
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@@
     (descr "SO-20, 12.8x7.5mm, https://www.nxp.com/docs/en/data-sheet/SA605.pdf")
     (tags "S0-20 ")
-    (property "Description" " Octal Edge-Triggered D-Flip-Flips With 3-State Outputs")
+    (property "Description" "Octal D-type 3-state transparent latch")
     (property "Manufacturer" "NXP")
-    (property "Part Number" "74HC574D")
+    (property "Part Number" "74HC573D")
     (property "Sheetfile" "quench-trigger.kicad_sch")
     (property "Sheetname" "Quench trigger")
@@
       (effects (font (size 1 1) (thickness 0.15)))
     )
-    (fp_text value "74HC574" (at 0 7.99) (layer "F.Fab")
+    (fp_text value "74HC573" (at 0 7.99) (layer "F.Fab")
       (effects (font (size 1 1) (thickness 0.15)))
     )
